File: hardware/mixer.brd (EAGLE design)
At the start: 92 x 56 mm, 86 parts, among them IC1 PGA2311, IC2 PGA2311, IC3 PGA2311, IC4 PGA2311, IC5 PGA2311, IC6 OPA2336U, K1 RT424F124, K2 RT424F124, Q1 si2305cd, Q3 IRLML9301, Q4 IRLML9301, Q5 IRLML9301, Q7 IRLML9301, T1 BC846, T2 BC846, T3 BC846, T4 BC846, U1 SPX5205 3v3, Y1 32768Hz CFPX-217 12.5pF

Commit message: add png
Parts:
- removed C23: 22pF, rcl:C0805
- removed D1, D2, D3, D4: M4, SparkFun-DiscreteSemi:SMA-DIODE
- removed K1, K2: RT424F124, relay:RT424
- removed LED1: green, led:CHIP-LED0805
- removed LED2: orange, led:CHIP-LED0805
- removed Q1: si2305cd, Simplex-DiscreteSemi:SOT23-3_POWER
- removed Q3, Q4, Q5, Q7: IRLML9301, Simplex-DiscreteSemi:SOT23-3_POWER
- removed R22: 8.2K, rcl:R0805W
- removed R27: 1K, rcl:R0805W
- removed T1, T2, T3, T4: BC846, transistor:SOT23
- removed U1: SPX5205 3v3, SparkFun:SOT23-5
- removed Y1: 32768Hz CFPX-217 12.5pF, Simplex-FreqCtrl:CRYSTAL-SMD-3.2X1.5
- added C15, C16, C18, C55, C57, C59, C61, C63: 47p, rcl:C0805
- added C19, C21, C22, C25, C26, C28, C29, C30, C31, C32, C33, C34, C35, C36, C37, C38, C39, C40, C41, C42, C43, C44, C46, C47, C48, C49, C51, C52, C53, C54, C79, C80: 100n, rcl:C0805
- added C56, C58, C60, C62, C64, C65, C66, C67, C68, C69, C70, C71, C72, C73, C74, C75, C76, C77, C78: 10u, SparkFun-Capacitors:PANASONIC_D
- added IC11, IC12, IC7, IC8, IC9: OPA2134P, burr-brown:DIL08
- added R41, R43, R45: 47K, rcl:R0805W
- added R42, R44: 1K, rcl:R0805W
- added U$2: INDUCTOR, Simplex-rlc:L0805W
- added U$3: RESETTABLE, Simplex-Fuses:1210
- added U$5: MOLEX_4HORIZONTAL, Simplex-Connectors:0530480401
- C1, C13, C14, C5, C6, C9: value 100nF -> 100n
- C10: value 470nF -> 100n
- C11: value 220nF -> 47p
- C12, C17, C7, C8: value 100nF -> 47p
- C2, C20: value 10uF -> 100n; device rcl:C1206 -> rcl:C0805
- C24: value 22pF -> 100n
- C3: value 10uF -> 47p; device rcl:C1206 -> rcl:C0805
- C4: value 1uF -> 47p
- IC6: value OPA2336U -> OPA2134P; device burr-brown:SO08 -> burr-brown:DIL08
- R1, R11, R20, R3: value 100k -> 47K
- R12, R2, R8: value 10k -> 1K
- R13, R15, R32, R9: value 100K -> 47K
- R14: value 100K -> 1K
- R16: value 100k -> 1K
- R17: value 8K -> 22K
- R18, R24, R25, R28: value 20K -> 47K
- R19, R21: value 10k -> 47K
- R23: value 160K -> 22K
- R26: value 8K -> 47K
- R29: value 8.2K -> 22K
- R30: value 160K -> 47K
- R31: value 68K -> 10
- R33: value 50 -> 10
- R34: value 47k -> 10
- R35: value 47k -> 22K
- R36, R39: value 470 -> 47K
- R37, R38: value 470 -> 10
- R4, R6: value 4.7k -> 1K
- R40: value 50 -> 47K
- R5, R7: value 4.7k -> 47K
- U$1: value F55[0/1]X---PT48 -> INDUCTOR; device TI_MSP430_v16:PT48 -> Simplex-rlc:L0805W
- U$4: value INDUCTOR -> RESETTABLE; device Simplex-rlc:L0805W -> Simplex-Fuses:1210
- moved R39 568.3 mm to (-185.3, -480.4), turned to 0 degrees
- moved R34 437.6 mm to (-173.3, -330.3), turned to 0 degrees
- moved U$1 426.0 mm to (-150.3, -324.6), turned to 0 degrees
- moved R37 424.8 mm to (-177.3, -330.3), turned to 0 degrees
- moved U$4 423.7 mm to (-154.2, -332.0)
- moved R38 417.2 mm to (-181.3, -330.3), turned to 0 degrees
- moved R35 345.0 mm to (-98.3, -263.6), turned to 0 degrees
- moved R36 328.2 mm to (-118.3, -269.7), turned to 0 degrees
- moved C24 323.1 mm to (-102.3, -222.7)
- moved R21 301.5 mm to (-110.3, -222.7)
- moved R19 296.9 mm to (-86.3, -222.7)
- moved R20 296.0 mm to (-106.3, -222.7)
- moved C17 280.5 mm to (-61.6, -195.8)
- moved R16 274.5 mm to (-66.3, -212.3)
- moved C20 267.6 mm to (-66.3, -206.2), turned to 0 degrees
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Connections:
- removed net +30V: R30.2
- removed net +3V: R32.2
- removed net +3V3: C1.1, C2.1, U1.5
- removed net -30V: R23.2
- removed net 3V: IC6.8
- removed net 41: U$1.41
- removed net 42: U$1.42
- removed net 46: U$1.46
- removed net A+3: C14.2, R31.2, R32.1, U$1.5
- removed net A+30: C13.2, R29.2, R30.1, U$1.3
- removed net A+5: C12.2, R26.2, R28.1, U$1.1
- removed net A-30: IC6.7, R25.2, R9.2, U$1.4
- removed net A-5: IC6.1, R13.2, R24.2, U$1.2
- removed net AGNDL: IC1.15, IC2.15, IC3.15, IC4.15, IC5.15
- removed net AGNDR: IC1.10, IC2.10, IC3.10, IC4.10, IC5.10
- removed net CHARGE_OFF: R20.2, U$1.19
- removed net CHARGE_ON: R16.2, U$1.18
- removed net CS: U$1.35
- removed net EN: R8.1, U$1.20
- removed net GND: C1.2, C10.2, C11.2, C12.1, C13.1, C14.1, C17.1, C2.2, C20.2, C23.2, C24.2, C3.2, C4.2, C5.1, C6.2, C7.1, C8.1, C9.1, IC6.4, LED1.C, R17.1, R22.1, R26.1, R27.1, R29.1, R31.1, R33.1, R35.2, R40.1, T1.2, T2.2, T3.2, T4.2, U$1.10, U$1.12, U$1.27, U$1.37, U$1.39, U$1.44, U1.2
- removed net LED: R10.2, U$1.36
- removed net MISO: U$1.31
- removed net N$13: R7.2, U$1.33
- removed net N$14: Q1.1, R3.1, R8.2
- removed net N$24: C5.2, R15.1, R22.2, R23.1
- removed net N$25: C24.1, U$1.9, Y1.P$1
- removed net N$3: R16.1, T1.1
- removed net N$35: D3.C, K1.A2, Q7.3, R37.1
- removed net N$39: LED2.C, R27.2
- removed net N$6: C10.1, U$1.13
- removed net P1.0: U$1.14
- removed net P1.1: U$1.15
- removed net P1.2: U$1.16
- removed net P1.3: U$1.17
- removed net P4.0: U$1.29
- removed net RST: R34.1, U$1.48
- removed net RX: R6.1
- removed net R_OFF: R11.2, U$1.22
- removed net R_ON: R1.2, U$1.21
- removed net SCK: U$1.32
- removed net SCL: R4.2
- removed net SDA: R5.2
- removed net TEST: R35.1, U$1.47
- removed net TX: R7.1
- removed net VA+: IC1.12, IC2.12, IC3.12, IC4.12, IC5.12
- removed net VA-: IC1.13, IC2.13, IC3.13, IC4.13, IC5.13
- removed net VBAT: Q3.2, Q4.2, Q5.2, Q7.2, R12.1, R19.1, R2.1, R21.1
- removed net VBAT_GND: D1.A, D2.A, D3.A, D4.A, K1.A3, K2.A3, R36.2, R37.2, R38.2, R39.2
- removed net VCC: C17.2, C8.2, C9.2, Q1.2, R3.2, R34.2, U$1.11, U$1.28, U$1.7
- removed net VCC_EN: C20.1, R4.1, R5.1, U$4.2
- removed net VD+: IC1.4, IC2.4, IC3.4, IC4.4, IC5.4
- removed net VIN: C3.1, C6.1, U1.1, U1.3
- new net AGND: C11.1, C12.1, C15.1, C16.1, C17.1, C18.1, C29.2, C3.1, C30.2, C31.2, C34.2, C35.2, C36.2, C37.2, C38.2, C39.2, C4.1, C40.2, C41.2, C42.2, C43.2, C44.2, C46.2, C47.2, C48.2, C49.2, C51.2, C52.2, C53.2, C54.2, C65.-, C66.-, C67.-, C68.-, C69.-, C7.1, C70.+, C71.+, C72.+, C73.+, C74.+, C75.-, C76.-, C77.+, C78.+, C8.1, IC1.10, IC1.15, IC2.10, IC2.15, IC3.10, IC3.15, IC4.10, IC4.15, IC5.10, IC5.15, R1.1, R11.1, R13.1, R15.1, R17.1, R23.1, R29.1, R3.1, R35.1, R41.1, R43.1, R5.1, R7.1, R9.1, U$5.3
- new net CLK: IC1.6, IC2.6, IC3.6, IC4.6, IC5.6
- new net CS1: IC1.2
- new net CS2: IC2.2
- new net CS3: IC3.2
- new net CS4: IC4.2
- new net CS5: IC5.2
- new net FRONT_L: C1.1
- new net FRONT_R: C2.1
- new net LINE_L: C9.1
- new net LINE_R: C10.1
- new net M1: IC1.8
- new net M2: IC2.8
- new net M3: IC3.8
- new net M4: IC4.8
- new net M5: IC5.8
- new net M_FRONT_L: C19.1, IC11.1, R18.1
- new net M_FRONT_R: C20.1, IC11.7, R28.1
- new net M_REAR_L: IC12.1, R30.1
- new net M_REAR_R: IC12.7, R40.1
- new net N$29: IC7.5
- new net N$33: C15.2, IC7.3, R41.2, R42.2
- new net N$36: C17.2, IC5.16, R13.2, R14.2
- new net N$40: C16.2, R43.2, R44.2
- new net N$42: C19.2, R14.1
- new net N$43: C20.2, R16.1
- new net N$46: IC11.3, R17.2
- new net N$47: IC11.2, R18.2, R19.1, R20.1, R21.1
- new net N$48: C21.1, R19.2
- new net N$49: C24.1, R20.2
- new net N$50: C22.1, R21.2
- new net N$51: IC12.6, R36.1, R40.2, R45.1
- new net N$52: IC11.5, R23.2
- new net N$53: IC11.6, R24.1, R25.1, R26.1, R28.2
- new net N$54: C25.1, R24.2
- new net N$55: C28.1, R25.2
- new net N$56: C26.1, R26.2
- new net N$58: IC12.3, R29.2
- new net N$60: U$1.1, U$3.P$1
- new net N$61: C32.1, R32.2
- new net N$62: U$2.1, U$4.P$1
- new net N$63: U$3.P$2, U$5.1
- new net N$64: IC12.5, R35.2
- new net N$66: C33.1, R36.2
- new net N$67: U$4.P$2, U$5.4
- new net N$68: IC5.4, R31.2
- new net N$69: C55.2, C56.+, IC1.1, IC1.4, R38.2
- new net N$70: C57.2, C58.+, IC2.4, R37.2
- new net N$71: C59.2, C60.+, IC3.4, R34.2
- new net N$72: C61.2, C62.+, IC4.4, R33.2
- new net N$73: C63.2, C64.+
- new net N$74: IC12.2, R30.2, R32.1, R39.1
- new net N$75: C79.1, R39.2
- new net N$77: C80.1, R45.2
- new net REAR_L: C5.1
- new net REAR_R: C6.1
- new net SPDIF_L: C13.1
- new net SPDIF_R: C14.1
- new net V_FRONT_L: C24.2, IC1.14
- new net V_FRONT_R: C28.2, IC1.11
- new net V_LINE_L: C22.2, IC3.14
- new net V_LINE_R: C26.2, IC3.11
- new net V_REAR_L: C32.2, IC2.14
- new net V_REAR_PAN_L: C79.2, IC5.14
- new net V_REAR_PAN_R: C80.2, IC5.11
- new net V_REAR_R: C33.2, IC2.11
- new net V_SPDIF_L: C21.2, IC4.14
- new net V_SPDIF_R: C25.2, IC4.11
- net +5V: now also C29.1, C30.1, C31.1, C34.1, C35.1, C36.1, C37.1, C46.1, C47.1, C48.1, C49.1, C65.+, C66.+, C67.+, C68.+, C69.+, C75.+, C76.+, IC1.12, IC11.8, IC12.8, IC2.12, IC3.12, IC4.12, IC5.12, IC6.8, IC7.8, IC8.8, IC9.8, R31.1, R33.1, R34.1, R37.1, R38.1, U$1.2; no longer R28.2
- net -5V: now also C38.1, C39.1, C40.1, C41.1, C42.1, C43.1, C44.1, C51.1, C52.1, C53.1, C54.1, C70.-, C71.-, C72.-, C73.-, C74.-, C77.-, C78.-, IC1.13, IC11.4, IC12.4, IC2.13, IC3.13, IC4.13, IC5.13, IC6.4, IC7.4, IC8.4, IC9.4, U$2.2; no longer R18.2, R24.1, R25.1
- net DGND: now also C55.1, C56.-, C57.1, C58.-, C59.1, C60.-, C61.1, C62.-, C63.1, C64.-, U$5.2
- net MOSI: now also IC1.3, IC2.3, IC3.3, IC4.3, IC5.3; no longer U$1.30
- net N$1: now also C1.2, R42.1; no longer LED1.A, R10.1
- net N$10: now also C4.2, R3.2, R4.2; no longer Q3.1, R2.2, T2.3
- net N$11: now also C5.2, R2.1; no longer R6.2, U$1.34
- net N$12: now also C6.2, R4.1; no longer D1.C, K2.A1, Q3.3, R38.1
- net N$15: now also IC3.16, IC8.1, IC8.2; no longer R11.1, T4.1
- net N$16: now also IC3.9, IC8.6, IC8.7; no longer Q5.1, R12.2, T4.3
- net N$17: now also IC7.6, IC7.7
- net N$18: now also IC8.5; no longer D4.C, K2.A2, Q5.3, R36.1
- net N$19: now also IC9.1, IC9.2; no longer IC2.11, IC2.14, IC2.16, IC2.9, IC3.11, IC3.14, IC3.16, IC3.9, IC4.11, IC4.14, IC4.9, IC5.11, IC5.14, IC5.16, IC5.9
- net N$2: now also C2.2, R44.1; no longer C4.1, U1.4
- net N$20: now also C7.2, IC8.3, R5.2, R6.2; no longer IC6.2, R13.1, R14.2
- net N$21: now also C8.2, R7.2, R8.2; no longer IC6.6, R15.2, R9.1
- net N$22: now also C9.2, R6.1; no longer IC6.3, R33.2
- net N$23: now also C10.2, R8.1; no longer IC6.5, R40.2
- net N$26: now also IC4.9, IC9.6, IC9.7; no longer C23.1, U$1.8, Y1.P$2
- net N$27: now also IC9.5; no longer C7.2, R14.1, R17.2, R18.1
- net N$28: now also C11.2, IC9.3, R10.2, R9.2; no longer Q4.1, R19.2, T1.3
- net N$30: now also C12.2, R11.2, R12.2; no longer D2.C, K1.A1, Q4.3, R39.1
- net N$31: now also C13.2, R10.1; no longer R20.1, T3.1
- net N$32: now also C14.2, R12.1; no longer Q7.1, R21.2, T3.3
- net N$37: now also C18.2, IC5.9, R15.2, R16.2; no longer Q1.3, U$4.1
- net N$4: now also IC2.16, IC6.1, IC6.2; no longer IC1.14
- net N$5: now also IC7.1, IC7.2
- net N$7: now also IC2.9, IC6.6, IC6.7; no longer C11.1, U$1.43
- net N$8: now also IC6.5; no longer R1.1, T2.1
- net N$9: now also C3.2, IC6.3, R1.2, R2.2; no longer IC1.11

Commit message: power tweaked
Parts:
- removed C55, C57, C59, C61, C63: 47p, rcl:C0805
- removed C56, C58, C60, C62, C64: 10u, SparkFun-Capacitors:PANASONIC_D
- removed R31, R33, R34, R37, R38: 10, rcl:R0805W
- added C45, C50, C81, C82, C83, C84, C85, C86: 100n, rcl:C0805
- added C87, C88, C89, C90, C91, C94: 10u, SparkFun-Capacitors:PANASONIC_D
- added U$10, U$8: RESETTABLE, Simplex-Fuses:1210
- added U$6, U$9: bead, Simplex-rlc:L0805W
- U$1, U$2: value INDUCTOR -> bead
- U$5: value MOLEX_4HORIZONTAL -> MOLEX_6HORIZONTAL; device Simplex-Connectors:0530480401 -> Simplex-Connectors:0530480610
- moved U$5 197.4 mm to (-195.2, -524.8)
Connections:
- net -5V renamed A-5V
- removed net N$10: C4.2, R3.2, R4.2
- removed net N$21: C8.2, R7.2, R8.2
- removed net N$30: C12.2, R11.2, R12.2
- removed net N$40: C16.2, R43.2, R44.2
- removed net N$67: U$4.P$2, U$5.4
- removed net N$68: IC5.4, R31.2
- removed net N$69: C55.2, C56.+, IC1.1, IC1.4, R38.2
- removed net N$70: C57.2, C58.+, IC2.4, R37.2
- removed net N$71: C59.2, C60.+, IC3.4, R34.2
- removed net N$72: C61.2, C62.+, IC4.4, R33.2
- removed net N$73: C63.2, C64.+
- new net +3V: C84.1, C85.1, C86.1, C87.-, U$9.2
- new net A+5V: C29.1, C30.1, C31.1, C34.1, C35.1, C36.1, C37.1, C46.1, C47.1, C48.1, C49.1, C65.+, C66.+, C67.+, C68.+, C69.+, C75.+, C76.+, IC1.12, IC11.8, IC12.8, IC2.12, IC3.12, IC4.12, IC5.12, IC6.8, IC7.8, IC8.8, IC9.8, U$1.2
- new net N$24: U$4.P$2, U$5.3
- new net N$25: U$5.4, U$8.P$2
- new net N$3: U$6.1, U$8.P$1
- new net N$34: U$10.P$2, U$5.5
- new net N$6: U$10.P$1, U$9.1
- net +5V: now also C45.1, C50.1, C81.1, C82.1, C83.1, C88.-, C89.-, C90.-, C91.-, C94.-, IC1.1, IC1.4, IC2.1, IC2.4, IC3.1, IC3.4, IC4.1, IC4.4, IC5.1, IC5.4, U$6.2; no longer C29.1, C30.1, C31.1, C34.1, C35.1, C36.1, C37.1, C46.1, C47.1, C48.1, C49.1, C65.+, C66.+, C67.+, C68.+, C69.+, C75.+, C76.+, IC1.12, IC11.8, IC12.8, IC2.12, IC3.12, IC4.12, IC5.12, IC6.8, IC7.8, IC8.8, IC9.8, R31.1, R33.1, R34.1, R37.1, R38.1, U$1.2
- net AGND: now also U$5.1; no longer U$5.3
- net DGND: now also C45.2, C50.2, C81.2, C82.2, C83.2, C84.2, C85.2, C86.2, C87.+, C88.+, C89.+, C90.+, C91.+, C94.+, U$5.6; no longer C55.1, C56.-, C57.1, C58.-, C59.1, C60.-, C61.1, C62.-, C63.1, C64.-, U$5.2
- net M_FRONT_L: now also C20.1; no longer C19.1
- net M_FRONT_R: now also C19.1; no longer C20.1
- net N$18: now also C8.2, R7.2, R8.2
- net N$27: now also C12.2, R11.2, R12.2
- net N$29: now also C16.2, R43.2, R44.2
- net N$63: now also U$5.2; no longer U$5.1
- net N$8: now also C4.2, R3.2, R4.2

Commit message: add msp
Parts:
- added C23: 470nF, rcl:C0805
- added C27: 220nF, rcl:C0805
- added C55, C56: 22pF, rcl:C0805
- added LED2: green, led:CHIPLED_0805
- added R22, R27: 4.7k, rcl:R0805W
- added R31, R34: 47k, rcl:R0805W
- added R33: 100k, rcl:R0805W
- added U$11: F55[0/1]X---PT48, TI_MSP430_v16:PT48
- added U$12: prog, Simplex-Connectors:0530480610
- added Y1: 32768Hz CFPX-217 12.5pF, Simplex-FreqCtrl:CRYSTAL-SMD-3.2X1.5
Connections:
- new net 41: U$11.41
- new net 42: U$11.42
- new net 46: U$11.46
- new net GND: C23.2, C27.2, C55.2, C56.2, R31.2, R33.1, U$11.10, U$11.12, U$11.27, U$11.37, U$11.44, U$12.1
- new net N$10: C23.1, U$11.13
- new net N$13: C27.1, U$11.43
- new net N$14: R22.2, U$11.34
- new net N$21: R27.2, U$11.33
- new net N$30: C56.1, U$11.9, Y1.P$1
- new net N$35: C55.1, U$11.8, Y1.P$2
- new net N$38: LED2.C, R33.2
- new net N$39: LED2.A, U$11.22
- new net RST: R34.1, U$11.48, U$12.2
- new net RX: R22.1, U$12.5
- new net TEST: R31.1, U$11.47, U$12.3
- new net TX: R27.1, U$12.6
- new net VCC: R34.2, U$11.11, U$11.28, U$11.7, U$12.4
Changed lines of the file:
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@@
 <element name="U$10" library="Simplex-Fuses" package="1210" value="RESETTABLE" x="-186.6" y="-542"/>
 <element name="C87" library="SparkFun-Capacitors" package="PANASONIC_D" value="10u" x="-192.8" y="-531.2"/>
+<element name="U$11" library="TI_MSP430_v16" package="PT48" value="F55[0/1]X---PT48" x="-187" y="-551.7"/>
+<element name="C23" library="rcl" package="C0805" value="470nF" x="-185.3" y="-560.8"/>
+<element name="C27" library="rcl" package="C0805" value="220nF" x="-181.3" y="-560.8"/>
+<element name="R22" library="rcl" package="R0805W" value="4.7k" x="-190.7" y="-570.7"/>
+<element name="R27" library="rcl" package="R0805W" value="4.7k" x="-186.7" y="-570.7"/>
+<element name="Y1" library="Simplex-FreqCtrl" package="CRYSTAL-SMD-3.2X1.5" value="32768Hz CFPX-217 12.5pF" x="-180.6" y="-574.8"/>
+<element name="C55" library="rcl" package="C0805" value="22pF" x="-177.3" y="-560.8"/>
+<element name="C56" library="rcl" package="C0805" value="22pF" x="-194.7" y="-570.7"/>
+<element name="R34" library="rcl" package="R0805W" value="47k" x="-194.7" y="-576.8"/>
+<element name="R31" library="rcl" package="R0805W" value="47k" x="-182.7" y="-570.7"/>
+<element name="U$12" library="Simplex-Connectors" package="0530480610" value="prog" x="-195.2" y="-564.6"/>
+<element name="LED2" library="led" package="CHIPLED_0805" value="green" x="-189.7" y="-575.5"/>
+<element name="R33" library="rcl" package="R0805W" value="100k" x="-178.7" y="-570.7"/>
 </elements>
 <signals>
@@
 <wire x1="-190.2" y1="-524.8" x2="-185.1" y2="-542" width="0" layer="19" extent="1-1"/>
 </signal>
+<signal name="41">
+<contactref element="U$11" pad="41"/>
+</signal>
+<signal name="42">
+<contactref element="U$11" pad="42"/>
+</signal>
+<signal name="46">
+<contactref element="U$11" pad="46"/>
+</signal>
+<signal name="GND">
+<contactref element="U$11" pad="12"/>
+<contactref element="U$11" pad="37"/>
+<contactref element="C55" pad="2"/>
+<contactref element="C56" pad="2"/>
+<contactref element="U$11" pad="27"/>
+<contactref element="U$11" pad="10"/>
+<contactref element="U$11" pad="44"/>
+<contactref element="U$12" pad="1"/>
+<contactref element="R31" pad="2"/>
+<contactref element="C23" pad="2"/>
+<contactref element="C27" pad="2"/>
+<contactref element="R33" pad="1"/>
+<wire x1="-193.75" y1="-570.7" x2="-195.2" y2="-564.6" width="0" layer="19" extent="1-1"/>
+<wire x1="-191.3" y1="-554.45" x2="-195.2" y2="-564.6" width="0" layer="19" extent="1-1"/>
+<wire x1="-191.3" y1="-553.45" x2="-191.3" y2="-554.45" width="0" layer="19" extent="1-1"/>
+<wire x1="-187.75" y1="-547.4" x2="-191.3" y2="-553.45" width="0" layer="19" extent="1-1"/>
+<wire x1="-184.25" y1="-547.4" x2="-187.75" y2="-547.4" width="0" layer="19" extent="1-1"/>
+<wire x1="-182.7" y1="-553.45" x2="-184.25" y2="-547.4" width="0" layer="19" extent="1-1"/>
+<wire x1="-184.35" y1="-560.8" x2="-182.7" y2="-553.45" width="0" layer="19" extent="1-1"/>
+<wire x1="-180.35" y1="-560.8" x2="-184.35" y2="-560.8" width="0" layer="19" extent="1-1"/>
+<wire x1="-176.35" y1="-560.8" x2="-180.35" y2="-560.8" width="0" layer="19" extent="1-1"/>
+<wire x1="-179.7525" y1="-570.7" x2="-180.35" y2="-560.8" width="0" layer="19" extent="1-1"/>
+<wire x1="-181.6475" y1="-570.7" x2="-179.7525" y2="-570.7" width="0" layer="19" extent="1-1"/>
+</signal>
+<signal name="N$10">
+<contactref element="C23" pad="1"/>
+<contactref element="U$11" pad="13"/>
+<wire x1="-189.75" y1="-556" x2="-186.25" y2="-560.8" width="0" layer="19" extent="1-1"/>
+</signal>
+<signal name="N$13">
+<contactref element="U$11" pad="43"/>
+<contactref element="C27" pad="1"/>
+<wire x1="-187.25" y1="-547.4" x2="-182.25" y2="-560.8" width="0" layer="19" extent="1-1"/>
+</signal>
+<signal name="N$14">
+<contactref element="U$11" pad="34"/>
+<contactref element="R22" pad="2"/>
+<wire x1="-182.7" y1="-549.95" x2="-189.6475" y2="-570.7" width="0" layer="19" extent="1-1"/>
+</signal>
+<signal name="N$21">
+<contactref element="U$11" pad="33"/>
+<contactref element="R27" pad="2"/>
+<wire x1="-182.7" y1="-550.45" x2="-185.6475" y2="-570.7" width="0" layer="19" extent="1-1"/>
+</signal>
+<signal name="RX">
+<contactref element="R22" pad="1"/>
+<contactref element="U$12" pad="5"/>
+<wire x1="-190.2" y1="-564.6" x2="-191.7525" y2="-570.7" width="0" layer="19" extent="1-1"/>
+</signal>
+<signal name="TX">
+<contactref element="R27" pad="1"/>
+<contactref element="U$12" pad="6"/>
+<wire x1="-188.95" y1="-564.6" x2="-187.7525" y2="-570.7" width="0" layer="19" extent="1-1"/>
+</signal>
+<signal name="N$30">
+<contactref element="C56" pad="1"/>
+<contactref element="Y1" pad="P$1"/>
+<contactref element="U$11" pad="9"/>
+<wire x1="-195.65" y1="-570.7" x2="-181.85" y2="-574.8" width="0" layer="19" extent="1-1"/>
+<wire x1="-191.3" y1="-552.95" x2="-195.65" y2="-570.7" width="0" layer="19" extent="1-1"/>
+</signal>
+<signal name="N$35">
+<contactref element="Y1" pad="P$2"/>
+<contactref element="C55" pad="1"/>
+<contactref element="U$11" pad="8"/>
+<wire x1="-178.25" y1="-560.8" x2="-179.35" y2="-574.8" width="0" layer="19" extent="1-1"/>
+<wire x1="-191.3" y1="-552.45" x2="-178.25" y2="-560.8" width="0" layer="19" extent="1-1"/>
+</signal>
+<signal name="VCC">
+<contactref element="U$11" pad="11"/>
+<contactref element="R34" pad="2"/>
+<contactref element="U$12" pad="4"/>
+<contactref element="U$11" pad="7"/>
+<contactref element="U$11" pad="28"/>
+<wire x1="-191.3" y1="-553.95" x2="-191.45" y2="-564.6" width="0" layer="19" extent="1-1"/>
+<wire x1="-191.3" y1="-551.95" x2="-191.3" y2="-553.95" width="0" layer="19" extent="1-1"/>
+<wire x1="-182.7" y1="-552.95" x2="-191.3" y2="-553.95" width="0" layer="19" extent="1-1"/>
+<wire x1="-193.6475" y1="-576.8" x2="-191.45" y2="-564.6" width="0" layer="19" extent="1-1"/>
+</signal>
+<signal name="RST">
+<contactref element="U$11" pad="48"/>
+<contactref element="R34" pad="1"/>
+<contactref element="U$12" pad="2"/>
+<wire x1="-195.7525" y1="-576.8" x2="-193.95" y2="-564.6" width="0" layer="19" extent="1-1"/>
+<wire x1="-189.75" y1="-547.4" x2="-193.95" y2="-564.6" width="0" layer="19" extent="1-1"/>
+</signal>
+<signal name="TEST">
+<contactref element="U$11" pad="47"/>
+<contactref element="R31" pad="1"/>
+<contactref element="U$12" pad="3"/>
+<wire x1="-183.7525" y1="-570.7" x2="-192.7" y2="-564.6" width="0" layer="19" extent="1-1"/>
+<wire x1="-189.25" y1="-547.4" x2="-192.7" y2="-564.6" width="0" layer="19" extent="1-1"/>
+</signal>
+<signal name="N$38">
+<contactref element="LED2" pad="C"/>
+<contactref element="R33" pad="2"/>
+<wire x1="-189.7" y1="-574.45" x2="-177.6475" y2="-570.7" width="0" layer="19" extent="1-1"/>
+</signal>
+<signal name="N$39">
+<contactref element="LED2" pad="A"/>
+<contactref element="U$11" pad="22"/>
+<wire x1="-189.7" y1="-576.55" x2="-185.25" y2="-556" width="0" layer="19" extent="1-1"/>
+</signal>
 </signals>

Commit message: change C footprints
Parts:
- removed C94: 10u, SparkFun-Capacitors:PANASONIC_D
- removed U$12: prog, Simplex-Connectors:0530480610
- removed U$5: MOLEX_6HORIZONTAL, Simplex-Connectors:0530480610
- added C57: 100nF, rcl:C0805
- added C58, C59, C60, C61, C62: 100n, rcl:C0805
- added C64: 10u, rcl:153CLV-0405
- added Q1: SI2305, Simplex-DiscreteSemi:SOT23-3_POWER
- added Q2: MOSFET-NCHANNEL_SOT23-3, Simplex-DiscreteSemi:SOT23-3
- added R37, R38, R46: 10K, rcl:R0805W
- added R47, R48, R49, R50, R51: 47K, rcl:R0805W
- added X1: MOLEX_6HORIZONTAL, Simplex-Connectors:0530480610
- added X2: MOLEX_6VERTICAL, Simplex-Connectors:0530470610
- added X3: MOLEX_4VERTICAL, Simplex-Connectors:0530470410
- C65, C66, C67, C68, C69, C70, C71, C72, C73, C74, C75, C76, C77, C78, C87, C88, C89, C90, C91: device SparkFun-Capacitors:PANASONIC_D -> rcl:153CLV-0405
- R22, R27: value 4.7k -> 2.2K
- moved C65 274.3 mm to (-264.3, -656.4)
- moved C66 269.9 mm to (-270.7, -656.4)
- moved C67 265.8 mm to (-277.1, -656.4)
- moved C73 262.5 mm to (-315.5, -656.4)
- moved C68 261.9 mm to (-283.5, -656.4)
- moved C71 261.7 mm to (-302.7, -656.4)
- moved C69 258.3 mm to (-289.9, -656.4)
- moved C74 256.0 mm to (-321.9, -656.4)
- moved C72 255.1 mm to (-309.1, -656.4)
- moved C70 255.0 mm to (-296.3, -656.4)
- moved C90 254.0 mm to (-366.7, -656.4)
- moved C75 254.0 mm to (-328.3, -656.4)
- moved C76 252.3 mm to (-334.7, -656.4)
- moved C77 250.9 mm to (-341.1, -656.4)
- moved C78 249.9 mm to (-347.5, -656.4)
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Connections:
- removed net +5V: C45.1, C50.1, C81.1, C82.1, C83.1, C88.-, C89.-, C90.-, C91.-, C94.-, IC1.1, IC1.4, IC2.1, IC2.4, IC3.1, IC3.4, IC4.1, IC4.4, IC5.1, IC5.4, U$6.2
- removed net GND: C23.2, C27.2, C55.2, C56.2, R31.2, R33.1, U$11.10, U$11.12, U$11.27, U$11.37, U$11.44, U$12.1
- new net +5V_DIG: Q1.2, R37.2, U$6.2
- new net +5V_PGA: C45.1, C50.1, C57.2, C78.+, C81.1, C82.1, C83.1, C88.+, C89.+, C90.+, C91.+, IC1.1, IC1.4, IC2.1, IC2.4, IC3.1, IC3.4, IC4.1, IC4.4, IC5.1, IC5.4, Q1.3
- new net N$40: C57.1, Q1.1, Q2.3, R37.1
- new net N$41: Q2.1, R38.2, R46.1
- new net N$44: IC1.7, R49.1
- new net N$45: IC3.7, R47.1
- new net N$57: IC2.7, R48.1
- new net N$59: IC4.7, R50.1
- new net N$65: IC5.7, R51.1
- new net PGA_EN: R46.2
- net +3V: now also C87.+; no longer C87.-
- net A+5V: now also C58.2, C59.2, C60.2, C61.2, C62.2, C64.+, C70.+; no longer C75.+, C76.+
- net A-5V: now also C58.1, C59.1, C60.1, C61.1, C62.1, C75.-, C76.-; no longer C70.-, C78.-
- net AGND: now also C64.-, C70.-, C75.+, C76.+, X2.1; no longer C70.+, C75.-, C76.-, C78.+, U$5.1
- net DGND: now also C23.2, C27.2, C55.2, C56.2, C78.-, C87.-, C88.-, C89.-, C90.-, C91.-, Q2.2, R31.2, R33.1, R38.1, R47.2, R48.2, R49.2, R50.2, R51.2, U$11.10, U$11.12, U$11.27, U$11.37, U$11.44, X1.1, X2.6, X3.1, X3.4; no longer C87.+, C88.+, C89.+, C90.+, C91.+, C94.+, U$5.6
- net N$24: now also X2.3; no longer U$5.3
- net N$25: now also X2.4; no longer U$5.4
- net N$34: now also X2.5; no longer U$5.5
- net N$63: now also X2.2; no longer U$5.2
- net RST: now also X1.2; no longer U$12.2
- net RX: now also X1.5, X3.2; no longer U$12.5
- net TEST: now also X1.3; no longer U$12.3
- net TX: now also X1.6, X3.3; no longer U$12.6
- net VCC: now also X1.4; no longer U$12.4

Commit message: change input filters
Parts:
- removed C21, C22, C24, C25, C26, C28, C32, C33, C79, C80: 100n, rcl:C0805
- added R52, R53, R54, R55, R56, R57, R58, R59, R60, R61: 100K, rcl:R0805W
- C1, C10, C13, C14, C19, C2, C20, C5, C6, C9: value 100n -> 10u
- C11, C12, C15, C16, C17, C18, C3, C4, C7, C8: value 47p -> 1n
- R1, R11, R13, R15, R3, R41, R43, R5, R7, R9: value 47K -> 100K
- R17, R23, R29, R35: value 22K -> 5K
- R18, R19, R20, R21, R24, R25, R26, R28, R30, R32, R36, R39, R40, R45: value 47K -> 10K
Connections:
- removed net N$48: C21.1, R19.2
- removed net N$49: C24.1, R20.2
- removed net N$50: C22.1, R21.2
- removed net N$54: C25.1, R24.2
- removed net N$55: C28.1, R25.2
- removed net N$56: C26.1, R26.2
- removed net N$61: C32.1, R32.2
- removed net N$66: C33.1, R36.2
- removed net N$75: C79.1, R39.2
- removed net N$77: C80.1, R45.2
- net AGND: now also R52.1, R53.1, R54.1, R55.1, R56.1, R57.1, R58.1, R59.1, R60.1, R61.1
- net FRONT_L: now also R60.2
- net FRONT_R: now also R61.2
- net LINE_L: now also R54.2
- net LINE_R: now also R55.2
- net M_FRONT_L: now also R59.2
- net M_FRONT_R: now also R58.2
- net REAR_L: now also R52.2
- net REAR_R: now also R53.2
- net SPDIF_L: now also R56.2
- net SPDIF_R: now also R57.2
- net V_FRONT_L: now also R20.2; no longer C24.2
- net V_FRONT_R: now also R25.2; no longer C28.2
- net V_LINE_L: now also R21.2; no longer C22.2
- net V_LINE_R: now also R26.2; no longer C26.2
- net V_REAR_L: now also R32.2; no longer C32.2
- net V_REAR_PAN_L: now also R39.2; no longer C79.2
- net V_REAR_PAN_R: now also R45.2; no longer C80.2
- net V_REAR_R: now also R36.2; no longer C33.2
- net V_SPDIF_L: now also R19.2; no longer C21.2
- net V_SPDIF_R: now also R24.2; no longer C25.2
