File: hardware/mixer.brd (EAGLE design)
At the start: 92 x 56 mm, 169 parts, among them IC1 PGA2311, IC11 OPA2134P, IC12 OPA2134P, IC2 PGA2311, IC3 PGA2311, IC4 PGA2311, IC5 PGA2311, IC6 OPA2134P, IC7 OPA2134P, IC8 OPA2134P, IC9 OPA2134P, Q1 SI2305, Q2 MOSFET-NCHANNEL_SOT23-3, X1 MOLEX_6HORIZONTAL, X2 MOLEX_6VERTICAL, X3 MOLEX_4VERTICAL, Y1 32768Hz CFPX-217 12.5pF

Commit message: add jumper for pan input
Parts:
- removed C17, C18: 1n, rcl:C0805
- removed C19, C20: 10u, rcl:C0805
- removed R13, R15, R58, R59: 100K, rcl:R0805W
- removed R14, R16: 1K, rcl:R0805W
- added JP1, JP2: (no value), SparkFun-Connectors:1X03
- R17, R23, R29, R35: value 5K -> 4K7
Connections:
- removed net N$37: C18.2, IC5.9, R15.2, R16.2
- removed net N$43: C20.2, R16.1
- net AGND: no longer C17.1, C18.1, R13.1, R15.1, R58.1, R59.1
- net M_FRONT_L: now also JP1.3, JP2.1; no longer C20.1, R59.2
- net M_FRONT_R: now also JP1.1, JP2.3; no longer C19.1, R58.2
- net N$36: now also JP1.2; no longer C17.2, R13.2, R14.2
- net N$42: now also IC5.9, JP2.2; no longer C19.2, R14.1
Changed lines of the file:
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@@
 <element name="C13" library="rcl" package="C0805" value="10u" x="-70.3" y="-183.6"/>
 <element name="C14" library="rcl" package="C0805" value="10u" x="-66.3" y="-183.6"/>
-<element name="R13" library="rcl" package="R0805W" value="100K" x="-62.3" y="-206.2"/>
-<element name="C17" library="rcl" package="C0805" value="1n" x="-61.6" y="-195.8"/>
-<element name="R14" library="rcl" package="R0805W" value="1K" x="-74.3" y="-212.3"/>
-<element name="R15" library="rcl" package="R0805W" value="100K" x="-70.3" y="-212.3"/>
-<element name="C18" library="rcl" package="C0805" value="1n" x="-74.3" y="-206.2"/>
-<element name="R16" library="rcl" package="R0805W" value="1K" x="-66.3" y="-212.3"/>
-<element name="C19" library="rcl" package="C0805" value="10u" x="-70.3" y="-206.2"/>
-<element name="C20" library="rcl" package="C0805" value="10u" x="-66.3" y="-206.2"/>
 <element name="IC11" library="burr-brown" package="DIL08" value="OPA2134P" x="-68.8" y="-220.6">
 <attribute name="OC_NEWARK" value="74K3897" x="-68.8" y="-220.6" size="1.778" layer="27" display="off"/>
@@
 <attribute name="OC_FARNELL" value="1097574" x="-68.8" y="-220.6" size="1.778" layer="27" display="off"/>
 </element>
-<element name="R17" library="rcl" package="R0805W" value="5K" x="-78.3" y="-222.7"/>
+<element name="R17" library="rcl" package="R0805W" value="4K7" x="-78.3" y="-222.7"/>
 <element name="R18" library="rcl" package="R0805W" value="10K" x="-82.3" y="-222.7"/>
 <element name="R19" library="rcl" package="R0805W" value="10K" x="-86.3" y="-222.7"/>
 <element name="R20" library="rcl" package="R0805W" value="10K" x="-106.3" y="-222.7"/>
 <element name="R21" library="rcl" package="R0805W" value="10K" x="-110.3" y="-222.7"/>
-<element name="R23" library="rcl" package="R0805W" value="5K" x="-110.3" y="-234.9"/>
+<element name="R23" library="rcl" package="R0805W" value="4K7" x="-110.3" y="-234.9"/>
 <element name="R24" library="rcl" package="R0805W" value="10K" x="-106.3" y="-234.9"/>
 <element name="R25" library="rcl" package="R0805W" value="10K" x="-114.3" y="-241"/>
@@
 <attribute name="OC_FARNELL" value="1097574" x="-112.8" y="-249.3" size="1.778" layer="27" display="off"/>
 </element>
-<element name="R29" library="rcl" package="R0805W" value="5K" x="-98.3" y="-257.5"/>
+<element name="R29" library="rcl" package="R0805W" value="4K7" x="-98.3" y="-257.5"/>
 <element name="R30" library="rcl" package="R0805W" value="10K" x="-118.3" y="-263.6"/>
 <element name="R32" library="rcl" package="R0805W" value="10K" x="-110.3" y="-263.6"/>
-<element name="R35" library="rcl" package="R0805W" value="5K" x="-98.3" y="-263.6"/>
+<element name="R35" library="rcl" package="R0805W" value="4K7" x="-98.3" y="-263.6"/>
 <element name="R36" library="rcl" package="R0805W" value="10K" x="-118.3" y="-269.7"/>
 <element name="R40" library="rcl" package="R0805W" value="10K" x="-102.3" y="-269.7"/>
@@
 <element name="R56" library="rcl" package="R0805W" value="100K" x="-380.6" y="-688.1"/>
 <element name="R57" library="rcl" package="R0805W" value="100K" x="-380.6" y="-694.2"/>
-<element name="R58" library="rcl" package="R0805W" value="100K" x="-380.6" y="-700.3"/>
-<element name="R59" library="rcl" package="R0805W" value="100K" x="-380.6" y="-706.4"/>
 <element name="R60" library="rcl" package="R0805W" value="100K" x="-380.6" y="-712.5"/>
 <element name="R61" library="rcl" package="R0805W" value="100K" x="-380.6" y="-718.6"/>
+<element name="JP1" library="SparkFun-Connectors" package="1X03" value="" x="-380.7" y="-725.2"/>
+<element name="JP2" library="SparkFun-Connectors" package="1X03" value="" x="-380.7" y="-730.1"/>
 </elements>
 <signals>
@@
 <contactref element="R11" pad="1"/>
 <contactref element="C12" pad="1"/>
-<contactref element="R13" pad="1"/>
-<contactref element="C17" pad="1"/>
-<contactref element="R15" pad="1"/>
-<contactref element="C18" pad="1"/>
 <contactref element="R17" pad="1"/>
 <contactref element="R23" pad="1"/>
@@
 <contactref element="R56" pad="1"/>
 <contactref element="R57" pad="1"/>
-<contactref element="R58" pad="1"/>
-<contactref element="R59" pad="1"/>
 <contactref element="R60" pad="1"/>
 <contactref element="R61" pad="1"/>
@@
 <wire x1="-63.3525" y1="-138.4" x2="-71.3525" y2="-144.5" width="0" layer="19" extent="1-1"/>
 <wire x1="-62.55" y1="-128" x2="-63.3525" y2="-138.4" width="0" layer="19" extent="1-1"/>
-<wire x1="-62.55" y1="-195.8" x2="-71.3525" y2="-189.7" width="0" layer="19" extent="1-1"/>
-<wire x1="-63.3525" y1="-206.2" x2="-62.55" y2="-195.8" width="0" layer="19" extent="1-1"/>
-<wire x1="-71.3525" y1="-212.3" x2="-63.3525" y2="-206.2" width="0" layer="19" extent="1-1"/>
-<wire x1="-75.25" y1="-206.2" x2="-71.3525" y2="-212.3" width="0" layer="19" extent="1-1"/>
 <wire x1="-63.3525" y1="-115.8" x2="-62.55" y2="-128" width="0" layer="19" extent="1-1"/>
 <wire x1="-67.25" y1="-115.8" x2="-63.3525" y2="-115.8" width="0" layer="19" extent="1-1"/>
 <wire x1="-63.25" y1="-109.7" x2="-63.3525" y2="-115.8" width="0" layer="19" extent="1-1"/>
 <wire x1="-59.3525" y1="-109.7" x2="-63.25" y2="-109.7" width="0" layer="19" extent="1-1"/>
-<wire x1="-79.3525" y1="-222.7" x2="-71.3525" y2="-212.3" width="0" layer="19" extent="1-1"/>
+<wire x1="-79.3525" y1="-222.7" x2="-71.3525" y2="-189.7" width="0" layer="19" extent="1-1"/>
 <wire x1="-111.3525" y1="-234.9" x2="-79.3525" y2="-222.7" width="0" layer="19" extent="1-1"/>
 <wire x1="-99.3525" y1="-257.5" x2="-111.3525" y2="-234.9" width="0" layer="19" extent="1-1"/>
@@
 <wire x1="-381.6525" y1="-688.1" x2="-381.6525" y2="-682" width="0" layer="19" extent="1-1"/>
 <wire x1="-381.6525" y1="-694.2" x2="-381.6525" y2="-688.1" width="0" layer="19" extent="1-1"/>
-<wire x1="-381.6525" y1="-700.3" x2="-381.6525" y2="-694.2" width="0" layer="19" extent="1-1"/>
-<wire x1="-381.6525" y1="-706.4" x2="-381.6525" y2="-700.3" width="0" layer="19" extent="1-1"/>
-<wire x1="-381.6525" y1="-712.5" x2="-381.6525" y2="-706.4" width="0" layer="19" extent="1-1"/>
+<wire x1="-381.6525" y1="-712.5" x2="-381.6525" y2="-694.2" width="0" layer="19" extent="1-1"/>
 <wire x1="-381.6525" y1="-718.6" x2="-381.6525" y2="-712.5" width="0" layer="19" extent="1-1"/>
 </signal>
@@
 <signal name="N$36">
 <contactref element="IC5" pad="16"/>
-<contactref element="R13" pad="2"/>
-<contactref element="C17" pad="2"/>
-<contactref element="R14" pad="2"/>
-<wire x1="-60.65" y1="-195.8" x2="0.555" y2="-47.8" width="0" layer="19" extent="1-1"/>
-<wire x1="-61.2475" y1="-206.2" x2="-60.65" y2="-195.8" width="0" layer="19" extent="1-1"/>
-<wire x1="-73.2475" y1="-212.3" x2="-61.2475" y2="-206.2" width="0" layer="19" extent="1-1"/>
-</signal>
-<signal name="N$37">
-<contactref element="IC5" pad="9"/>
-<contactref element="R15" pad="2"/>
-<contactref element="C18" pad="2"/>
-<contactref element="R16" pad="2"/>
-<wire x1="-73.35" y1="-206.2" x2="9.445" y2="-47.8" width="0" layer="19" extent="1-1"/>
-<wire x1="-69.2475" y1="-212.3" x2="-73.35" y2="-206.2" width="0" layer="19" extent="1-1"/>
-<wire x1="-65.2475" y1="-212.3" x2="-69.2475" y2="-212.3" width="0" layer="19" extent="1-1"/>
-</signal>
-<signal name="N$42">
-<contactref element="R14" pad="1"/>
-<contactref element="C19" pad="2"/>
-<wire x1="-69.35" y1="-206.2" x2="-75.3525" y2="-212.3" width="0" layer="19" extent="1-1"/>
-</signal>
-<signal name="N$43">
-<contactref element="R16" pad="1"/>
-<contactref element="C20" pad="2"/>
-<wire x1="-65.35" y1="-206.2" x2="-67.3525" y2="-212.3" width="0" layer="19" extent="1-1"/>
+<contactref element="JP1" pad="2"/>
+<wire x1="0.555" y1="-47.8" x2="-378.16" y2="-725.2" width="0" layer="19" extent="1-1"/>
 </signal>
 <signal name="N$46">
@@
 <contactref element="R18" pad="1"/>
 <contactref element="IC11" pad="1"/>
-<contactref element="C20" pad="1"/>
-<contactref element="R59" pad="2"/>
-<wire x1="-83.3525" y1="-222.7" x2="-379.5475" y2="-706.4" width="0" layer="19" extent="1-1"/>
+<contactref element="JP1" pad="3"/>
+<contactref element="JP2" pad="1"/>
+<wire x1="-375.62" y1="-725.2" x2="-380.7" y2="-730.1" width="0" layer="19" extent="1-1"/>
+<wire x1="-83.3525" y1="-222.7" x2="-375.62" y2="-725.2" width="0" layer="19" extent="1-1"/>
 <wire x1="-72.61" y1="-224.41" x2="-83.3525" y2="-222.7" width="0" layer="19" extent="1-1"/>
-<wire x1="-67.25" y1="-206.2" x2="-72.61" y2="-224.41" width="0" layer="19" extent="1-1"/>
 </signal>
 <signal name="V_FRONT_L">
@@
 <contactref element="IC11" pad="7"/>
 <contactref element="R28" pad="1"/>
-<contactref element="C19" pad="1"/>
-<contactref element="R58" pad="2"/>
+<contactref element="JP1" pad="1"/>
+<contactref element="JP2" pad="3"/>
 <wire x1="-70.07" y1="-216.79" x2="-119.3525" y2="-241" width="0" layer="19" extent="1-1"/>
-<wire x1="-71.25" y1="-206.2" x2="-70.07" y2="-216.79" width="0" layer="19" extent="1-1"/>
-<wire x1="-379.5475" y1="-700.3" x2="-119.3525" y2="-241" width="0" layer="19" extent="1-1"/>
+<wire x1="-380.7" y1="-725.2" x2="-119.3525" y2="-241" width="0" layer="19" extent="1-1"/>
+<wire x1="-375.62" y1="-730.1" x2="-380.7" y2="-725.2" width="0" layer="19" extent="1-1"/>
 </signal>
 <signal name="N$58">
@@
 <wire x1="8.175" y1="-57" x2="-247.3525" y2="-657.6" width="0" layer="19" extent="1-1"/>
 </signal>
+<signal name="N$42">
+<contactref element="IC5" pad="9"/>
+<contactref element="JP2" pad="2"/>
+<wire x1="9.445" y1="-47.8" x2="-378.16" y2="-730.1" width="0" layer="19" extent="1-1"/>
+</signal>
 </signals>

Commit message: change input filters - agin
Parts:
- added R13, R14: 100K, rcl:R0805W
- added R15, R16, R58, R59, R62, R63: DNP, rcl:R0805W
- C1, C10, C13, C14, C2, C5, C6, C9: value 10u -> 1u
- R41, R43, R52, R53, R54, R55, R56, R57, R60, R61: value 100K -> DNP
- moved R41 746.6 mm to (-392.7, -777.2)
- moved R43 741.1 mm to (-396.7, -777.2)
- moved R1 675.8 mm to (-380.6, -734.5)
- moved R3 672.0 mm to (-380.6, -740.6)
- moved R5 666.6 mm to (-380.6, -746.7)
- moved R7 662.8 mm to (-380.6, -752.8)
- moved R9 657.5 mm to (-380.6, -758.9)
- moved R11 653.6 mm to (-380.6, -765.0)
Connections:
- net AGND: now also R13.1, R14.1, R15.1, R16.1, R58.1, R59.1, R62.1, R63.1
- net N$1: now also R1.2
- net N$11: now also R5.2
- net N$12: now also R7.2
- net N$18: now also R59.2; no longer R7.2
- net N$2: now also R3.2
- net N$20: now also R58.2; no longer R5.2
- net N$22: now also R9.2
- net N$23: now also R11.2
- net N$27: now also R63.2; no longer R11.2
- net N$28: now also R62.2; no longer R9.2
- net N$29: now also R16.2; no longer R43.2
- net N$31: now also R13.2
- net N$32: now also R14.2
- net N$33: now also R15.2; no longer R41.2
- net N$8: now also R43.2; no longer R3.2
- net N$9: now also R41.2; no longer R1.2

Commit message: started routing
Parts:
- removed U$1, U$2, U$6, U$9: bead, Simplex-rlc:L0805W
- added IC10, IC13: OPA2134P, burr-brown:DIL08
- added R64, R65, R78, R80, R81, R82, R83, R84, R88, R91, R92, R93, R94, R95: 0R_0805, Simplex-Jumpers:R0805W
- added R66, R79: 0R, rcl:R0805W
- added R67, R70, R73, R76: 4K7, rcl:R0805W
- added R68, R69, R71, R72, R74, R77, R86, R89: 10K, rcl:R0805W
- added R75, R85, R87, R90: DNP, rcl:R0805W
- JP1: value (none) -> J1
- JP2: value (none) -> J2
- X2: value MOLEX_6VERTICAL -> MOLEX_6HORIZONTAL; device Simplex-Connectors:0530470610 -> Simplex-Connectors:0530480610
- X3: value MOLEX_4VERTICAL -> MOLEX_4HORIZONTAL; device Simplex-Connectors:0530470410 -> Simplex-Connectors:0530480401
- moved R16 978.1 mm to (61.9, 90.9), turned to 180 degrees
- moved R59 967.3 mm to (63.7, 69.2), turned to 180 degrees
- moved R15 966.2 mm to (43.8, 88.8)
- moved R58 956.0 mm to (43.8, 69.2)
- moved R63 955.2 mm to (63.7, 50.7), turned to 180 degrees
- moved R11 950.5 mm to (63.7, 75.3)
- moved R3 945.5 mm to (61.9, 95.0)
- moved R14 945.0 mm to (63.7, 56.9)
- moved R62 943.5 mm to (43.8, 50.7)
- moved R9 936.0 mm to (43.8, 75.3), turned to 180 degrees
- moved R1 931.7 mm to (43.8, 94.9), turned to 180 degrees
- moved R43 931.2 mm to (63.7, 32.2), turned to 180 degrees
- moved R13 930.4 mm to (43.8, 56.9), turned to 180 degrees
- moved R61 926.0 mm to (57.9, 97.0)
- moved R41 919.6 mm to (43.8, 32.2)
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Connections:
- removed net 41: U$11.41
- new net N$37: IC6.2, R64.2
- new net N$43: IC6.6, R65.2
- new net N$48: IC7.2, R66.1
- new net N$49: IC10.1, R18.1, R84.2
- new net N$50: IC7.6, R79.1
- new net N$54: IC10.5, R67.2
- new net N$55: IC10.6, R68.2, R69.1
- new net N$56: IC8.2, R80.2
- new net N$61: IC11.5, R70.2
- new net N$66: IC11.6, R71.2, R72.1
- new net N$67: IC8.6, R81.2
- new net N$68: IC12.5, R73.2
- new net N$69: IC12.6, R74.2, R86.1
- new net N$70: IC9.2, R82.2
- new net N$71: IC13.5, R76.2
- new net N$72: IC13.6, R77.2, R89.1
- new net N$73: IC9.6, R83.2
- new net N$75: IC11.1, R28.1, R78.2
- new net N$76: IC12.1, R30.1, R88.2
- new net N$77: R69.2, R84.1, R85.1
- new net N$78: IC13.1, R40.1, R91.2
- new net N$81: R72.2, R75.1, R78.1
- new net N$84: R86.2, R87.1, R88.1
- new net N$87: R89.2, R90.1, R91.1
- net +3V: now also R95.2; no longer U$9.2
- net +5V_DIG: now also R92.1; no longer U$6.2
- net A+5V: now also IC10.8, IC13.8, R94.1; no longer U$1.2
- net A-5V: now also IC10.4, IC13.4, R93.1; no longer U$2.2
- net AGND: now also R67.1, R70.1, R73.1, R75.2, R76.1, R85.2, R87.2, R90.2, X2.6; no longer X2.1
- net DGND: now also U$11.39, U$11.41, X2.1; no longer X2.6
- net M_FRONT_L: now also IC10.7, R68.1; no longer IC11.1, R18.1
- net M_FRONT_R: now also R71.1; no longer R28.1
- net M_REAR_L: now also IC12.7, R74.1; no longer IC12.1, R30.1
- net M_REAR_R: now also IC13.7, R77.1; no longer IC12.7, R40.1
- net N$15: now also R80.1; no longer IC8.2
- net N$16: now also R81.1; no longer IC8.6
- net N$17: now also IC6.7, R65.1; no longer IC7.6, IC7.7
- net N$19: now also R82.1; no longer IC9.2
- net N$24: now also X2.4; no longer X2.3
- net N$25: now also X2.3; no longer X2.4
- net N$26: now also R83.1; no longer IC9.6
- net N$29: now also IC6.5; no longer IC7.5
- net N$3: now also R92.2; no longer U$6.1
- net N$33: now also IC6.3; no longer IC7.3
- net N$34: now also X2.2; no longer X2.5
- net N$4: now also IC7.1, R66.2; no longer IC6.1, IC6.2
- net N$46: now also IC10.3; no longer IC11.3
- net N$47: now also IC10.2; no longer IC11.2
- net N$5: now also IC6.1, R64.1; no longer IC7.1, IC7.2
- net N$51: now also IC13.2; no longer IC12.6
- net N$52: now also IC11.3; no longer IC11.5
- net N$53: now also IC11.2; no longer IC11.6
- net N$6: now also R95.1; no longer U$9.1
- net N$60: now also R94.2; no longer U$1.1
- net N$62: now also R93.2; no longer U$2.1
- net N$63: now also X2.5; no longer X2.2
- net N$64: now also IC13.3; no longer IC12.5
- net N$7: now also IC7.7, R79.2; no longer IC6.6, IC6.7
- net N$8: now also IC7.5; no longer IC6.5
- net N$9: now also IC7.3; no longer IC6.3
- net V_FRONT_L: now also R19.2; no longer R20.2
- net V_FRONT_R: now also R24.2; no longer R25.2
- net V_LINE_L: now also R20.2; no longer R21.2
- net V_LINE_R: now also R25.2; no longer R26.2
- net V_REAR_L: now also R39.2; no longer R32.2
- net V_REAR_PAN_L: now also R32.2; no longer R39.2
- net V_REAR_PAN_R: now also R36.2; no longer R45.2
- net V_REAR_R: now also R45.2; no longer R36.2
- net V_SPDIF_L: now also R21.2; no longer R19.2
- net V_SPDIF_R: now also R26.2; no longer R24.2
Routing:
- net AGND: track 0.00 -> 26.3 mm, vias 0 -> 13
- net N$72: track 0.00 -> 11.6 mm
- net N$66: track 0.00 -> 11.5 mm
- net N$55: track 0.00 -> 11.5 mm
- net N$69: track 0.00 -> 11.5 mm
- net N$47: track 0.00 -> 10.6 mm
- net N$53: track 0.00 -> 10.4 mm
- net N$74: track 0.00 -> 8.25 mm
- net N$51: track 0.00 -> 8.24 mm
- net N$78: track 0.00 -> 5.71 mm
- net N$76: track 0.00 -> 5.66 mm
- net N$75: track 0.00 -> 5.64 mm
- net N$49: track 0.00 -> 5.64 mm
- net N$34: track 0.00 -> 5.36 mm
- net N$63: track 0.00 -> 5.18 mm
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- added copper zone on layer 15, net AGND
- added copper zone on layer 15, net DGND
Other:
- board size 92 x 56 mm -> 113.2 x 100 mm
