File: hardware/mixer.brd (EAGLE design)
At the start: 100 x 100 mm, 262 parts, among them IC1 PGA2311, IC10 OPA2134P, IC11 OPA2134P, IC12 OPA2134P, IC13 OPA2134P, IC14 PGA2311, IC2 PGA2311, IC3 PGA2311, IC4 PGA2311, IC5 PGA2311, IC6 OPA2134P, IC7 OPA2134P, IC8 OPA2134P, IC9 OPA2134P, Q1 SI2305, Q2 MOSFET-NCHANNEL_SOT23-3, U1 V_REG_LDOSMD, X1 MOLEX_6HORIZONTAL, X3 display, X4 input, X5 2512-5, X6 2512-5, Y1 32768Hz CFPX-217 12.5pF

Commit message: mosfets purchased
Parts:
- removed C27: 220nF, rcl:C0805
Connections:
- removed net N$13: C27.1, U$11.43
- new net 43: U$11.43
- net DGND: no longer C27.2
Routing:
- net N$13: track 4.55 -> 0.00 mm
- net DGND: track 95.9 -> 94.5 mm, vias 55 -> 54
Changed lines of the file:
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@@
 <element name="U$11" library="TI_MSP430_v16" package="PT48" value="F55[0/1]X---PT48" x="14.25" y="67.25"/>
 <element name="C23" library="rcl" package="C0805" value="470nF" x="9.2" y="61.55" rot="R180"/>
-<element name="C27" library="rcl" package="C0805" value="220nF" x="11.05" y="74.45" rot="R180"/>
 <element name="R22" library="rcl" package="R0805W" value="2.2K" x="11.05" y="76.5"/>
 <element name="R27" library="rcl" package="R0805W" value="2.2K" x="11.05" y="78.55"/>
@@
 <contactref element="R33" pad="1"/>
 <contactref element="U$11" pad="27"/>
-<contactref element="C27" pad="2"/>
 <contactref element="U$11" pad="44"/>
 <contactref element="U$11" pad="37"/>
@@
 <wire x1="9.95" y1="64.5" x2="9.95" y2="64" width="0.3048" layer="1"/>
 <wire x1="9.95" y1="64" x2="9.75" y2="63.8" width="0.3048" layer="1"/>
-<via x="9.4" y="73.3" extent="1-16" drill="0.4"/>
-<wire x1="10.1" y1="74.45" x2="9.4" y2="73.3" width="0.3048" layer="1"/>
 <wire x1="26.15" y1="32.8525" x2="26.1975" y2="33.05" width="0.4064" layer="1"/>
 <wire x1="26.1975" y1="33.05" x2="27.45" y2="33.05" width="0.4064" layer="1"/>
@@
 <contactref element="X5" pad="10"/>
 <contactref element="X5" pad="12"/>
+<wire x1="29.05" y1="88.915" x2="30.05" y2="85.6" width="0" layer="19" extent="1-16"/>
+<wire x1="28.75" y1="78.15" x2="30.8" y2="84" width="0" layer="19" extent="1-1"/>
+<wire x1="29.05" y1="69.815" x2="28.75" y2="78.15" width="0" layer="19" extent="1-1"/>
+<wire x1="30.1" y1="66.55" x2="29.05" y2="69.815" width="0" layer="19" extent="1-16"/>
+<wire x1="24.3975" y1="67.25" x2="27.4" y2="69.8" width="0" layer="19" extent="1-1"/>
+<wire x1="18.55" y1="65.5" x2="23.8" y2="65.45" width="0" layer="19" extent="1-16"/>
+<wire x1="17" y1="70.05" x2="17.2" y2="65.5" width="0" layer="19" extent="1-1"/>
+<wire x1="16.05" y1="70.05" x2="17" y2="70.05" width="0" layer="19" extent="1-1"/>
+<wire x1="15.05" y1="70.05" x2="16" y2="70.05" width="0" layer="19" extent="1-1"/>
+<wire x1="13.5" y1="71.55" x2="15" y2="71.55" width="0" layer="19" extent="1-1"/>
+<wire x1="16.85" y1="74.85" x2="17" y2="71.55" width="0" layer="19" extent="1-1"/>
+<wire x1="8.8" y1="68.1" x2="13.5" y2="70.05" width="0" layer="19" extent="1-1"/>
+<wire x1="8.6" y1="68.6" x2="8.8" y2="68.1" width="0" layer="19" extent="1-1"/>
+<wire x1="8.6" y1="63.8" x2="8.8" y2="64.3" width="0" layer="19" extent="1-1"/>
+<wire x1="2.35" y1="68.65" x2="2.85" y2="68.85" width="0" layer="19" extent="1-1"/>
+<wire x1="2.35" y1="63.75" x2="2.9" y2="63.55" width="0" layer="19" extent="1-1"/>
+<wire x1="9.95" y1="64.5" x2="9.95" y2="65.5" width="0" layer="19" extent="1-1"/>
+<wire x1="4.75" y1="65.15" x2="3.15" y2="65" width="0" layer="19" extent="1-16"/>
+<wire x1="4.75" y1="69.1" x2="2.85" y2="68.85" width="0" layer="19" extent="1-1"/>
+<wire x1="8.25" y1="61.55" x2="8.05" y2="63.55" width="0" layer="19" extent="1-1"/>
+<wire x1="5" y1="58.75" x2="7.05" y2="61.55" width="0" layer="19" extent="1-1"/>
+<wire x1="6.0025" y1="72.95" x2="4.75" y2="69.1" width="0" layer="19" extent="1-1"/>
+<wire x1="28.55" y1="59.55" x2="30.7" y2="64.75" width="0" layer="19" extent="1-1"/>
+<wire x1="3.2" y1="51.8" x2="4.95" y2="57.5525" width="0" layer="19" extent="1-1"/>
+<wire x1="4.2" y1="48.55" x2="3.2" y2="51.8" width="0" layer="19" extent="1-1"/>
+<wire x1="3.85" y1="45.2" x2="3.45" y2="47.25" width="0" layer="19" extent="1-1"/>
+<wire x1="3.6" y1="42.4" x2="3.85" y2="45.2" width="0" layer="19" extent="1-1"/>
+<wire x1="5.05" y1="39.8" x2="4.6999" y2="42.4" width="0" layer="19" extent="1-1"/>
+<wire x1="3.5" y1="37.8" x2="3.75" y2="39.75" width="0" layer="19" extent="1-1"/>
+<wire x1="11.05" y1="39.8" x2="5.05" y2="39.8" width="0" layer="19" extent="1-1"/>
+<wire x1="6.2" y1="79.55" x2="6.0025" y2="72.95" width="0" layer="19" extent="1-1"/>
+<wire x1="6.2" y1="82.7" x2="6.2" y2="79.55" width="0" layer="19" extent="1-1"/>
+<wire x1="12.1025" y1="86" x2="6.2" y2="82.7" width="0" layer="19" extent="1-1"/>
+<wire x1="4.58" y1="29.05" x2="4.2" y2="36.45" width="0" layer="19" extent="1-1"/>
+<wire x1="4.58" y1="26.51" x2="4.58" y2="29.05" width="0" layer="19" extent="1-1"/>
+<wire x1="29.05" y1="51.615" x2="28.75" y2="59.35" width="0" layer="19" extent="1-1"/>
+<wire x1="30.05" y1="48.35" x2="29.05" y2="51.615" width="0" layer="19" extent="1-16"/>
+<wire x1="25.2" y1="42.3" x2="30.05" y2="47.3" width="0" layer="19" extent="16-16"/>
+<wire x1="19.35" y1="46.35" x2="25.2" y2="42.3" width="0" layer="19" extent="1-1"/>
+<wire x1="17.55" y1="51.6" x2="19.35" y2="46.35" width="0" layer="19" extent="1-1"/>
+<wire x1="19.45" y1="35.2" x2="12.2" y2="39.2" width="0" layer="19" extent="1-1"/>
+<wire x1="18.95" y1="30.2" x2="18.55" y2="33.8" width="0" layer="19" extent="1-1"/>
+<wire x1="21.8" y1="24.85" x2="18.55" y2="28.9" width="0" layer="19" extent="1-1"/>
+<wire x1="26.15" y1="32.8525" x2="19.45" y2="33.8" width="0" layer="19" extent="1-1"/>
+<wire x1="30.05" y1="29.75" x2="29.05" y2="33.065" width="0" layer="19" extent="1-16"/>
+<wire x1="30" y1="22.2" x2="30.55" y2="28.2" width="0" layer="19" extent="1-1"/>
+<wire x1="29.05" y1="13.515" x2="28.75" y2="22.1" width="0" layer="19" extent="1-1"/>
+<wire x1="30.05" y1="10.2" x2="29.05" y2="13.515" width="0" layer="19" extent="1-16"/>
+<wire x1="21.75" y1="13.1" x2="26.15" y2="13.2525" width="0" layer="19" extent="1-1"/>
+<wire x1="21.75" y1="6.95" x2="21.75" y2="13.1" width="0" layer="19" extent="1-1"/>
+<wire x1="13.8" y1="3.8" x2="21.75" y2="6.95" width="0" layer="19" extent="1-1"/>
+<wire x1="13.75" y1="3.85" x2="13.8" y2="3.8" width="0" layer="19" extent="1-1"/>
+<wire x1="12.25" y1="3.86" x2="13.75" y2="3.85" width="0" layer="19" extent="1-1"/>
+<wire x1="12.25" y1="2.05" x2="12.25" y2="3.86" width="0" layer="19" extent="1-1"/>
+<wire x1="66.25" y1="8.3975" x2="31.55" y2="10.15" width="0" layer="19" extent="1-1"/>
+<wire x1="70.9" y1="5.05" x2="66.25" y2="6.9" width="0" layer="19" extent="1-1"/>
+<wire x1="67.05" y1="13.5" x2="66.25" y2="8.3975" width="0" layer="19" extent="1-1"/>
+<wire x1="71.25" y1="13.2" x2="68.65" y2="13.515" width="0" layer="19" extent="1-16"/>
 </signal>
 <signal name="N$5">
@@
 <wire x1="11.15" y1="61.55" x2="10.15" y2="61.55" width="0.3048" layer="1"/>
 </signal>
-<signal name="N$13">
-<contactref element="U$11" pad="43"/>
-<contactref element="C27" pad="1"/>
-<wire x1="14" y1="71.55" x2="14" y2="73.85" width="0.3048" layer="1"/>
-<wire x1="14" y1="73.85" x2="13.4" y2="74.45" width="0.3048" layer="1"/>
-<wire x1="13.4" y1="74.45" x2="12" y2="74.45" width="0.3048" layer="1"/>
-</signal>
 <signal name="N$14">
 <contactref element="U$11" pad="34"/>
@@
 <wire x1="9.15" y1="41" x2="9.15" y2="39.8" width="0.4064" layer="1"/>
 </signal>
+<signal name="43">
+<contactref element="U$11" pad="43"/>
+</signal>
 </signals>

Commit message: tweak filters
Parts:
- R1, R105, R106, R11, R13, R14, R3, R5, R7, R9: value 100K -> DNP
- R103, R104, R107, R108, R15, R16, R41, R43, R52, R53, R54, R55, R56, R57, R58, R59, R60, R61, R62, R63: value DNP -> 100K
- R33: value 100k -> 47k
Changed lines of the file:
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@@
 <grid distance="0.05" unitdist="mm" unit="mm" style="dots" multiple="1" display="yes" altdistance="0.127" altunitdist="mm" altunit="mm"/>
 <layers>
-<layer number="1" name="Top" color="4" fill="1" visible="yes" active="yes"/>
-<layer number="2" name="Route2" color="5" fill="1" visible="yes" active="yes"/>
+<layer number="1" name="Top" color="4" fill="1" visible="no" active="yes"/>
+<layer number="2" name="Route2" color="5" fill="1" visible="no" active="yes"/>
 <layer number="3" name="Route3" color="4" fill="3" visible="no" active="no"/>
 <layer number="14" name="Route14" color="1" fill="6" visible="no" active="no"/>
-<layer number="15" name="Route15" color="3" fill="1" visible="yes" active="yes"/>
+<layer number="15" name="Route15" color="3" fill="1" visible="no" active="yes"/>
 <layer number="16" name="Bottom" color="1" fill="1" visible="yes" active="yes"/>
 <layer number="17" name="Pads" color="2" fill="1" visible="yes" active="yes"/>
@@
 <layer number="25" name="tNames" color="7" fill="1" visible="no" active="yes"/>
 <layer number="26" name="bNames" color="7" fill="1" visible="no" active="yes"/>
-<layer number="27" name="tValues" color="7" fill="1" visible="no" active="yes"/>
-<layer number="28" name="bValues" color="7" fill="1" visible="no" active="yes"/>
+<layer number="27" name="tValues" color="7" fill="1" visible="yes" active="yes"/>
+<layer number="28" name="bValues" color="7" fill="1" visible="yes" active="yes"/>
 <layer number="29" name="tStop" color="7" fill="3" visible="no" active="yes"/>
 <layer number="30" name="bStop" color="7" fill="6" visible="no" active="yes"/>
@@
 <element name="R31" library="rcl" package="R0805W" value="47k" x="11.05" y="86"/>
 <element name="LED2" library="led" package="CHIPLED_0805" value="green" x="4.95" y="71.25" rot="R90"/>
-<element name="R33" library="rcl" package="R0805W" value="100k" x="4.95" y="72.95" rot="R180"/>
+<element name="R33" library="rcl" package="R0805W" value="47k" x="4.95" y="72.95" rot="R180"/>
 <element name="C57" library="rcl" package="C0805" value="100nF" x="7" y="56.5" rot="R90"/>
 <element name="R37" library="rcl" package="R0805W" value="10K" x="9.8" y="53.15"/>
@@
 <element name="C91" library="rcl" package="153CLV-0405" value="10u" x="28.75" y="61.15" rot="R90"/>
 <element name="C87" library="rcl" package="153CLV-0405" value="10u" x="16.75" y="33.8" rot="R180"/>
-<element name="R52" library="rcl" package="R0805W" value="DNP" x="65.2" y="39.85"/>
-<element name="R53" library="rcl" package="R0805W" value="DNP" x="81.2" y="39.85" rot="R180"/>
-<element name="R54" library="rcl" package="R0805W" value="DNP" x="65.25" y="76.6"/>
-<element name="R55" library="rcl" package="R0805W" value="DNP" x="81.2" y="76.6" rot="R180"/>
-<element name="R56" library="rcl" package="R0805W" value="DNP" x="65.2" y="58.3"/>
-<element name="R57" library="rcl" package="R0805W" value="DNP" x="81.2" y="58.35" rot="R180"/>
-<element name="R60" library="rcl" package="R0805W" value="DNP" x="65.25" y="95.7"/>
-<element name="R61" library="rcl" package="R0805W" value="DNP" x="81.2" y="95.7" rot="R180"/>
+<element name="R52" library="rcl" package="R0805W" value="100K" x="65.2" y="39.85"/>
+<element name="R53" library="rcl" package="R0805W" value="100K" x="81.2" y="39.85" rot="R180"/>
+<element name="R54" library="rcl" package="R0805W" value="100K" x="65.25" y="76.6"/>
+<element name="R55" library="rcl" package="R0805W" value="100K" x="81.2" y="76.6" rot="R180"/>
+<element name="R56" library="rcl" package="R0805W" value="100K" x="65.2" y="58.3"/>
+<element name="R57" library="rcl" package="R0805W" value="100K" x="81.2" y="58.35" rot="R180"/>
+<element name="R60" library="rcl" package="R0805W" value="100K" x="65.25" y="95.7"/>
+<element name="R61" library="rcl" package="R0805W" value="100K" x="81.2" y="95.7" rot="R180"/>
 <element name="JP1" library="SparkFun-Connectors" package="1X03" value="J1" x="56.45" y="11.6" rot="R90"/>
 <element name="JP2" library="SparkFun-Connectors" package="1X03" value="J2" x="53.85" y="11.6" rot="R90"/>
-<element name="R1" library="rcl" package="R0805W" value="100K" x="65.25" y="91.6" rot="R180"/>
-<element name="R3" library="rcl" package="R0805W" value="100K" x="81.2" y="91.6"/>
-<element name="R5" library="rcl" package="R0805W" value="100K" x="65.2" y="35.75" rot="R180"/>
-<element name="R7" library="rcl" package="R0805W" value="100K" x="81.2" y="35.75"/>
-<element name="R9" library="rcl" package="R0805W" value="100K" x="65.25" y="72.5" rot="R180"/>
-<element name="R11" library="rcl" package="R0805W" value="100K" x="81.2" y="72.5"/>
-<element name="R13" library="rcl" package="R0805W" value="100K" x="65.2" y="54.2" rot="R180"/>
-<element name="R14" library="rcl" package="R0805W" value="100K" x="81.2" y="54.25"/>
-<element name="R15" library="rcl" package="R0805W" value="DNP" x="65.25" y="85.45"/>
-<element name="R16" library="rcl" package="R0805W" value="DNP" x="81.2" y="87.5" rot="R180"/>
-<element name="R41" library="rcl" package="R0805W" value="DNP" x="65.2" y="29.6"/>
-<element name="R43" library="rcl" package="R0805W" value="DNP" x="81.2" y="29.6" rot="R180"/>
-<element name="R58" library="rcl" package="R0805W" value="DNP" x="65.25" y="66.35"/>
-<element name="R59" library="rcl" package="R0805W" value="DNP" x="81.2" y="66.35" rot="R180"/>
-<element name="R62" library="rcl" package="R0805W" value="DNP" x="65.2" y="48.05"/>
-<element name="R63" library="rcl" package="R0805W" value="DNP" x="81.2" y="48.1" rot="R180"/>
+<element name="R1" library="rcl" package="R0805W" value="DNP" x="65.25" y="91.6" rot="R180"/>
+<element name="R3" library="rcl" package="R0805W" value="DNP" x="81.2" y="91.6"/>
+<element name="R5" library="rcl" package="R0805W" value="DNP" x="65.2" y="35.75" rot="R180"/>
+<element name="R7" library="rcl" package="R0805W" value="DNP" x="81.2" y="35.75"/>
+<element name="R9" library="rcl" package="R0805W" value="DNP" x="65.25" y="72.5" rot="R180"/>
+<element name="R11" library="rcl" package="R0805W" value="DNP" x="81.2" y="72.5"/>
+<element name="R13" library="rcl" package="R0805W" value="DNP" x="65.2" y="54.2" rot="R180"/>
+<element name="R14" library="rcl" package="R0805W" value="DNP" x="81.2" y="54.25"/>
+<element name="R15" library="rcl" package="R0805W" value="100K" x="65.25" y="85.45"/>
+<element name="R16" library="rcl" package="R0805W" value="100K" x="81.2" y="87.5" rot="R180"/>
+<element name="R41" library="rcl" package="R0805W" value="100K" x="65.2" y="29.6"/>
+<element name="R43" library="rcl" package="R0805W" value="100K" x="81.2" y="29.6" rot="R180"/>
+<element name="R58" library="rcl" package="R0805W" value="100K" x="65.25" y="66.35"/>
+<element name="R59" library="rcl" package="R0805W" value="100K" x="81.2" y="66.35" rot="R180"/>
+<element name="R62" library="rcl" package="R0805W" value="100K" x="65.2" y="48.05"/>
+<element name="R63" library="rcl" package="R0805W" value="100K" x="81.2" y="48.1" rot="R180"/>
 <element name="R67" library="rcl" package="R0805W" value="4K7" x="61.4" y="85.5" rot="R90"/>
 <element name="R68" library="rcl" package="R0805W" value="10K" x="61.4" y="89.55" rot="R270"/>
@@
 <element name="C67" library="rcl" package="C0805" value="1u" x="92.65" y="17.5" rot="R270"/>
 <element name="C68" library="rcl" package="C0805" value="1u" x="92.65" y="12.1" rot="R270"/>
-<element name="R103" library="rcl" package="R0805W" value="DNP" x="94.7" y="17.5" rot="R90"/>
-<element name="R104" library="rcl" package="R0805W" value="DNP" x="94.7" y="12.1" rot="R90"/>
-<element name="R105" library="rcl" package="R0805W" value="100K" x="90.6" y="17.5" rot="R270"/>
-<element name="R106" library="rcl" package="R0805W" value="100K" x="90.6" y="12.1" rot="R270"/>
-<element name="R107" library="rcl" package="R0805W" value="DNP" x="84.45" y="17.5" rot="R90"/>
-<element name="R108" library="rcl" package="R0805W" value="DNP" x="84.45" y="12.1" rot="R90"/>
+<element name="R103" library="rcl" package="R0805W" value="100K" x="94.7" y="17.5" rot="R90"/>
+<element name="R104" library="rcl" package="R0805W" value="100K" x="94.7" y="12.1" rot="R90"/>
+<element name="R105" library="rcl" package="R0805W" value="DNP" x="90.6" y="17.5" rot="R270"/>
+<element name="R106" library="rcl" package="R0805W" value="DNP" x="90.6" y="12.1" rot="R270"/>
+<element name="R107" library="rcl" package="R0805W" value="100K" x="84.45" y="17.5" rot="R90"/>
+<element name="R108" library="rcl" package="R0805W" value="100K" x="84.45" y="12.1" rot="R90"/>
 <element name="U1" library="SparkFun-PowerIC" package="SOT23-5" value="V_REG_LDOSMD" x="6" y="42.4" rot="R270"/>
 <element name="C71" library="rcl" package="C0805" value="100nF" x="6" y="39.8"/>
