File: hardware/mixer.brd (EAGLE design)
At the start: 100 x 100 mm, 261 parts, among them IC1 PGA2311, IC10 OPA2134P, IC11 OPA2134P, IC12 OPA2134P, IC13 OPA2134P, IC14 PGA2311, IC2 PGA2311, IC3 PGA2311, IC4 PGA2311, IC5 PGA2311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

Commit message: small tweaks
Parts:
- removed Q2: MOSFET-NCHANNEL_SOT23-3, Simplex-DiscreteSemi:SOT23-3
- removed R79: 0R, rcl:R0805W
- added R114: 0R_0805, Simplex-Jumpers:R0805W
- added T1: BC846, transistor:SOT23
- R66: value 0R -> 0R_0805; device rcl:R0805W -> Simplex-Jumpers:R0805W
- moved R66 14.2 mm to (80.2, 33.7), turned to 270 degrees
Connections:
- net DGND: now also T1.2; no longer Q2.2
- net N$4: now also R114.1; no longer R66.2
- net N$40: now also T1.3; no longer Q2.3
- net N$41: now also T1.1; no longer Q2.1
- net N$48: now also R114.2; no longer R66.1
- net N$50: now also R66.2; no longer R79.1
- net N$7: now also R66.1; no longer R79.2
Routing:
- net N$4: track 36.9 -> 40.3 mm
- net N$48: track 3.52 -> 6.64 mm
- net N$7: track 63.5 -> 66.3 mm
- net N$50: track 3.19 -> 5.92 mm
- net DGND: track 94.5 -> 93.6 mm, vias 54 -> 53
Changed lines of the file:
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@@
 <layer number="19" name="Unrouted" color="6" fill="1" visible="yes" active="yes"/>
 <layer number="20" name="Dimension" color="15" fill="1" visible="yes" active="yes"/>
-<layer number="21" name="tPlace" color="7" fill="1" visible="yes" active="yes"/>
+<layer number="21" name="tPlace" color="7" fill="1" visible="no" active="yes"/>
 <layer number="22" name="bPlace" color="7" fill="1" visible="yes" active="yes"/>
 <layer number="23" name="tOrigins" color="15" fill="1" visible="yes" active="yes"/>
@@
 <wire x1="88.1" y1="58.55" x2="93.7" y2="58.55" width="0.1" layer="108"/>
 <wire x1="93.75" y1="56.05" x2="99.45" y2="56.05" width="0.1" layer="108"/>
-<text x="10.45" y="20.6" size="1.016" layer="108" font="vector" ratio="15" rot="R90">power</text>
+<text x="11.5" y="20.55" size="1.016" layer="108" font="vector" ratio="15" rot="R90">power</text>
 <text x="30.25" y="45.2" size="0.8128" layer="108" font="vector" ratio="15">-5V</text>
 <text x="30.25" y="43.4" size="0.8128" layer="108" font="vector" ratio="15">+5V</text>
@@
 <element name="Q1" library="Simplex-DiscreteSemi" package="SOT23-3_POWER" value="SI2305" x="9.8" y="56.5"/>
 <element name="X1" library="Simplex-Connectors" package="0530480610" value="MOLEX_6HORIZONTAL" x="6.2" y="82.7" rot="R90"/>
-<element name="Q2" library="Simplex-DiscreteSemi" package="SOT23-3" value="MOSFET-NCHANNEL_SOT23-3" x="4.2" y="52.75" rot="R270"/>
 <element name="R38" library="rcl" package="R0805W" value="10K" x="4.95" y="56.5" rot="R270"/>
 <element name="R46" library="rcl" package="R0805W" value="10K" x="2.85" y="56.5" rot="R90"/>
@@
 <attribute name="OC_FARNELL" value="1097574" x="73.25" y="33.7" size="1.778" layer="27" rot="R270" display="off"/>
 </element>
-<element name="R66" library="rcl" package="R0805W" value="0R" x="66.2" y="36.3" rot="MR90"/>
-<element name="R79" library="rcl" package="R0805W" value="0R" x="80.2" y="33.7" rot="MR90"/>
 <element name="R85" library="rcl" package="R0805W" value="DNP" x="51.3" y="98" rot="R180"/>
 <element name="R84" library="Simplex-Jumpers" package="R0805W" value="0R_0805" x="51.3" y="95.95" rot="R180"/>
@@
 <attribute name="OC_FARNELL" value="1788673" x="5.85" y="22.7" size="1.778" layer="27" rot="R90" display="off"/>
 </element>
+<element name="T1" library="transistor" package="SOT23" value="BC846" x="4.25" y="52.85" rot="R270"/>
+<element name="R114" library="Simplex-Jumpers" package="R0805W" value="0R_0805" x="66.2" y="36.3" rot="MR270"/>
+<element name="R66" library="Simplex-Jumpers" package="R0805W" value="0R_0805" x="80.15" y="33.7" rot="MR270"/>
 </elements>
 <signals>
@@
 <contactref element="U$11" pad="44"/>
 <contactref element="U$11" pad="37"/>
-<contactref element="Q2" pad="2"/>
 <contactref element="R38" pad="1"/>
 <contactref element="R31" pad="2"/>
@@
 <wire x1="8.25" y1="61.55" x2="7.05" y2="61.55" width="0.3048" layer="1"/>
 <via x="5" y="58.75" extent="1-16" drill="0.4"/>
-<via x="2.25" y="51.8" extent="1-16" drill="0.4"/>
-<wire x1="3.2" y1="51.8" x2="2.25" y2="51.8" width="0.4064" layer="1"/>
 <via x="7.2" y="72.9" extent="1-16" drill="0.4"/>
 <wire x1="6.0025" y1="72.95" x2="7.15" y2="72.95" width="0.3048" layer="1"/>
@@
 <contactref element="X5" pad="10"/>
 <contactref element="X5" pad="12"/>
+<contactref element="T1" pad="2"/>
 </signal>
 <signal name="N$5">
@@
 <contactref element="IC2" pad="16"/>
 <contactref element="IC7" pad="1"/>
-<contactref element="R66" pad="2"/>
 <via x="39.8" y="38.15" extent="1-16" drill="0.4"/>
 <wire x1="38.25" y1="38.145" x2="38.25" y2="38.15" width="0.4064" layer="1"/>
 <wire x1="38.25" y1="38.15" x2="39.8" y2="38.15" width="0.4064" layer="1"/>
 <wire x1="69.44" y1="37.51" x2="66.2" y2="37.51" width="0.4064" layer="16"/>
-<wire x1="66.2" y1="37.51" x2="66.2" y2="37.3525" width="0.4064" layer="16"/>
 <wire x1="39.8" y1="38.15" x2="42.2" y2="38.15" width="0.4064" layer="16"/>
 <wire x1="42.2" y1="38.15" x2="42.85" y2="38.8" width="0.4064" layer="16" curve="90"/>
@@
 <wire x1="60.85" y1="38.25" x2="61.75" y2="37.35" width="0.4064" layer="16" curve="90"/>
 <wire x1="61.75" y1="37.35" x2="66.1975" y2="37.35" width="0.4064" layer="16"/>
-<wire x1="66.1975" y1="37.35" x2="66.2" y2="37.3525" width="0.4064" layer="16" curve="90"/>
 <contactref element="R112" pad="2"/>
-<wire x1="64.15" y1="37.3525" x2="66.2" y2="37.3525" width="0.6096" layer="16"/>
+<contactref element="R114" pad="1"/>
+<wire x1="64.15" y1="37.3525" x2="66.0875" y2="37.3525" width="0.4064" layer="16"/>
+<wire x1="66.0875" y1="37.3525" x2="66.2" y2="37.24" width="0.4064" layer="16"/>
+<wire x1="66.2" y1="37.24" x2="66.47" y2="37.51" width="0.4064" layer="16"/>
+<wire x1="66.47" y1="37.51" x2="69.44" y2="37.51" width="0.4064" layer="16"/>
+<wire x1="66.1975" y1="37.35" x2="66.2" y2="37.3475" width="0.4064" layer="16"/>
+<wire x1="66.2" y1="37.3475" x2="66.2" y2="37.24" width="0.4064" layer="16"/>
 </signal>
 <signal name="N$7">
 <contactref element="IC2" pad="9"/>
 <contactref element="IC7" pad="7"/>
-<contactref element="R79" pad="2"/>
 <via x="39.8" y="29.25" extent="1-16" drill="0.4"/>
 <wire x1="38.25" y1="29.255" x2="38.25" y2="29.25" width="0.4064" layer="1"/>
 <wire x1="38.25" y1="29.25" x2="39.8" y2="29.25" width="0.4064" layer="1"/>
 <wire x1="77.06" y1="34.97" x2="79.75" y2="34.97" width="0.4064" layer="16"/>
-<wire x1="79.75" y1="34.97" x2="80.2" y2="34.7525" width="0.4064" layer="16"/>
 <wire x1="39.8" y1="29.25" x2="43.05" y2="29.25" width="0.4064" layer="16"/>
 <wire x1="43.05" y1="29.25" x2="43.85" y2="30.05" width="0.4064" layer="16" curve="90"/>
@@
 <wire x1="61.25" y1="41.45" x2="79.2" y2="41.45" width="0.4064" layer="16"/>
 <wire x1="79.2" y1="41.45" x2="80.2" y2="40.45" width="0.4064" layer="16" curve="-90"/>
-<wire x1="80.2" y1="40.45" x2="80.2" y2="34.7525" width="0.4064" layer="16"/>
 <contactref element="R100" pad="2"/>
-<wire x1="80.2" y1="34.7525" x2="82.25" y2="34.7525" width="0.6096" layer="16"/>
+<contactref element="R66" pad="1"/>
+<wire x1="80.15" y1="34.64" x2="79.82" y2="34.97" width="0.4064" layer="16"/>
+<wire x1="79.82" y1="34.97" x2="77.06" y2="34.97" width="0.4064" layer="16"/>
+<wire x1="82.25" y1="34.7525" x2="82.1375" y2="34.64" width="0.4064" layer="16"/>
+<wire x1="82.1375" y1="34.64" x2="80.15" y2="34.64" width="0.4064" layer="16"/>
+<wire x1="79.82" y1="34.97" x2="80.2" y2="35.35" width="0.4064" layer="16"/>
+<wire x1="80.2" y1="35.35" x2="80.2" y2="40.45" width="0.4064" layer="16"/>
 </signal>
 <signal name="N$8">
@@
 <contactref element="R37" pad="1"/>
 <contactref element="Q1" pad="1"/>
-<contactref element="Q2" pad="3"/>
-<wire x1="5.3" y1="52.75" x2="8.3475" y2="52.75" width="0.4064" layer="1"/>
-<wire x1="8.3475" y1="52.75" x2="8.7475" y2="53.15" width="0.4064" layer="1"/>
 <wire x1="8.8612" y1="55.11586875" x2="8.8612" y2="53.2637" width="0.4064" layer="1"/>
 <wire x1="8.8612" y1="53.2637" x2="8.7475" y2="53.15" width="0.3048" layer="1"/>
 <wire x1="7" y1="55.55" x2="7.43413125" y2="55.11586875" width="0.4064" layer="1"/>
 <wire x1="7.43413125" y1="55.11586875" x2="8.8612" y2="55.11586875" width="0.4064" layer="1"/>
+<contactref element="T1" pad="3"/>
+<wire x1="5.35" y1="52.85" x2="8.4475" y2="52.85" width="0.4064" layer="1"/>
+<wire x1="8.4475" y1="52.85" x2="8.7475" y2="53.15" width="0.4064" layer="1"/>
 </signal>
 <signal name="N$41">
 <contactref element="R46" pad="1"/>
-<contactref element="Q2" pad="1"/>
 <contactref element="R38" pad="2"/>
-<wire x1="2.85" y1="55.4475" x2="2.85" y2="54.05" width="0.4064" layer="1"/>
-<wire x1="2.85" y1="54.05" x2="3.2" y2="53.7" width="0.4064" layer="1"/>
 <wire x1="2.85" y1="55.4475" x2="4.95" y2="55.4475" width="0.4064" layer="1"/>
+<contactref element="T1" pad="1"/>
+<wire x1="2.85" y1="55.4475" x2="2.85" y2="54.1" width="0.4064" layer="1"/>
+<wire x1="2.85" y1="54.1" x2="3.15" y2="53.8" width="0.4064" layer="1"/>
 </signal>
 <signal name="PGA_EN">
@@
 <signal name="N$48">
 <contactref element="IC7" pad="2"/>
-<contactref element="R66" pad="1"/>
-<wire x1="66.2" y1="35.2475" x2="66.2" y2="34.97" width="0.4064" layer="16"/>
 <wire x1="66.2" y1="34.97" x2="69.44" y2="34.97" width="0.4064" layer="16"/>
+<contactref element="R114" pad="2"/>
+<wire x1="66.2" y1="35.36" x2="66.59" y2="34.97" width="0.4064" layer="16"/>
+<wire x1="66.59" y1="34.97" x2="69.44" y2="34.97" width="0.4064" layer="16"/>
 </signal>
 <signal name="N$50">
 <contactref element="IC7" pad="6"/>
-<contactref element="R79" pad="1"/>
 <wire x1="77.06" y1="32.43" x2="79.75" y2="32.43" width="0.4064" layer="16"/>
-<wire x1="79.75" y1="32.43" x2="80.2" y2="32.6475" width="0.4064" layer="16"/>
+<contactref element="R66" pad="2"/>
+<wire x1="80.15" y1="32.76" x2="79.82" y2="32.43" width="0.4064" layer="16"/>
+<wire x1="79.82" y1="32.43" x2="77.06" y2="32.43" width="0.4064" layer="16"/>
 </signal>
 <signal name="N$56">

Commit message: board rev 1.1
Parts:
- removed R97: 0R_0805, Simplex-Jumpers:R0805W
- added R79: 10K, rcl:R0805W
- R96: value 0R_0805 -> 10K; device Simplex-Jumpers:R0805W -> rcl:R0805W
- R98, R99: value DNP -> 4K7
- turned R96 to 180 degrees
Connections:
- net N$36: now also R96.1; no longer R96.2
- net N$42: now also R96.2; no longer R96.1
- net N$79: now also R79.2; no longer R97.1
- net N$80: now also R79.1; no longer R97.2
Changed lines of the file:
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@@
 <setting verticaltext="up"/>
 </settings>
-<grid distance="0.05" unitdist="mm" unit="mm" style="dots" multiple="1" display="yes" altdistance="0.127" altunitdist="mm" altunit="mm"/>
+<grid distance="0.05" unitdist="mm" unit="mm" style="dots" multiple="1" display="yes" altdistance="0.005" altunitdist="inch" altunit="inch"/>
 <layers>
-<layer number="1" name="Top" color="4" fill="1" visible="no" active="yes"/>
-<layer number="2" name="Route2" color="5" fill="1" visible="no" active="yes"/>
+<layer number="1" name="Top" color="4" fill="1" visible="yes" active="yes"/>
+<layer number="2" name="Route2" color="5" fill="1" visible="yes" active="yes"/>
 <layer number="3" name="Route3" color="4" fill="3" visible="no" active="no"/>
 <layer number="14" name="Route14" color="1" fill="6" visible="no" active="no"/>
-<layer number="15" name="Route15" color="3" fill="1" visible="no" active="yes"/>
+<layer number="15" name="Route15" color="3" fill="1" visible="yes" active="yes"/>
 <layer number="16" name="Bottom" color="1" fill="1" visible="yes" active="yes"/>
 <layer number="17" name="Pads" color="2" fill="1" visible="yes" active="yes"/>
@@
 <element name="R83" library="Simplex-Jumpers" package="R0805W" value="0R_0805" x="80.2" y="52.35" rot="MR270"/>
 <element name="X3" library="Simplex-Connectors" package="0530480401" value="display" x="6.2" y="75.8" rot="R90"/>
-<element name="R96" library="Simplex-Jumpers" package="R0805W" value="0R_0805" x="49.15" y="15.5"/>
-<element name="R97" library="Simplex-Jumpers" package="R0805W" value="0R_0805" x="49.15" y="13.4"/>
-<element name="R98" library="rcl" package="R0805W" value="DNP" x="49.15" y="17.6" rot="R180"/>
-<element name="R99" library="rcl" package="R0805W" value="DNP" x="49.15" y="11.3" rot="R180"/>
+<element name="R98" library="rcl" package="R0805W" value="4K7" x="49.15" y="17.6" rot="R180"/>
+<element name="R99" library="rcl" package="R0805W" value="4K7" x="49.15" y="11.3" rot="R180"/>
 <element name="C19" library="rcl" package="C0805" value="100n" x="54.4" y="29.95" rot="MR180"/>
 <element name="C20" library="rcl" package="C0805" value="100n" x="54.4" y="48.35" rot="MR180"/>
@@
 <element name="R114" library="Simplex-Jumpers" package="R0805W" value="0R_0805" x="66.2" y="36.3" rot="MR270"/>
 <element name="R66" library="Simplex-Jumpers" package="R0805W" value="0R_0805" x="80.15" y="33.7" rot="MR270"/>
+<element name="R79" library="rcl" package="R0805W" value="10K" x="49.17" y="13.34" rot="R180"/>
+<element name="R96" library="rcl" package="R0805W" value="10K" x="49.15" y="15.54" rot="R180"/>
 </elements>
 <signals>
@@
 <signal name="N$36">
 <contactref element="JP1" pad="2"/>
-<contactref element="R96" pad="2"/>
-<wire x1="50.09" y1="15.5" x2="50.19" y2="15.4" width="0.4064" layer="1"/>
 <wire x1="50.19" y1="15.4" x2="55.29" y2="15.4" width="0.3048" layer="1"/>
 <wire x1="55.29" y1="15.4" x2="56.45" y2="14.14" width="0.4064" layer="1" curve="-90"/>
+<contactref element="R96" pad="1"/>
+<wire x1="50.19" y1="15.4" x2="50.2025" y2="15.4" width="0.4064" layer="1"/>
+<wire x1="50.2025" y1="15.4" x2="50.2025" y2="15.54" width="0.4064" layer="1"/>
 </signal>
 <signal name="N$42">
-<contactref element="R96" pad="1"/>
 <contactref element="IC5" pad="16"/>
 <contactref element="R98" pad="2"/>
 <wire x1="38.25" y1="18.595" x2="39.795" y2="18.595" width="0.4064" layer="1"/>
 <via x="40.2" y="18.6" extent="1-16" drill="0.4"/>
-<wire x1="48.21" y1="15.5" x2="48.21" y2="17.6" width="0.6096" layer="1"/>
 <wire x1="48.21" y1="17.6" x2="48.0975" y2="17.6" width="0.4064" layer="1"/>
 <wire x1="40.2" y1="18.6" x2="43.6" y2="18.6" width="0.4064" layer="16"/>
@@
 <wire x1="39.795" y1="18.595" x2="39.795" y2="18.6" width="0.4064" layer="1"/>
 <wire x1="39.795" y1="18.6" x2="40.2" y2="18.6" width="0.4064" layer="1"/>
+<contactref element="R96" pad="2"/>
+<wire x1="48.0975" y1="15.54" x2="48.0975" y2="17.6" width="0.4064" layer="1"/>
 </signal>
 <signal name="N$79">
-<contactref element="R97" pad="1"/>
 <contactref element="IC5" pad="9"/>
 <contactref element="R99" pad="2"/>
@@
 <wire x1="44.55" y1="11.25" x2="48.0475" y2="11.25" width="0.4064" layer="1"/>
 <wire x1="48.0475" y1="11.25" x2="48.0975" y2="11.3" width="0.4064" layer="1" curve="90"/>
-<wire x1="48.0975" y1="11.3" x2="48.0975" y2="13.4" width="0.6096" layer="1"/>
-<wire x1="48.0975" y1="13.4" x2="48.21" y2="13.4" width="0.4064" layer="1"/>
+<wire x1="48.0975" y1="11.3" x2="48.0975" y2="13.25" width="0.6096" layer="1"/>
+<contactref element="R79" pad="2"/>
+<wire x1="48.0975" y1="13.25" x2="48.0975" y2="13.4" width="0.6096" layer="1"/>
+<wire x1="48.1175" y1="13.34" x2="48.1175" y2="13.27" width="0.4064" layer="1"/>
+<wire x1="48.1175" y1="13.27" x2="48.0975" y2="13.25" width="0.4064" layer="1" curve="-90"/>
 </signal>
 <signal name="N$80">
-<contactref element="R97" pad="2"/>
 <contactref element="JP2" pad="2"/>
-<wire x1="50.09" y1="13.4" x2="53.01" y2="13.4" width="0.4064" layer="1"/>
-<wire x1="53.01" y1="13.4" x2="53.85" y2="14.14" width="0.4064" layer="1" curve="90"/>
+<contactref element="R79" pad="1"/>
+<wire x1="50.2225" y1="13.34" x2="53.05" y2="13.34" width="0.4064" layer="1"/>
+<wire x1="53.05" y1="13.34" x2="53.85" y2="14.14" width="0.4064" layer="1" curve="90"/>
 </signal>
 <signal name="+5V">

Commit message: new power amp
Parts:
- added JP3: (no value), SparkFun-Passives:SJ_2S-NO
- added R115, R97: NA/4K7, rcl:R0805W
Connections:
- net N$14 renamed P4.5
- net N$21 renamed P4.4
- removed net RX: R22.1, X1.5, X3.2
- removed net TX: R27.1, X1.6, X3.3
- new net N$13: JP3.1, R115.1, R97.1
- new net RX/SDA: R22.1, R97.2, X1.5, X3.2
- new net TX/SCL: R115.2, R27.1, X1.6, X3.3
- net 3V3: now also JP3.2
Routing:
- net RX/SDA: track 0.00 -> 24.0 mm, vias 0 -> 1
- net TX/SCL: track 0.00 -> 22.3 mm
- net RX: track 20.0 -> 0.00 mm, vias 1 -> 0
- net TX: track 17.9 -> 0.00 mm
- net 3V3: track 150.9 -> 162.8 mm
- net N$13: track 0.00 -> 5.09 mm
Changed lines of the file:
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@@
 <element name="R79" library="rcl" package="R0805W" value="10K" x="49.17" y="13.34" rot="R180"/>
 <element name="R96" library="rcl" package="R0805W" value="10K" x="49.15" y="15.54" rot="R180"/>
+<element name="R97" library="rcl" package="R0805W" value="NA/4K7" x="11.05" y="88.2" rot="R180"/>
+<element name="R115" library="rcl" package="R0805W" value="NA/4K7" x="11.05" y="90.3" rot="R180"/>
+<element name="JP3" library="SparkFun-Passives" package="SJ_2S-NO" value="" x="15.5" y="89.3"/>
 </elements>
 <signals>
@@
 <wire x1="11.15" y1="61.55" x2="10.15" y2="61.55" width="0.3048" layer="1"/>
 </signal>
-<signal name="N$14">
+<signal name="P4.5">
 <contactref element="U$11" pad="34"/>
 <contactref element="R22" pad="2"/>
@@
 <wire x1="12.5" y1="76.5" x2="12.1025" y2="76.5" width="0.3048" layer="1"/>
 </signal>
-<signal name="N$21">
+<signal name="P4.4">
 <contactref element="U$11" pad="33"/>
 <contactref element="R27" pad="2"/>
@@
 <wire x1="20.6" y1="68.5" x2="18.55" y2="68.5" width="0.3048" layer="1"/>
 </signal>
-<signal name="RX">
+<signal name="RX/SDA">
 <contactref element="R22" pad="1"/>
 <contactref element="X1" pad="5"/>
@@
 <wire x1="6.2" y1="87.7" x2="3.4" y2="87.7" width="0.4064" layer="16"/>
 <wire x1="3.4" y1="87.7" x2="3.35" y2="87.75" width="0.4064" layer="16"/>
+<contactref element="R97" pad="2"/>
+<wire x1="9.9975" y1="88.2" x2="7.85" y2="88.2" width="0.4064" layer="1"/>
+<wire x1="7.85" y1="88.2" x2="7.35" y2="87.7" width="0.4064" layer="1"/>
+<wire x1="7.35" y1="87.7" x2="6.2" y2="87.7" width="0.4064" layer="1"/>
 </signal>
-<signal name="TX">
+<signal name="TX/SCL">
 <contactref element="R27" pad="1"/>
 <contactref element="X1" pad="6"/>
@@
 <wire x1="4.3" y1="88.55" x2="4.7" y2="88.95" width="0.4064" layer="1"/>
 <wire x1="4.7" y1="88.95" x2="6.2" y2="88.95" width="0.4064" layer="1"/>
+<contactref element="R115" pad="2"/>
+<wire x1="6.2" y1="88.95" x2="7.45" y2="88.95" width="0.4064" layer="1"/>
+<wire x1="7.45" y1="88.95" x2="8.8" y2="90.3" width="0.4064" layer="1"/>
+<wire x1="8.8" y1="90.3" x2="9.9975" y2="90.3" width="0.4064" layer="1"/>
 </signal>
 <signal name="N$30">
@@
 <wire x1="20.8" y1="63.5" x2="20.8" y2="65.6" width="0.4064" layer="1"/>
 <wire x1="20.8" y1="65.6" x2="20.75" y2="65.65" width="0.4064" layer="1"/>
+<wire x1="8.05" y1="87.05" x2="7.45" y2="86.45" width="0.4064" layer="1"/>
+<wire x1="7.45" y1="86.45" x2="6.2" y2="86.45" width="0.4064" layer="1"/>
+<contactref element="JP3" pad="2"/>
+<wire x1="8.05" y1="87.05" x2="15.35" y2="87.05" width="0.4064" layer="1"/>
+<wire x1="15.35" y1="87.05" x2="15.95" y2="87.65" width="0.4064" layer="1"/>
+<wire x1="15.95" y1="87.65" x2="15.95" y2="89.3" width="0.4064" layer="1"/>
 </signal>
 <signal name="CENTER">
@@
 <contactref element="U$11" pad="43"/>
 </signal>
+<signal name="N$13">
+<contactref element="R97" pad="1"/>
+<contactref element="R115" pad="1"/>
+<wire x1="12.1025" y1="90.3" x2="12.1025" y2="89.4" width="0.4064" layer="1"/>
+<contactref element="JP3" pad="1"/>
+<wire x1="12.1025" y1="89.4" x2="12.1025" y2="88.2" width="0.4064" layer="1"/>
+<wire x1="15.05" y1="89.3" x2="12.2025" y2="89.3" width="0.4064" layer="1"/>
+<wire x1="12.2025" y1="89.3" x2="12.1025" y2="89.4" width="0.4064" layer="1"/>
+</signal>
 </signals>
