File: hardware/amp.brd (EAGLE design)
At the start: 100 x 100 mm, 1 part

Commit message: amp update
Parts:
- added U$1: STK465HORIZ-BOTTOM, Simplex-ICs:STK465-HB
- moved U$7 83.1 mm to (5.35, 12.7), turned to 90 degrees
Connections:
- new net GND: U$1.3
Other:
- board text added: "2x15W amplifier circuit rev 1.0 github.com/rodan/ampy author: petre rodan date: apr 2014"
- board text removed: "audio mixer rev 1.0 github.com/rodan/ampy author: petre rodan date: apr 2014"
Changed lines of the file:
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@@
 <circle x="95" y="5" radius="3.27299375" width="0.4064" layer="42"/>
 <circle x="5" y="5" radius="3.27299375" width="0.4064" layer="42"/>
-<text x="15.05" y="93.5" size="0.8128" layer="108" font="vector" ratio="15">audio mixer rev 1.0
+<text x="7.3" y="15.7" size="0.8128" layer="108" font="vector" ratio="15" rot="R90">2x15W amplifier circuit rev 1.0
 github.com/rodan/ampy
 author: petre rodan
@@
 </autorouter>
 <elements>
-<element name="U$7" library="SparkFun" package="OSHW-LOGO-M" value="OSHW-LOGOM" x="12" y="95.45"/>
+<element name="U$7" library="SparkFun" package="OSHW-LOGO-M" value="OSHW-LOGOM" x="5.35" y="12.65" rot="R90"/>
+<element name="U$1" library="Simplex-ICs" package="STK465-HB" value="STK465HORIZ-BOTTOM" x="50" y="50"/>
 </elements>
 <signals>
+<signal name="GND">
+<contactref element="U$1" pad="3"/>
+</signal>
 </signals>
 <errors>

Commit message: amplifier schematic
Parts:
- added C1, C13: 1u, rcl:PANASONIC_B
- added C10, C5: 47u, rcl:PANASONIC_F
- added C11, C3, C4: 100u, rcl:PANASONIC_G
- added C12, C2: 470p, rcl:C0805
- added C6, C9: 100n, rcl:C0805K
- added C7, C8: 10u, rcl:PANASONIC_F
- added JP1: (no value), SparkFun-Connectors:JST-3-PTH
- added R1, R17: 1K, rcl:R0805W
- added R10, R9: 4R7, rcl:0617/17
- added R11, R7: 0R33, rcl:0922/22
- added R12, R8: 33K, rcl:0617/17
- added R13, R5: 3K3, rcl:0617/17
- added R14, R6: 1K, rcl:0617/17
- added R15, R3: 330, rcl:0617/17
- added R16, R2: 33K, rcl:R0805W
- added R18, R19: 20K, rcl:RTRIM3339P
- added R4: 100R, rcl:0617/17
- added X1: 2508-5, Simplex-Connectors:PAK100/2500-5-08
- U$1: value STK465HORIZ-BOTTOM -> STK465
Connections:
- new net +24V: C7.+, JP1.1, R4.1, U$1.9
- new net -24V: C8.-, JP1.3, R14.1, R6.1, U$1.12
- new net GND_I: C12.2, C2.2, R16.1, R18.3, R19.3, R2.1, X1.2, X1.4
- new net IN_L: R18.1, X1.1
- new net IN_R: R19.1, X1.3
- new net N$1: C4.-, R3.2
- new net N$10: C1.+, R18.2
- new net N$11: C13.+, R19.2
- new net N$12: R11.1, U$1.11
- new net N$13: C11.-, R15.2
- new net N$14: R16.2, R17.1, U$1.16
- new net N$15: C12.1, C13.-, R17.2
- new net N$17: C11.+, R12.2, U$1.15
- new net N$18: C10.-, R13.1, R14.2
- new net N$19: R13.2, U$1.13
- new net N$2: C4.+, R8.2, U$1.2
- new net N$20: C9.2, R10.2
- new net N$3: C5.-, R5.1, R6.2
- new net N$4: C6.2, R9.2
- new net N$5: R7.1, U$1.6
- new net N$6: C3.+, R4.2, U$1.8
- new net N$7: R5.2, U$1.4
- new net N$8: R1.1, R2.2, U$1.1
- new net N$9: C1.-, C2.1, R1.2
- new net OUT_L: C5.+, C6.1, R7.2, R8.1, U$1.7, X1.5
- new net OUT_R: C10.+, C9.1, R11.2, R12.1, U$1.10, X1.7
- net GND: now also C3.-, C7.-, C8.+, JP1.2, R10.1, R15.1, R3.1, R9.1, U$1.14, U$1.5, X1.6, X1.8

Commit message: amp routed
Parts:
- added R20: 0R_0805, Simplex-Jumpers:R0805W
- C6, C9: device rcl:C0805K -> capacitor-wima:C10B5
- JP1: value (none) -> power; device SparkFun-Connectors:JST-3-PTH -> SparkFun-Connectors:1X03
- U$1: value STK465 -> STK465HORIZ-BOTTOM
- moved C7 250.8 mm to (82.7, 21.2), turned to 270 degrees
- moved C8 232.9 mm to (82.7, 8.95), turned to 270 degrees
- moved C2 217.8 mm to (94.8, 83.3), turned to 180 degrees
- moved R1 217.4 mm to (94.8, 85.4)
- moved R2 217.0 mm to (94.8, 87.5), turned to 180 degrees
- moved C1 216.9 mm to (94.8, 79.7)
- moved R12 216.8 mm to (12.4, 37.2), turned to 90 degrees
- moved R14 211.9 mm to (25.0, 37.2), turned to 270 degrees
- moved C13 209.2 mm to (6.10, 74.3)
- moved C9 206.7 mm to (22.5, 21.9), turned to 180 degrees
- moved R10 204.6 mm to (22.4, 13.8), turned to 180 degrees
- moved R17 204.0 mm to (5.95, 68.7), turned to 180 degrees
- moved R13 202.2 mm to (18.7, 37.2), turned to 90 degrees
- moved C11 200.6 mm to (9.50, 55.7)
- moved C12 200.2 mm to (5.95, 70.8)
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Connections:
- net -24V: now also U$1.5
- net GND: now also R20.2; no longer U$1.5
- net GND_I: now also R20.1
Routing:
- net OUT_R: track 0.00 -> 117.2 mm, vias 0 -> 1
- net -24V: track 0.00 -> 108.2 mm, vias 0 -> 4
- net N$11: track 0.00 -> 93.4 mm, vias 0 -> 1
- net OUT_L: track 0.00 -> 91.0 mm, vias 0 -> 2
- net +24V: track 0.00 -> 76.9 mm, vias 0 -> 4
- net N$8: track 0.00 -> 49.0 mm
- net N$6: track 0.00 -> 43.4 mm, vias 0 -> 1
- net IN_R: track 0.00 -> 40.6 mm
- net N$17: track 0.00 -> 37.8 mm, vias 0 -> 1
- net GND_I: track 0.00 -> 33.7 mm, vias 0 -> 22
- net N$14: track 0.00 -> 32.9 mm
- net IN_L: track 0.00 -> 27.9 mm
- net N$2: track 0.00 -> 25.9 mm
- net GND: track 0.00 -> 25.2 mm, vias 0 -> 49
- net N$19: track 0.00 -> 21.5 mm
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- added copper zone on layer 1, net GND
- added copper zone on layer 16, net GND
- added copper zone on layer 1, net GND_I
- added copper zone on layer 16, net GND_I
