File: hardware/amp.brd (EAGLE design)
At the start: 100 x 100 mm, 37 parts, among them X1 2508-5

Commit message: sent to manufacture
Parts:
- moved U$7 1.41 mm to (12.4, 4.15)
- moved R7 0.20 mm to (44.3, 33.1)
Other:
- board text added: "IO IN_L GND IN_R GND OUT_L GND OUT_R GND"
- board text added: "L"
- board text added: "R"
- board text added: "power +24V GND -24V"
Changed lines of the file:
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@@
 <circle x="95" y="5" radius="3.27299375" width="0.4064" layer="42"/>
 <circle x="5" y="5" radius="3.27299375" width="0.4064" layer="42"/>
-<text x="16.65" y="3.05" size="0.8128" layer="108" font="vector" ratio="15">2x15W amplifier circuit rev 1.0
+<text x="16.2" y="2.3" size="0.8128" layer="108" font="vector" ratio="15">2x15W amplifier circuit rev 1.0
 github.com/rodan/ampy
 author: petre rodan
@@
 <text x="81.05" y="0.85" size="0.8128" layer="1" font="vector" ratio="20">1   </text>
 <text x="81.95" y="0.85" size="0.8128" layer="16" font="vector" ratio="20">2</text>
+<text x="92" y="12.3" size="0.8128" layer="108" font="vector" ratio="15">power
++24V
+GND
+-24V</text>
+<text x="89.3" y="21.05" size="0.8128" layer="108" font="vector" ratio="15">IO
+IN_L  GND
+IN_R  GND
+OUT_L GND
+OUT_R GND</text>
+<text x="90.8" y="68.4" size="0.8128" layer="108" font="vector" ratio="15">L</text>
+<text x="90.8" y="76.1" size="0.8128" layer="108" font="vector" ratio="15">R</text>
+<wire x1="88.6" y1="28.45" x2="96.45" y2="28.45" width="0.1" layer="108"/>
+<wire x1="96.45" y1="28.45" x2="96.45" y2="26.35" width="0.1" layer="108"/>
+<wire x1="96.45" y1="26.35" x2="96.45" y2="20.45" width="0.1" layer="108"/>
+<wire x1="96.45" y1="20.45" x2="88.6" y2="20.45" width="0.1" layer="108"/>
+<wire x1="88.6" y1="20.45" x2="88.6" y2="26.35" width="0.1" layer="108"/>
+<wire x1="88.6" y1="26.35" x2="88.6" y2="28.45" width="0.1" layer="108"/>
+<wire x1="88.6" y1="26.35" x2="96.45" y2="26.35" width="0.1" layer="108"/>
+<wire x1="91.8" y1="18.3" x2="96" y2="18.3" width="0.1" layer="108"/>
+<wire x1="96" y1="18.3" x2="96" y2="16.35" width="0.1" layer="108"/>
+<wire x1="96" y1="16.35" x2="96" y2="11.75" width="0.1" layer="108"/>
+<wire x1="96" y1="11.75" x2="91.8" y2="11.75" width="0.1" layer="108"/>
+<wire x1="91.8" y1="11.75" x2="91.8" y2="16.35" width="0.1" layer="108"/>
+<wire x1="91.8" y1="16.35" x2="91.8" y2="18.3" width="0.1" layer="108"/>
+<wire x1="91.8" y1="16.35" x2="96" y2="16.35" width="0.1" layer="108"/>
 </plain>
 <attributes>
@@
 </autorouter>
 <elements>
-<element name="U$7" library="SparkFun" package="OSHW-LOGO-M" value="OSHW-LOGOM" x="13.1" y="5.4"/>
+<element name="U$7" library="SparkFun" package="OSHW-LOGO-M" value="OSHW-LOGOM" x="12.45" y="4.15"/>
 <element name="R3" library="rcl" package="0617/17" value="330" x="79.9" y="37.2" rot="R90"/>
 <element name="R5" library="rcl" package="0617/17" value="3K3" x="67.25" y="37.2" rot="R90"/>
 <element name="R6" library="rcl" package="0617/17" value="1K" x="60.95" y="37.2" rot="R270"/>
-<element name="R7" library="rcl" package="0922/22" value="0R33" x="44.1" y="33.15" rot="R270"/>
+<element name="R7" library="rcl" package="0922/22" value="0R33" x="44.3" y="33.15" rot="R270"/>
 <element name="R8" library="rcl" package="0617/17" value="33K" x="73.6" y="37.2" rot="R90"/>
 <element name="C4" library="rcl" package="PANASONIC_G" value="100u" x="90.5" y="55.7" rot="R180"/>
@@
 <contactref element="R7" pad="1"/>
 <contactref element="U$1" pad="6"/>
-<wire x1="44.1" y1="44.58" x2="49.88" y2="44.58" width="1.016" layer="16"/>
+<wire x1="44.3" y1="44.58" x2="49.88" y2="44.58" width="1.016" layer="16"/>
 <wire x1="49.88" y1="44.58" x2="53.15" y2="47.85" width="1.016" layer="16"/>
 <wire x1="53.15" y1="47.85" x2="55.6" y2="47.85" width="1.016" layer="16"/>
@@
 <wire x1="56.85" y1="38.4" x2="56.85" y2="34.15" width="1.016" layer="1"/>
 <wire x1="51.57" y1="21.85" x2="51.34" y2="21.72" width="1.016" layer="1"/>
-<wire x1="51.34" y1="21.72" x2="44.1" y2="21.72" width="1.016" layer="1"/>
+<wire x1="51.34" y1="21.72" x2="44.3" y2="21.72" width="1.016" layer="1"/>
 <wire x1="56.85" y1="34.15" x2="56.85" y2="27.13" width="1.016" layer="16"/>
 <via x="55.8" y="38.65" extent="1-16" drill="0.7"/>
@@
 <contactref element="X1" pad="3"/>
 <wire x1="84.08" y1="38.47" x2="82.6" y2="39.95" width="0.6096" layer="16"/>
-<wire x1="88.45" y1="70.84" x2="92.26" y2="73.5" width="0.6096" layer="16"/>
-<wire x1="87.8" y1="49.5" x2="87.8" y2="70.19" width="0.6096" layer="16"/>
-<wire x1="87.8" y1="70.19" x2="88.45" y2="70.84" width="0.6096" layer="16"/>
 <wire x1="87.8" y1="49.5" x2="82.6" y2="44.3" width="0.6096" layer="16"/>
 <wire x1="82.6" y1="44.3" x2="82.6" y2="39.95" width="0.6096" layer="16"/>
 <wire x1="84.08" y1="38.47" x2="84.63" y2="38.47" width="0.6096" layer="16"/>
+<wire x1="87.8" y1="69.04" x2="92.26" y2="73.5" width="0.6096" layer="16"/>
+<wire x1="87.8" y1="49.5" x2="87.8" y2="69.04" width="0.6096" layer="16"/>
 </signal>
 <signal name="N$10">

Commit message: board rev 1.1
Parts:
- C7, C8: device rcl:PANASONIC_F -> rcl:PANASONIC_D
- R10, R12, R13, R14, R15, R3, R4, R5, R6, R8, R9: device rcl:0617/17 -> rcl:P0613/15
- R11, R7: device rcl:0922/22 -> rcl:P0613/15
- moved R9 20.3 mm to (43.5, 29.4), turned to 270 degrees
- moved C7 18.4 mm to (69.4, 8.45), turned to 90 degrees
- moved R10 17.7 mm to (30.9, 29.4), turned to 270 degrees
- moved C4 17.4 mm to (78.1, 43.5)
- moved C5 13.5 mm to (60.5, 12.8)
- moved C9 12.3 mm to (31.1, 13.1), turned to 90 degrees
- moved C11 12.2 mm to (10.8, 43.5)
- moved C6 11.4 mm to (49.4, 13.1), turned to 270 degrees
- moved C10 10.8 mm to (15.1, 12.8)
- moved R3 7.99 mm to (81.4, 29.4)
- moved R4 7.99 mm to (56.1, 29.4)
- moved R5 7.99 mm to (68.8, 29.4)
- moved R6 7.99 mm to (62.5, 29.4)
- moved R8 7.99 mm to (75.1, 29.4)
- moved R12 7.91 mm to (12.1, 29.4)
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Connections:
- net IN_L: now also X1.3; no longer X1.1
- net IN_R: now also X1.1; no longer X1.3
- net N$12: now also R11.2; no longer R11.1
- net N$5: now also R7.2; no longer R7.1
- net OUT_L: now also R7.1, X1.7; no longer R7.2, X1.5
- net OUT_R: now also R11.1, X1.5; no longer R11.2, X1.7
Routing:
- net OUT_R: track 117.2 -> 138.2 mm, vias 1 -> 4
- net GND: track 25.2 -> 10.0 mm, vias 50 -> 37
- net N$1: track 19.0 -> 7.18 mm
- net N$6: track 43.4 -> 53.4 mm, vias 1 -> 0
- net +24V: track 76.9 -> 67.3 mm, vias 4 -> 2
- net N$7: track 7.44 -> 16.1 mm
- net N$19: track 21.5 -> 29.5 mm
- net N$2: track 25.9 -> 18.3 mm
- net N$17: track 37.8 -> 30.7 mm, vias 1 -> 0
- net N$4: track 9.75 -> 16.1 mm
- net -24V: track 108.2 -> 102.1 mm, vias 4 -> 2
- net N$20: track 9.67 -> 3.63 mm
- net IN_R: track 40.2 -> 34.8 mm
- net IN_L: track 27.9 -> 32.9 mm, vias 0 -> 2
- net N$3: track 12.9 -> 17.6 mm
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Other:
- board text added: "2x25W amplifier circuit rev 1.1 github.com/rodan/ampy author: petre rodan date: apr 2014"
- board text added: "IO IN_R GND IN_L GND OUT_R GND OUT_L GND"
- board text removed: "2x15W amplifier circuit rev 1.0 github.com/rodan/ampy author: petre rodan date: apr 2014"
- board text removed: "IO IN_L GND IN_R GND OUT_L GND OUT_R GND"

Commit message: add pic link
Parts:
- moved C6 0.45 mm to (49.8, 13.1)
Routing:
- net N$8: track 49.0 -> 50.3 mm
- net GND: vias 37 -> 55
Changed lines of the file:
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@@
 <circle x="95" y="5" radius="3.27299375" width="0.4064" layer="42"/>
 <circle x="5" y="5" radius="3.27299375" width="0.4064" layer="42"/>
-<text x="16.2" y="2.3" size="0.8128" layer="108" font="vector" ratio="15">2x25W amplifier circuit rev 1.1
+<text x="16.1" y="1.95" size="0.8128" layer="108" font="vector" ratio="15">2x25W amplifier circuit rev 1.1
 github.com/rodan/ampy
 author: petre rodan
@@
 <element name="U$1" library="Simplex-ICs" package="STK465-HB" value="STK465HORIZ-BOTTOM" x="50" y="50"/>
 <element name="R20" library="Simplex-Jumpers" package="R0805W" value="0R_0805" x="50" y="60.7" rot="R270"/>
-<element name="C6" library="capacitor-wima" package="C10B5" value="100n" x="49.35" y="13.1" rot="R270"/>
+<element name="C6" library="capacitor-wima" package="C10B5" value="100n" x="49.8" y="13.1" rot="R270"/>
 <element name="C9" library="capacitor-wima" package="C10B5" value="100n" x="31.15" y="13.1" rot="R90"/>
 <element name="JP1" library="SparkFun-Connectors" package="1X03" value="power" x="81.75" y="17.7" rot="R270"/>
@@
 <via x="74.9" y="6.7" extent="1-16" drill="0.8"/>
 <via x="74.9" y="5.4" extent="1-16" drill="0.8"/>
+<via x="53.1" y="14.55" extent="1-16" drill="0.8"/>
+<via x="53" y="18.55" extent="1-16" drill="0.8"/>
+<via x="59.35" y="23.9" extent="1-16" drill="0.8"/>
+<via x="65.55" y="23.95" extent="1-16" drill="0.8"/>
+<via x="74.35" y="23.95" extent="1-16" drill="0.8"/>
+<via x="74.4" y="28.35" extent="1-16" drill="0.8"/>
+<via x="65.65" y="28.4" extent="1-16" drill="0.8"/>
+<via x="59.3" y="28.4" extent="1-16" drill="0.8"/>
+<via x="46.65" y="28.4" extent="1-16" drill="0.8"/>
+<via x="46.7" y="23.75" extent="1-16" drill="0.8"/>
+<via x="80.15" y="33.95" extent="1-16" drill="0.8"/>
+<via x="82.55" y="25.95" extent="1-16" drill="0.8"/>
+<via x="46.7" y="40.15" extent="1-16" drill="0.8"/>
+<via x="63.4" y="18.2" extent="1-16" drill="0.8"/>
+<via x="68.25" y="15" extent="1-16" drill="0.8"/>
+<via x="91.45" y="47.95" extent="1-16" drill="0.8"/>
+<via x="42.5" y="8.25" extent="1-16" drill="0.8"/>
+<via x="42.55" y="6.85" extent="1-16" drill="0.8"/>
 </signal>
 <signal name="N$1">
@@
 <contactref element="C6" pad="1"/>
 <contactref element="R7" pad="1"/>
-<wire x1="49.85" y1="21.73" x2="49.85" y2="18.68" width="1.27" layer="1"/>
-<wire x1="49.85" y1="18.68" x2="49.35" y2="18.18" width="1.27" layer="1"/>
 <wire x1="64.05" y1="15.15" x2="66.7" y2="17.8" width="1.27" layer="1"/>
 <wire x1="66.7" y1="17.8" x2="71.17" y2="17.8" width="1.27" layer="1"/>
@@
 <wire x1="64.05" y1="12.75" x2="60.8" y2="9.5" width="1.27" layer="1"/>
 <wire x1="60.8" y1="9.5" x2="53.85" y2="9.5" width="1.27" layer="1"/>
-<wire x1="53.85" y1="9.5" x2="49.35" y2="14" width="1.27" layer="1"/>
-<wire x1="49.35" y1="14" x2="49.35" y2="18.18" width="1.27" layer="1"/>
 <wire x1="64.05" y1="12.75" x2="64.05" y2="15.15" width="1.27" layer="1"/>
 <contactref element="X1" pad="7"/>
@@
 <wire x1="50.7" y1="33.7" x2="53.81" y2="36.81" width="1.27" layer="1"/>
 <wire x1="53.81" y1="36.81" x2="53.81" y2="50" width="1.27" layer="1"/>
+<wire x1="49.85" y1="21.73" x2="49.8" y2="21.73" width="1.27" layer="1"/>
+<wire x1="49.8" y1="21.73" x2="49.8" y2="18.18" width="1.27" layer="1"/>
+<wire x1="49.8" y1="18.18" x2="49.8" y2="13.55" width="1.27" layer="1"/>
+<wire x1="49.8" y1="13.55" x2="53.85" y2="9.5" width="1.27" layer="1"/>
 </signal>
 <signal name="N$7">
@@
 <contactref element="R9" pad="2"/>
 <contactref element="C6" pad="2"/>
-<wire x1="49.35" y1="8.02" x2="46" y2="11.37" width="1.27" layer="1"/>
-<wire x1="46" y1="11.37" x2="46" y2="19.28" width="1.27" layer="1"/>
-<wire x1="46" y1="19.28" x2="43.55" y2="21.73" width="1.27" layer="1"/>
+<wire x1="43.55" y1="21.73" x2="46.5" y2="18.78" width="1.27" layer="1"/>
+<wire x1="46.5" y1="18.78" x2="46.5" y2="11.32" width="1.27" layer="1"/>
+<wire x1="46.5" y1="11.32" x2="49.8" y2="8.02" width="1.27" layer="1"/>
 </signal>
 <signal name="N$6">
@@
 <contactref element="U$1" pad="1"/>
 <wire x1="93.6975" y1="87.45" x2="93.6975" y2="85.4" width="0.6096" layer="1"/>
-<wire x1="69.05" y1="50" x2="71.4" y2="50" width="0.6096" layer="1"/>
-<wire x1="71.4" y1="50" x2="88.65" y2="67.25" width="0.6096" layer="1"/>
-<wire x1="88.65" y1="67.25" x2="89.55" y2="68.15" width="0.6096" layer="1"/>
-<wire x1="89.55" y1="68.15" x2="89.55" y2="81.2525" width="0.6096" layer="1"/>
-<wire x1="89.55" y1="81.2525" x2="93.6975" y2="85.4" width="0.6096" layer="1"/>
+<wire x1="69.05" y1="50" x2="71.4" y2="50" width="1.016" layer="1"/>
+<wire x1="71.4" y1="50" x2="89.55" y2="68.15" width="1.016" layer="1"/>
+<wire x1="89.55" y1="68.15" x2="89.55" y2="83.4" width="1.016" layer="1"/>
+<wire x1="89.55" y1="83.4" x2="91.55" y2="85.4" width="1.016" layer="1"/>
+<wire x1="91.55" y1="85.4" x2="93.6975" y2="85.4" width="1.016" layer="1"/>
 </signal>
 <signal name="N$9">
@@
 <contactref element="U$1" pad="16"/>
 <wire x1="7.0025" y1="68.65" x2="7.0025" y2="66.5" width="0.6096" layer="1"/>
-<wire x1="7.0025" y1="66.5" x2="14.45" y2="66.5" width="0.6096" layer="1"/>
-<wire x1="14.45" y1="66.5" x2="30.95" y2="50" width="0.6096" layer="1"/>
+<wire x1="7.0025" y1="66.5" x2="14.45" y2="66.5" width="1.016" layer="1"/>
+<wire x1="14.45" y1="66.5" x2="30.95" y2="50" width="1.016" layer="1"/>
 </signal>
 <signal name="N$15">
@@
 <contactref element="R19" pad="2"/>
 <contactref element="C13" pad="+"/>
-<wire x1="10.3" y1="71.7" x2="85.3" y2="71.7" width="0.6096" layer="1"/>
-<wire x1="85.3" y1="71.7" x2="86.85" y2="73.25" width="0.6096" layer="1"/>
-<via x="86.85" y="73.25" extent="1-16" drill="0.6"/>
-<wire x1="86.85" y1="73.25" x2="89.05" y2="73.25" width="0.6096" layer="16"/>
-<wire x1="89.05" y1="73.25" x2="91.15" y2="75.35" width="0.6096" layer="16"/>
-<wire x1="91.15" y1="75.35" x2="93.6" y2="75.35" width="0.6096" layer="16"/>
+<via x="87" y="71.75" extent="1-16" drill="0.6"/>
+<wire x1="90.6" y1="75.35" x2="93.6" y2="75.35" width="0.6096" layer="16"/>
 <wire x1="93.6" y1="75.35" x2="94.9" y2="74.05" width="0.6096" layer="16"/>
 <wire x1="94.9" y1="74.05" x2="94.8" y2="70.96" width="0.6096" layer="16"/>
-<wire x1="10.3" y1="71.7" x2="7.7" y2="74.3" width="0.6096" layer="1"/>
+<wire x1="87" y1="71.75" x2="10.25" y2="71.75" width="1.016" layer="1"/>
+<wire x1="10.25" y1="71.75" x2="7.7" y2="74.3" width="1.016" layer="1"/>
+<wire x1="90.6" y1="75.35" x2="87" y2="71.75" width="0.6096" layer="16"/>
 </signal>
 <signal name="GND_I">
@@
 <via x="90" y="98" extent="1-16" drill="0.8"/>
 <via x="10" y="69.55" extent="1-16" drill="0.8"/>
-<via x="92.35" y="81.65" extent="1-16" drill="0.8"/>
+<via x="91.85" y="82.4" extent="1-16" drill="0.8"/>
 <wire x1="89.27" y1="41.01" x2="89.27" y2="38.47" width="1.016" layer="16"/>
 <wire x1="89.27" y1="41.01" x2="89.27" y2="41.02" width="1.016" layer="16"/>
