File: hardware/power.brd (EAGLE design)
At the start: 92 x 56 mm, 74 parts, among them IC1 7805T, IC2 7905, IC3 7805T, Q1 SI2305, Q3 MOSFET-NCHANNEL_SOT23-3, Q4 MOSFET-NCHANNEL_SOT23-3, Q7 IRFR5305, Q8 IRFR1205, Q9 IRML6246, U1 SPX5205 3v3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

Commit message: cleanup
Connections:
- removed net +3V3: C1.1, C2.1, R32.2, U1.5
- removed net VCC_EN: R4.1, R5.1
- net VCC: now also C1.1, C2.1, R32.2, R4.1, R5.1, U1.5
Changed lines of the file:
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@@
 <hole x="3.6" y="52.1" drill="4.2"/>
 <hole x="87.5" y="4.1" drill="4.2"/>
-<wire x1="34.1" y1="14.3" x2="35.2" y2="14.3" width="0.6096" layer="41"/>
 <text x="94.5" y="49.9" size="0.8128" layer="108" font="vector" ratio="15">gnd</text>
 </plain>
@@
 <wire x1="46.4" y1="48.5475" x2="67.7" y2="42.25" width="0" layer="19" extent="1-1"/>
 </signal>
-<signal name="+3V3">
-<contactref element="U1" pad="5"/>
-<contactref element="C1" pad="1"/>
-<contactref element="C2" pad="1"/>
-<contactref element="R32" pad="2"/>
-<wire x1="35.9001" y1="11.15" x2="-45.2475" y2="-99.3" width="0" layer="19" extent="1-1"/>
-<wire x1="40.4" y1="12.8" x2="35.9001" y2="11.15" width="0" layer="19" extent="1-1"/>
-<wire x1="42.5" y1="13.25" x2="40.4" y2="12.8" width="0" layer="19" extent="1-1"/>
-</signal>
 <signal name="SCL">
 <contactref element="R4" pad="2"/>
@@
 <contactref element="C11" pad="1"/>
 <wire x1="72.8" y1="28.25" x2="74.25" y2="33.3" width="0" layer="19" extent="1-1"/>
-</signal>
-<signal name="VCC_EN">
-<contactref element="R5" pad="1"/>
-<contactref element="R4" pad="1"/>
-<wire x1="85.2475" y1="45.5" x2="85.2475" y2="47.7" width="0" layer="19" extent="1-1"/>
 </signal>
 <signal name="N$11">
@@
 <contactref element="OK2" pad="16"/>
 <contactref element="OK2" pad="12"/>
+<contactref element="R5" pad="1"/>
+<contactref element="R4" pad="1"/>
+<contactref element="U1" pad="5"/>
+<contactref element="C1" pad="1"/>
+<contactref element="C2" pad="1"/>
+<contactref element="R32" pad="2"/>
 <wire x1="-233.36" y1="-238.235" x2="-233.36" y2="-240.775" width="0" layer="19" extent="1-1"/>
 <wire x1="-233.36" y1="-235.695" x2="-233.36" y2="-238.235" width="0" layer="19" extent="1-1"/>
 <wire x1="-233.36" y1="-233.155" x2="-233.36" y2="-235.695" width="0" layer="19" extent="1-1"/>
-<wire x1="43.8" y1="48.5475" x2="-233.36" y2="-233.155" width="0" layer="19" extent="1-1"/>
+<wire x1="-45.2475" y1="-99.3" x2="-233.36" y2="-233.155" width="0" layer="19" extent="1-1"/>
+<wire x1="35.9001" y1="11.15" x2="-45.2475" y2="-99.3" width="0" layer="19" extent="1-1"/>
+<wire x1="40.4" y1="12.8" x2="35.9001" y2="11.15" width="0" layer="19" extent="1-1"/>
+<wire x1="42.5" y1="13.25" x2="40.4" y2="12.8" width="0" layer="19" extent="1-1"/>
+<wire x1="43.8" y1="48.5475" x2="42.5" y2="13.25" width="0" layer="19" extent="1-1"/>
 <wire x1="67.7" y1="40.35" x2="43.8" y2="48.5475" width="0" layer="19" extent="1-1"/>
 <wire x1="69.7" y1="38.85" x2="67.7" y2="40.35" width="0" layer="19" extent="1-1"/>
@@
 <wire x1="82.35" y1="43.4" x2="78.3" y2="39.85" width="0" layer="19" extent="1-1"/>
 <wire x1="82.35" y1="45.5" x2="82.35" y2="43.4" width="0" layer="19" extent="1-1"/>
+<wire x1="85.2475" y1="45.5" x2="82.35" y2="45.5" width="0" layer="19" extent="1-1"/>
+<wire x1="85.2475" y1="47.7" x2="85.2475" y2="45.5" width="0" layer="19" extent="1-1"/>
 </signal>
 <signal name="LED">

Commit message: change C footprints
Parts:
- added C13, C15: 100nF, rcl:C0805
- added D1, D2, D3, D4, D5, D6, D7, D8, D9: M4, diode:SMA
- added IC4: 7805T, linear:TO220H
- added OK3, OK4: TLP283-4, optocoupler:MINI-FLAT-16
- added Q5: IRML6246, Simplex-DiscreteSemi:SOT23-3_POWER
- added R28: 560, rcl:R0805W
- added R29: 1K, rcl:R0805W
- added R30: 220R, rcl:R0805W
- added R33: 470R, rcl:R0805W
- added R36: 10K, rcl:R0805W
Connections:
- removed net N$22: R17.1, R18.2
- removed net N$43: C18.1, Q9.1, R46.1
- new net N$32: D8.C, IC4.1
- new net N$33: OK3.2, R28.1
- new net N$34: OK4.1, R29.1
- new net N$35: OK4.15, R30.2
- new net N$37: C13.1, IC4.2, Q5.2, R36.1
- new net N$42: C15.2, OK3.15, Q5.1, R36.2
- net $N1: now also D2.C
- net $N333: now also D1.A
- net +30V: now also D6.C
- net +5V_AN: now also D4.C
- net +5V_DIG: now also D3.A, OK3.1
- net -30V: now also D7.A
- net -5V_AN: now also C15.1, D5.A, D9.A, OK4.2, Q5.3
- net 5_EN: now also R28.2
- net A+5: now also R17.1, R18.2
- net A-5: now also R30.1, R33.2
- net AGND: now also C13.2, D4.A, D5.C, D6.A, D7.C, D8.A, D9.C, IC4.3, OK3.16, R29.2
- net DGND: now also R33.1
- net N$20: now also D3.C
- net N$3: now also D1.C
- net N$4: now also D2.A
- net N$9: now also C18.1, Q9.1, R46.1
- net VCC: now also OK4.16

Commit message: use 7905
Parts:
- removed C15, C18, C7: 100nF, rcl:C0805
- removed D5: M4, diode:SMA
- removed IC2: 7905, linear:TO220H
- removed Q5, Q9: IRML6246, Simplex-DiscreteSemi:SOT23-3_POWER
- removed R36, R46: 10K, rcl:R0805W
- removed U$2: MOLEX_6HORIZONTAL, Simplex-Connectors:0530480610
- added C12: 100nF, rcl:C0805
- added Q2: IRML6246, Simplex-DiscreteSemi:SOT23-3_POWER
- added R26: 10K, rcl:R0805W
- added X1: MOLEX_6VERTICAL, Simplex-Connectors:0530470610
- IC4: value 7805T -> 7905
- R15: value 220R -> 0R
- R16: value 560 -> 0R
- R21: value 470R -> 0R
- R8: value 1K -> 0R
- moved R16 177.5 mm to (-367.0, -333.9)
- moved R8 145.3 mm to (-359.0, -333.9)
- moved R21 113.4 mm to (-371.0, -333.9)
- moved R15 112.4 mm to (-363.0, -333.9)
- moved D2 56.6 mm to (-353.7, -325.4)
Connections:
- removed net $N1: C7.2, D2.C, IC2.3, Q9.2, R46.2
- removed net N$14: OK2.4, R8.1
- removed net N$17: OK1.4, R16.1
- removed net N$23: OK2.13, R15.2
- removed net N$24: R15.1, R21.2
- removed net N$37: C13.1, IC4.2, Q5.2, R36.1
- removed net N$4: D2.A, IC2.2
- removed net N$42: C15.2, OK3.15, Q5.1, R36.2
- removed net N$9: C18.1, OK1.13, Q9.1, R46.1
- new net $N2: C13.2, D8.C, IC4.3, Q2.2, R26.2
- new net N$22: C12.1, OK3.13, Q2.1, R26.1
- new net N$31: D8.A, IC4.2
- net +5V_DIG: now also D2.C, OK3.3; no longer OK1.3, OK3.1
- net -5V_AN: now also C12.2, Q2.3, R29.2; no longer C15.1, C18.2, D5.A, OK4.2, Q5.3, Q9.3, R8.2
- net 5_EN: no longer R16.2
- net A-5: no longer R30.1, R33.2
- net AGND: now also C13.1, IC4.1, OK3.14, OK4.3, R15.2, R16.2, R21.2, R8.2; no longer C13.2, C7.1, D5.C, D8.A, IC2.1, IC4.3, OK1.14, OK2.3, OK3.16, R29.2
- net DGND: now also D2.A, R15.1, R16.1, R8.1
- net GND: now also X1.1
- net N$32: now also OK3.4, R28.1; no longer D8.C, IC4.1
- net N$33: now also OK4.4, R29.1; no longer OK3.2, R28.1
- net N$34: now also OK4.13, R30.2; no longer OK4.1, R29.1
- net N$35: now also R30.1, R33.2; no longer OK4.15, R30.2
- net RST: now also X1.2
- net RX: now also X1.5
- net TEST: now also X1.3
- net TX: now also X1.6
- net VCC: now also OK4.14, X1.4; no longer OK2.14, OK4.16

Commit message: mosfets purchased
Parts:
- Q3, Q4: value MOSFET-NCHANNEL_SOT23-3 -> PMBF170
Changed lines of the file:
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@@
 </element>
 <element name="IC1" library="linear" package="TO220H" value="7805T" x="-194.9" y="-204.7"/>
-<element name="Q4" library="Simplex-DiscreteSemi" package="SOT23-3" value="MOSFET-NCHANNEL_SOT23-3" x="-223.2" y="-215.4"/>
+<element name="Q4" library="Simplex-DiscreteSemi" package="SOT23-3" value="PMBF170" x="-223.2" y="-215.4"/>
 <element name="R11" library="rcl" package="R0805W" value="10K" x="-226.8" y="-213.9"/>
 <element name="R12" library="rcl" package="R0805W" value="560" x="-230.8" y="-213.9"/>
 <element name="R19" library="rcl" package="R0805W" value="1K" x="-230.8" y="-226.1"/>
-<element name="Q3" library="Simplex-DiscreteSemi" package="SOT23-3" value="MOSFET-NCHANNEL_SOT23-3" x="-231.2" y="-231.5"/>
+<element name="Q3" library="Simplex-DiscreteSemi" package="SOT23-3" value="PMBF170" x="-231.2" y="-231.5"/>
 <element name="R20" library="rcl" package="R0805W" value="10K" x="-226.8" y="-226.1"/>
 <element name="R1" library="rcl" package="R0805W" value="560" x="-230.8" y="-236"/>

Commit message: add low voltage power source board
Parts:
- removed C11: 220nF, rcl:C0805
- added IC2: 7805, Simplex-ICs:D2PACK
- IC1: value 7805T -> 7805; device linear:TO220H -> Simplex-ICs:D2PACK
- IC3: value 7805T -> 7815DT; device linear:TO220H -> linear:TO252
- IC4: device linear:TO220H -> Simplex-ICs:D2PACK
- moved IC1 263.8 mm to (-424.9, -333.9)
- moved IC3 164.9 mm to (-400.8, -331.2)
- moved IC4 79.3 mm to (-412.5, -333.9)
Connections:
- removed net 41: U$1.41
- removed net N$7: C11.1, U$1.43
- new net 43: U$1.43
- net +5V_DIG: now also IC2.3; no longer IC3.3
- net AGND: now also IC1.4; no longer IC1.2
- net DGND: now also IC2.4; no longer IC3.2
- net GND: now also U$1.41; no longer C11.2
- net N$20: now also IC2.1; no longer IC3.1
- net N$31: now also IC4.4; no longer IC4.2
