File: hardware/power.sch (EAGLE design)
At the start: 74 parts, among them IC1 7805T, IC2 7905, IC3 7805T, Q1 SI2305, Q3 MOSFET-NCHANNEL_SOT23-3, Q4 MOSFET-NCHANNEL_SOT23-3, Q7 IRFR5305, Q8 IRFR1205, Q9 IRML6246, U1 SPX5205 3v3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

Commit message: cleanup
Connections:
- removed net +3V3: C1.1, C2.1, R32.2, U1.OUT
- removed net VCC_EN: R4.1, R5.1
- net VCC: now also C1.1, C2.1, R32.2, R4.1, R5.1, U1.OUT
Other:
- moved on the sheet: C1, C10, C11, C14, C16, C17, C18, C19, C2, C21, C23, C24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

Commit message: change C footprints
Parts:
- added C13, C15: 100nF, rcl:C-EUC0805
- added D1, D2, D3, D4, D5, D6, D7, D8, D9: M4, diode:MBRA340T3
- added IC4: 7805T, linear:7805T
- added OK3, OK4: TLP283-4, optocoupler:TLP283-4
- added Q5: IRML6246, Simplex-DiscreteSemi:MOSFET-NCHANNEL_SOT23-3_POWER
- added R28: 560, rcl:R-EU_R0805W
- added R29: 1K, rcl:R-EU_R0805W
- added R30: 220R, rcl:R-EU_R0805W
- added R33: 470R, rcl:R-EU_R0805W
- added R36: 10K, rcl:R-EU_R0805W
Connections:
- removed net N$22: R17.1, R18.2
- removed net N$43: C18.1, Q9.G, R46.1
- new net N$32: D8.C, IC4.VI
- new net N$33: OK3A.C, R28.1
- new net N$34: OK4A.A, R29.1
- new net N$35: OK4A.EMIT, R30.2
- new net N$37: C13.1, IC4.GND, Q5.S, R36.1
- new net N$42: C15.2, OK3A.EMIT, Q5.G, R36.2
- net $N1: now also D2.C
- net $N333: now also D1.A
- net +30V: now also D6.C
- net +5V_AN: now also D4.C
- net +5V_DIG: now also D3.A, OK3A.A
- net -30V: now also D7.A
- net -5V_AN: now also C15.1, D5.A, D9.A, OK4A.C, Q5.D
- net 5_EN: now also R28.2
- net A+5: now also R17.1, R18.2
- net A-5: now also R30.1, R33.2
- net AGND: now also C13.2, D4.A, D5.C, D6.A, D7.C, D8.A, D9.C, IC4.VO, OK3A.COL, R29.2
- net DGND: now also R33.1
- net N$20: now also D3.C
- net N$3: now also D1.C
- net N$4: now also D2.A
- net N$9: now also C18.1, Q9.G, R46.1
- net VCC: now also OK4A.COL
Other:
- moved on the sheet: C16, C5, IC1, OK1A, OK2A, Q1, R12, R17, R18, R3, R45

Commit message: use 7905
Parts:
- removed C15, C18, C7: 100nF, rcl:C-EUC0805
- removed D5: M4, diode:MBRA340T3
- removed IC2: 7905, linear:7905T
- removed Q5, Q9: IRML6246, Simplex-DiscreteSemi:MOSFET-NCHANNEL_SOT23-3_POWER
- removed R36, R46: 10K, rcl:R-EU_R0805W
- removed U$2: MOLEX_6HORIZONTAL, Simplex-Connectors:MOLEX_6HORIZONTAL
- added C12: 100nF, rcl:C-EUC0805
- added Q2: IRML6246, Simplex-DiscreteSemi:MOSFET-NCHANNEL_SOT23-3_POWER
- added R26: 10K, rcl:R-EU_R0805W
- added X1: MOLEX_6VERTICAL, Simplex-Connectors:MOLEX_6VERTICAL
- IC4: value 7805T -> 7905; device linear:7805T -> linear:7905T
- R15: value 220R -> 0R
- R16: value 560 -> 0R
- R21: value 470R -> 0R
- R8: value 1K -> 0R
Connections:
- removed net $N1: C7.2, D2.C, IC2.VO, Q9.S, R46.2
- removed net N$14: OK2B.C, R8.1
- removed net N$17: OK1B.C, R16.1
- removed net N$23: OK2B.EMIT, R15.2
- removed net N$24: R15.1, R21.2
- removed net N$37: C13.1, IC4.GND, Q5.S, R36.1
- removed net N$4: D2.A, IC2.VI
- removed net N$42: C15.2, OK3A.EMIT, Q5.G, R36.2
- removed net N$9: C18.1, OK1B.EMIT, Q9.G, R46.1
- new net $N2: C13.2, D8.C, IC4.VO, Q2.S, R26.2
- new net N$22: C12.1, OK3B.EMIT, Q2.G, R26.1
- new net N$31: D8.A, IC4.VI
- net +5V_DIG: now also D2.C, OK3B.A; no longer OK1B.A, OK3A.A
- net -5V_AN: now also C12.2, Q2.D, R29.2; no longer C15.1, C18.2, D5.A, OK4A.C, Q5.D, Q9.D, R8.2
- net 5_EN: no longer R16.2
- net A-5: no longer R30.1, R33.2
- net AGND: now also C13.1, IC4.GND, OK3B.COL, OK4B.A, R15.2, R16.2, R21.2, R8.2; no longer C13.2, C7.1, D5.C, D8.A, IC2.GND, IC4.VO, OK1B.COL, OK2B.A, OK3A.COL, R29.2
- net DGND: now also D2.A, R15.1, R16.1, R8.1
- net GND: now also X1.1
- net N$32: now also OK3B.C, R28.1; no longer D8.C, IC4.VI
- net N$33: now also OK4B.C, R29.1; no longer OK3A.C, R28.1
- net N$34: now also OK4B.EMIT, R30.2; no longer OK4A.A, R29.1
- net N$35: now also R30.1, R33.2; no longer OK4A.EMIT, R30.2
- net RST: now also X1.2
- net RX: now also X1.5
- net TEST: now also X1.3
- net TX: now also X1.6
- net VCC: now also OK4B.COL, X1.4; no longer OK2B.COL, OK4A.COL
Other:
- note added: "INPUTS 2x5V ac 2x30V ac OUTPUTS 3V3 dc digital 5V dc digital 5V dc analog -5V dc analog 24V dc analog -24V dc analog"
- moved on the sheet: C1, C10, C11, C13, C14, C16, C19, C2, C21, C23, C24, C3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

Commit message: mosfets purchased
Parts:
- Q3, Q4: value MOSFET-NCHANNEL_SOT23-3 -> PMBF170
Changed lines of the file:
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@@
 <part name="OK1" library="optocoupler" deviceset="TLP283-4" device=""/>
 <part name="IC1" library="linear" deviceset="78*" device="T" technology="05"/>
-<part name="Q4" library="Simplex-DiscreteSemi" deviceset="MOSFET-NCHANNEL" device="_SOT23-3"/>
+<part name="Q4" library="Simplex-DiscreteSemi" deviceset="MOSFET-NCHANNEL" device="_SOT23-3" value="PMBF170"/>
 <part name="SUPPLY17" library="supply2" deviceset="DGND" device=""/>
 <part name="R11" library="rcl" deviceset="R-EU_" device="R0805W" value="10K"/>
@@
 <part name="R12" library="rcl" deviceset="R-EU_" device="R0805W" value="560"/>
 <part name="R19" library="rcl" deviceset="R-EU_" device="R0805W" value="1K"/>
-<part name="Q3" library="Simplex-DiscreteSemi" deviceset="MOSFET-NCHANNEL" device="_SOT23-3"/>
+<part name="Q3" library="Simplex-DiscreteSemi" deviceset="MOSFET-NCHANNEL" device="_SOT23-3" value="PMBF170"/>
 <part name="SUPPLY5" library="supply2" deviceset="DGND" device=""/>
 <part name="R20" library="rcl" deviceset="R-EU_" device="R0805W" value="10K"/>

Commit message: add low voltage power source board
Parts:
- removed C11: 220nF, rcl:C-EUC0805
- added IC2: 7805, Simplex-ICs:78XX
- IC1: value 7805T -> 7805; device linear:7805T -> Simplex-ICs:78XX
- IC3: value 7805T -> 7815DT; device linear:7805T -> linear:7815DT
- IC4: device linear:7905T -> Simplex-ICs:79XX
Connections:
- removed net N$7: C11.1, U$1.43
- net +5V_DIG: now also IC2.VO; no longer IC3.VO
- net DGND: now also IC2.GND; no longer IC3.GND
- net GND: now also U$1.41; no longer C11.2
- net N$20: now also IC2.VI; no longer IC3.VI
Other:
- moved on the sheet: IC3
Changed lines of the file:
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@@
 <part name="GND22" library="SparkFun" deviceset="GND" device=""/>
 <part name="C10" library="rcl" deviceset="C-EU" device="C0805" value="470nF"/>
-<part name="C11" library="rcl" deviceset="C-EU" device="C0805" value="220nF"/>
-<part name="GND23" library="SparkFun" deviceset="GND" device=""/>
 <part name="GND24" library="SparkFun" deviceset="GND" device=""/>
 <part name="R6" library="rcl" deviceset="R-EU_" device="R0805W" value="4.7k"/>
@@
 <part name="Q8" library="Simplex-DiscreteSemi" deviceset="MOSFET-NCHANNEL" device="_D-PAK" value="IRFR1205"/>
 <part name="OK1" library="optocoupler" deviceset="TLP283-4" device=""/>
-<part name="IC1" library="linear" deviceset="78*" device="T" technology="05"/>
 <part name="Q4" library="Simplex-DiscreteSemi" deviceset="MOSFET-NCHANNEL" device="_SOT23-3" value="PMBF170"/>
 <part name="SUPPLY17" library="supply2" deviceset="DGND" device=""/>
@@
 <part name="SUPPLY25" library="supply2" deviceset="DGND" device=""/>
 <part name="R14" library="rcl" deviceset="R-EU_" device="R0805W" value="0R"/>
-<part name="IC3" library="linear" deviceset="78*" device="T" technology="05"/>
 <part name="SUPPLY26" library="supply2" deviceset="DGND" device=""/>
 <part name="SUPPLY27" library="supply2" deviceset="DGND" device=""/>
@@
 <part name="Q2" library="Simplex-DiscreteSemi" deviceset="MOSFET-NCHANNEL" device="_SOT23-3_POWER" value="IRML6246"/>
 <part name="OK3" library="optocoupler" deviceset="TLP283-4" device=""/>
-<part name="IC4" library="linear" deviceset="79*" device="T" technology="05" value="7905"/>
 <part name="SUPPLY7" library="supply2" deviceset="AGND" device=""/>
 <part name="R28" library="rcl" deviceset="R-EU_" device="R0805W" value="560"/>
@@
 <part name="R16" library="rcl" deviceset="R-EU_" device="R0805W" value="0R"/>
 <part name="R21" library="rcl" deviceset="R-EU_" device="R0805W" value="0R"/>
+<part name="IC3" library="linear" deviceset="78*" device="DT" technology="15"/>
+<part name="IC4" library="Simplex-ICs" deviceset="79XX" device="" value="7905"/>
+<part name="IC1" library="Simplex-ICs" deviceset="78XX" device="" value="7805"/>
+<part name="IC2" library="Simplex-ICs" deviceset="78XX" device="" value="7805"/>
 </parts>
 <sheets>
@@
 <instance part="GND22" gate="1" x="347.98" y="167.64"/>
 <instance part="C10" gate="G$1" x="347.98" y="175.26"/>
-<instance part="C11" gate="G$1" x="414.02" y="195.58" rot="R90"/>
-<instance part="GND23" gate="1" x="421.64" y="195.58" rot="R90"/>
 <instance part="GND24" gate="1" x="449.58" y="175.26"/>
 <instance part="R6" gate="G$1" x="419.1" y="172.72" rot="R180"/>
@@
 <instance part="OK1" gate="C" x="215.9" y="416.56"/>
 <instance part="OK1" gate="D" x="215.9" y="312.42"/>
-<instance part="IC1" gate="A1" x="25.4" y="452.12"/>
 <instance part="Q4" gate="G$1" x="116.84" y="114.3"/>
 <instance part="SUPPLY17" gate="G$1" x="116.84" y="96.52"/>
@@
 <instance part="SUPPLY25" gate="G$1" x="220.98" y="68.58"/>
 <instance part="R14" gate="G$1" x="210.82" y="76.2" rot="R180"/>
-<instance part="IC3" gate="A1" x="-154.94" y="452.12"/>
 <instance part="SUPPLY26" gate="G$1" x="-154.94" y="439.42"/>
 <instance part="SUPPLY27" gate="G$1" x="-132.08" y="426.72"/>
@@
 <instance part="Q2" gate="G$1" x="81.28" y="347.98" rot="MR90"/>
 <instance part="OK3" gate="B" x="68.58" y="312.42"/>
-<instance part="IC4" gate="A1" x="25.4" y="345.44" rot="MR180"/>
 <instance part="SUPPLY7" gate="G$1" x="78.74" y="302.26"/>
 <instance part="R28" gate="G$1" x="43.18" y="309.88" rot="R180"/>
@@
 <instance part="R16" gate="G$1" x="210.82" y="99.06" rot="R180"/>
 <instance part="R21" gate="G$1" x="210.82" y="106.68" rot="R180"/>
+<instance part="IC3" gate="A1" x="-152.4" y="350.52"/>
+<instance part="IC4" gate="IC$1" x="25.4" y="345.44"/>
+<instance part="IC1" gate="IC$1" x="25.4" y="449.58"/>
+<instance part="IC2" gate="IC$1" x="-154.94" y="449.58"/>
 </instances>
 <busses>
@@
 <pinref part="U$1" gate="G$1" pin="12"/>
 <wire x1="342.9" y1="180.34" x2="360.68" y2="180.34" width="0.1524" layer="91"/>
-</segment>
-<segment>
-<pinref part="C11" gate="G$1" pin="2"/>
-<pinref part="GND23" gate="1" pin="GND"/>
 </segment>
 <segment>
@@
 <wire x1="411.48" y1="185.42" x2="416.56" y2="185.42" width="0.1524" layer="91"/>
 <junction x="416.56" y="180.34"/>
+<pinref part="U$1" gate="G$1" pin="41"/>
+<wire x1="411.48" y1="190.5" x2="416.56" y2="190.5" width="0.1524" layer="91"/>
+<wire x1="416.56" y1="190.5" x2="416.56" y2="185.42" width="0.1524" layer="91"/>
+<junction x="416.56" y="185.42"/>
 </segment>
 <segment>
@@
 <pinref part="U$1" gate="G$1" pin="13"/>
 <wire x1="347.98" y1="177.8" x2="360.68" y2="177.8" width="0.1524" layer="91"/>
-</segment>
-</net>
-<net name="N$7" class="0">
-<segment>
-<pinref part="U$1" gate="G$1" pin="43"/>
-<pinref part="C11" gate="G$1" pin="1"/>
 </segment>
 </net>
@@
 <wire x1="-144.78" y1="452.12" x2="-139.7" y2="452.12" width="0.1524" layer="91"/>
 <junction x="-132.08" y="452.12"/>
-<pinref part="IC3" gate="A1" pin="VO"/>
 <label x="-132.08" y="454.66" size="1.778" layer="95"/>
 <wire x1="-139.7" y1="452.12" x2="-132.08" y2="452.12" width="0.1524" layer="91"/>
@@
 <pinref part="D2" gate="G$1" pin="C"/>
 <wire x1="-139.7" y1="441.96" x2="-139.7" y2="452.12" width="0.1524" layer="91"/>
+<pinref part="IC2" gate="IC$1" pin="VO"/>
 </segment>
 <segment>
@@
 <segment>
 <pinref part="SUPPLY26" gate="G$1" pin="DGND"/>
-<pinref part="IC3" gate="A1" pin="GND"/>
 <wire x1="-154.94" y1="441.96" x2="-154.94" y2="444.5" width="0.1524" layer="91"/>
+<pinref part="IC2" gate="IC$1" pin="GND"/>
 </segment>
 <segment>
@@
 </segment>
 <segment>
-<pinref part="IC4" gate="A1" pin="GND"/>
 <wire x1="25.4" y1="340.36" x2="25.4" y2="332.74" width="0.1524" layer="91"/>
 <pinref part="SUPPLY15" gate="G$1" pin="AGND"/>
+<pinref part="IC4" gate="IC$1" pin="GND"/>
 </segment>
 <segment>
@@
 </segment>
 <segment>
-<pinref part="IC1" gate="A1" pin="GND"/>
 <wire x1="25.4" y1="444.5" x2="25.4" y2="434.34" width="0.1524" layer="91"/>
 <pinref part="SUPPLY55" gate="G$1" pin="AGND"/>
+<pinref part="IC1" gate="IC$1" pin="GND"/>
 </segment>
 </net>
 <net name="N$3" class="0">
 <segment>
-<pinref part="IC1" gate="A1" pin="VI"/>
 <wire x1="15.24" y1="452.12" x2="10.16" y2="452.12" width="0.1524" layer="91"/>
 <pinref part="D1" gate="G$1" pin="C"/>
@@
 <junction x="10.16" y="452.12"/>
 <wire x1="10.16" y1="452.12" x2="2.54" y2="452.12" width="0.1524" layer="91"/>
+<pinref part="IC1" gate="IC$1" pin="VI"/>
 </segment>
 </net>
@@
 <junction x="71.12" y="452.12"/>
 <pinref part="Q1" gate="G$1" pin="S"/>
-<pinref part="IC1" gate="A1" pin="VO"/>
 <wire x1="35.56" y1="452.12" x2="40.64" y2="452.12" width="0.1524" layer="91"/>
 <pinref part="C5" gate="G$1" pin="2"/>
@@
 <wire x1="27.94" y1="464.82" x2="40.64" y2="464.82" width="0.1524" layer="91"/>
 <wire x1="40.64" y1="464.82" x2="40.64" y2="452.12" width="0.1524" layer="91"/>
+<pinref part="IC1" gate="IC$1" pin="VO"/>
 </segment>
 </net>
 <net name="N$20" class="0">
 <segment>
-<pinref part="IC3" gate="A1" pin="VI"/>
 <wire x1="-165.1" y1="452.12" x2="-170.18" y2="452.12" width="0.1524" layer="91"/>
 <pinref part="D3" gate="G$1" pin="C"/>
@@
 <wire x1="-170.18" y1="452.12" x2="-177.8" y2="452.12" width="0.1524" layer="91"/>
 <junction x="-170.18" y="452.12"/>
+<pinref part="IC2" gate="IC$1" pin="VI"/>
 </segment>
 </net>
@@
 <net name="N$31" class="0">
 <segment>
-<pinref part="IC4" gate="A1" pin="VI"/>
 <wire x1="15.24" y1="347.98" x2="10.16" y2="347.98" width="0.1524" layer="91"/>
 <wire x1="10.16" y1="347.98" x2="2.54" y2="347.98" width="0.1524" layer="91"/>
@@
 <junction x="10.16" y="347.98"/>
 <pinref part="D8" gate="G$1" pin="A"/>
+<pinref part="IC4" gate="IC$1" pin="VI"/>
 </segment>
 </net>
@@
 <junction x="71.12" y="347.98"/>
 <pinref part="Q2" gate="G$1" pin="S"/>
-<pinref part="IC4" gate="A1" pin="VO"/>
 <wire x1="35.56" y1="347.98" x2="40.64" y2="347.98" width="0.1524" layer="91"/>
 <junction x="40.64" y="347.98"/>
@@
 <wire x1="40.64" y1="360.68" x2="40.64" y2="347.98" width="0.1524" layer="91"/>
 <pinref part="D8" gate="G$1" pin="C"/>
-</segment>
-</net>
+<pinref part="IC4" gate="IC$1" pin="VO"/>
+</segment>
+</net>
