File: hardware/power_amp.brd (EAGLE design)
At the start: 100 x 100 mm, 33 parts, among them X1 DEGSON_4, X2 DEGSON_3

Commit message: sent to manufacture
Other:
- board text added: "-24VDC GND +24VDC"
- board text added: "2x18VAC"
- board text added: "power circuit for amp rev 1.0 github.com/rodan/ampy author: petre rodan date: apr 2014"
- board text removed: "amp power source rev 1.0 github.com/rodan/ampy author: petre rodan date: apr 2014"
Changed lines of the file:
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@@
 <circle x="95" y="5" radius="3.27299375" width="0.4064" layer="42"/>
 <circle x="5" y="5" radius="3.27299375" width="0.4064" layer="42"/>
-<text x="11.25" y="2.15" size="0.8128" layer="108" font="vector" ratio="15">amp power source  rev 1.0
+<text x="11.25" y="2.15" size="0.8128" layer="108" font="vector" ratio="15">power circuit for amp rev 1.0
 github.com/rodan/ampy
 author: petre rodan
@@
 <text x="81.05" y="0.85" size="0.8128" layer="1" font="vector" ratio="20">1   </text>
 <text x="81.95" y="0.85" size="0.8128" layer="16" font="vector" ratio="20">2</text>
+<text x="17.25" y="95.15" size="1.27" layer="108" font="vector" ratio="15">2x18VAC</text>
+<text x="68.75" y="5.15" size="1.27" layer="108" font="vector" ratio="15">-24VDC GND +24VDC</text>
 </plain>
 <attributes>
