File: hardware/mixer.sch (EAGLE design)
At the start: 199 parts, among them IC1 PGA2311, IC10 OPA2134P, IC11 OPA2134P, IC12 OPA2134P, IC13 OPA2134P, IC2 PGA2311, IC3 PGA2311, IC4 PGA2311, IC5 PGA2311, IC6 OPA2134P, IC7 OPA2134P, IC8 OPA2134P, IC9 OPA2134P, Q1 SI2305, Q2 MOSFET-NCHANNEL_SOT23-3, X1 MOLEX_6HORIZONTAL, X2 MOLEX_6HORIZONTAL, X3 MOLEX_4HORIZONTAL, Y1 32768Hz CFPX-217 12.5pF

Commit message: routing
Parts:
- removed C47, C51, C52: 100n, rcl:C-EUC0805
- removed C64, C65, C66, C67, C68, C69, C71, C72, C73, C74, C75, C76, C78, C88, C89, C90: 10u, rcl:CPOL-EU153CLV-0405
- removed R92, R93, R94, R95: 0R_0805, Simplex-Jumpers:0R_0805
- removed U$10, U$3, U$4, U$8: RESETTABLE, Simplex-Fuses:RESETTABLE
- added C17, C18, C19, C20, C21, C22, C24, C25, C26, C28, C32, C33, C63, C79, C80: 100n, rcl:C-EUC0805
- added C92, C96: 10u, rcl:CPOL-EU153CLV-0405
- added R96, R97: 0R_0805, Simplex-Jumpers:0R_0805
- added R98, R99: DNP, rcl:R-EU_R0805W
- added U$12, U$13, U$2, U$5, U$6, U$9: RESETTABLE, Simplex-Fuses:RESETTABLE
- added X4: inputs, con-3m:2514-
- added X5: outputs, con-3m:2514-
- X2: value MOLEX_6HORIZONTAL -> 2514-; device Simplex-Connectors:MOLEX_6HORIZONTAL -> con-3m:2514-
- X3: value MOLEX_4HORIZONTAL -> display
Connections:
- removed net +3V: C84.1, C85.1, C86.1, C87.+, R95.P$2
- removed net +5V_DIG: Q1.S, R37.2, R92.P$1
- removed net A+5V: C29.1, C30.1, C31.1, C34.1, C35.1, C36.1, C37.1, C46.1, C47.1, C48.1, C49.1, C58.2, C59.2, C60.2, C61.2, C62.2, C64.+, C65.+, C66.+, C67.+, C68.+, C69.+, C70.+, IC1.VA+, IC10A.V+, IC11A.V+, IC12A.V+, IC13A.V+, IC2.VA+, IC3.VA+, IC4.VA+, IC5.VA+, IC6A.V+, IC7A.V+, IC8A.V+, IC9A.V+, R94.P$1
- removed net A-5V: C38.1, C39.1, C40.1, C41.1, C42.1, C43.1, C44.1, C51.1, C52.1, C53.1, C54.1, C58.1, C59.1, C60.1, C61.1, C62.1, C71.-, C72.-, C73.-, C74.-, C75.-, C76.-, C77.-, IC1.VA-, IC10A.V-, IC11A.V-, IC12A.V-, IC13A.V-, IC2.VA-, IC3.VA-, IC4.VA-, IC5.VA-, IC6A.V-, IC7A.V-, IC8A.V-, IC9A.V-, R93.P$1
- removed net N$24: U$4.P$2, X2.4
- removed net N$25: U$8.P$2, X2.3
- removed net N$3: R92.P$2, U$8.P$1
- removed net N$34: U$10.P$2, X2.2
- removed net N$6: R95.P$1, U$10.P$1
- removed net N$60: R94.P$2, U$3.P$1
- removed net N$62: R93.P$2, U$4.P$1
- removed net N$63: U$3.P$2, X2.5
- removed net VCC: R34.2, U$11.11, U$11.28, U$11.7, X1.4
- new net +15V: C17.1, C18.1, C24.1, C25.1, C33.1, C63.1, C79.1, C80.1, C92.+, IC10A.V+, IC11A.V+, IC12A.V+, IC13A.V+, U$2.P$2
- new net +5V: C26.2, C28.2, C29.1, C30.1, C31.1, C32.2, C34.1, C35.1, C36.1, C37.1, C46.2, C48.1, C49.1, C58.2, C59.2, C60.2, C61.2, C62.2, C70.+, IC1.VA+, IC2.VA+, IC3.VA+, IC4.VA+, IC5.VA+, IC6A.V+, IC7A.V+, IC8A.V+, IC9A.V+, U$6.P$2
- new net +5V/1: Q1.S, R37.2, U$12.P$2
- new net -15V: C19.1, C20.1, C21.1, C22.1, C33.2, C63.2, C79.2, C80.2, C96.+, IC10A.V-, IC11A.V-, IC12A.V-, IC13A.V-, U$5.P$2
- new net -5V: C26.1, C28.1, C32.1, C38.1, C39.1, C40.1, C41.1, C42.1, C43.1, C44.1, C46.1, C53.1, C54.1, C58.1, C59.1, C60.1, C61.1, C62.1, C77.-, IC1.VA-, IC2.VA-, IC3.VA-, IC4.VA-, IC5.VA-, IC6A.V-, IC7A.V-, IC8A.V-, IC9A.V-, U$9.P$2
- new net 3V3: C84.1, C85.1, C86.1, C87.+, R34.2, U$11.11, U$11.28, U$11.7, U$13.P$2, X1.4, X3.1
- new net N$79: IC5.VINR, R97.P$1, R99.2
- new net N$80: JP2.2, R97.P$2
- new net N$85: U$2.P$1, X2-12.KL
- new net N$86: U$5.P$1, X2-10.KL
- new net N$88: U$6.P$1, X2-8.KL
- new net N$89: U$9.P$1, X2-6.KL
- new net N$90: U$12.P$1, X2-4.KL
- new net N$91: U$13.P$1, X2-2.KL
- net +5V_PGA: no longer C78.+, C88.+, C89.+, C90.+
- net AGND: now also C17.2, C18.2, C19.2, C20.2, C21.2, C22.2, C24.2, C25.2, C92.-, C96.-, R98.1, R99.1, X2-11.KL, X2-13.KL, X2-7.KL, X2-9.KL, X4-1.KL, X4-10.KL, X4-13.KL, X4-4.KL, X4-7.KL, X5-10.KL, X5-12.KL, X5-14.KL, X5-2.KL, X5-4.KL, X5-6.KL, X5-8.KL; no longer C46.2, C47.2, C51.2, C52.2, C64.-, C65.-, C66.-, C67.-, C68.-, C69.-, C71.+, C72.+, C73.+, C74.+, C75.+, C76.+, X2.6
- net DGND: now also X2-1.KL, X2-3.KL, X2-5.KL; no longer C78.-, C88.-, C89.-, C90.-, X2.1, X3.1
- net FRONT_L: now also X4-2.KL
- net FRONT_R: now also X4-3.KL
- net LINE_L: now also X4-5.KL
- net LINE_R: now also X4-6.KL
- net M_FRONT_L: now also X5-11.KL
- net M_FRONT_R: now also X5-13.KL
- net M_REAR_L: now also X5-7.KL
- net M_REAR_R: now also X5-9.KL
- net N$36: now also R96.P$2; no longer IC5.VINL
- net N$42: now also IC5.VINL, R96.P$1, R98.2; no longer IC5.VINR, JP2.2
- net REAR_L: now also X4-11.KL
- net REAR_R: now also X4-12.KL
- net SPDIF_L: now also X4-8.KL
- net SPDIF_R: now also X4-9.KL
Other:
- moved on the sheet: C46, C70, C77, C84, C85, C86, C87

Commit message: routing
Parts:
- removed X4: inputs, con-3m:2514-
- removed X5: outputs, con-3m:2514-
- added C47, C51, C52, C64: 100n, rcl:C-EUC0805
- added C65, C66: 1n, rcl:C-EUC0805
- added C67, C68: 1u, rcl:C-EUC0805
- added C69: 10u, rcl:CPOL-EU153CLV-0405
- added IC14: PGA2311, Simplex-ICs:PGA2311
- added R101, R102: 1K, rcl:R-EU_R0805W
- added R103, R104, R107, R108: DNP, rcl:R-EU_R0805W
- added R105, R106: 100K, rcl:R-EU_R0805W
- added R92: 47K, rcl:R-EU_R0805W
- added X6: 2514-, con-3m:2514-
- added X7: 2516-, con-3m:2516-
Connections:
- net V_REAR_PAN_L renamed V_CENTER
- net V_REAR_PAN_R renamed V_SW
- removed net N$39: LED2.A, U$11.22
- new net CENTER: C67.1, R103.2, X7-14.KL
- new net CS6: IC14.CS, U$11.16
- new net M6: IC14.MUTE, U$11.15
- new net M_CENTER: IC14.VOUTL, X6-11.KL
- new net M_SW: IC14.VOUTR, X6-13.KL
- new net N$24: C65.2, IC14.VINL, R101.2, R107.2
- new net N$3: IC14.SDO, R92.1
- new net N$34: C66.2, IC14.VINR, R102.2, R108.2
- new net N$6: LED2.A, U$11.1
- new net N$62: C67.2, R101.1, R105.2
- new net N$63: C68.2, R102.1, R106.2
- new net SW: C68.1, R104.2, X7-16.KL
- net +5V: now also C51.2, C52.1, IC14.VA+
- net +5V/1: now also C69.+
- net +5V_PGA: now also C47.1, IC14.VD+, IC14.ZCEN
- net -15V: now also C96.-; no longer C96.+
- net -5V: now also C51.1, C64.1, IC14.VA-
- net AGND: now also C52.2, C64.2, C65.1, C66.1, C96.+, IC14.AGNDL, IC14.AGNDR, R103.1, R104.1, R105.1, R106.1, R107.1, R108.1, X2-5.KL, X6-10.KL, X6-12.KL, X6-14.KL, X6-2.KL, X6-4.KL, X6-6.KL, X6-8.KL, X7-1.KL, X7-10.KL, X7-13.KL, X7-15.KL, X7-4.KL, X7-7.KL; no longer C96.-, X4-1.KL, X4-10.KL, X4-13.KL, X4-4.KL, X4-7.KL, X5-10.KL, X5-12.KL, X5-14.KL, X5-2.KL, X5-4.KL, X5-6.KL, X5-8.KL
- net CLK: now also IC14.SCLK, U$11.32
- net CS2: now also U$11.20
- net CS4: now also U$11.22
- net CS5: now also U$11.18
- net DGND: now also C47.2, C69.-, IC14.DGND, R92.2; no longer X2-5.KL
- net FRONT_L: now also X7-2.KL; no longer X4-2.KL
- net FRONT_R: now also X7-3.KL; no longer X4-3.KL
- net LINE_L: now also X7-5.KL; no longer X4-5.KL
- net LINE_R: now also X7-6.KL; no longer X4-6.KL
- net M2: now also U$11.19
- net M4: now also U$11.21
- net M5: now also U$11.17
- net MOSI: now also IC14.SDI, U$11.30
- net M_FRONT_L: now also X6-5.KL; no longer X5-11.KL
- net M_FRONT_R: now also X6-3.KL; no longer X5-13.KL
- net M_REAR_L: now also X6-9.KL; no longer X5-7.KL
- net M_REAR_R: now also X6-7.KL; no longer X5-9.KL
- net PGA_EN: now also U$11.14
- net REAR_L: now also X7-11.KL; no longer X4-11.KL
- net REAR_R: now also X7-12.KL; no longer X4-12.KL
- net SPDIF_L: now also X7-8.KL; no longer X4-8.KL
- net SPDIF_R: now also X7-9.KL; no longer X4-9.KL
Other:
- note added: "center & sw"
- moved on the sheet: C46, C70, C77, C91, C96, LED2, R33

Commit message: routing
Parts:
- added C71, C72, C73: 100nF, rcl:C-EUC0805
- added C74, C75: (no value), resistor:CPOL-EU153CLV-0405
- added C76, C78, C88, C89, C90, C93, C94, C95: 10u, rcl:CPOL-EU153CLV-0405
- added R100, R109, R110, R111, R112, R93, R94, R95: DNP, rcl:R-EU_R0805W
- added U1: V_REG_LDOSMD, SparkFun-PowerIC:V_REG_LDOSMD
Connections:
- new net N$60: C73.2, U1.BP
- net +5V: now also C76.+, C78.+, C88.+, C89.+
- net +5V/1: now also C71.2, C74.+, U1.EN, U1.IN
- net -5V: now also C90.-, C93.-, C94.-, C95.-
- net 3V3: now also C72.2, C75.+, U1.OUT
- net AGND: now also C76.-, C78.-, C88.-, C89.-, C90.+, C93.+, C94.+, C95.+, R100.1, R109.1, R110.1, R111.1, R112.1, R93.1, R94.1, R95.1
- net DGND: now also C71.1, C72.1, C73.1, C74.-, C75.-, U1.GND
- net N$15: now also R110.2
- net N$16: now also R95.2
- net N$17: now also R94.2
- net N$19: now also R111.2
- net N$26: now also R93.2
- net N$4: now also R112.2
- net N$5: now also R109.2
- net N$7: now also R100.2
Other:
- moved on the sheet: C69, X6-1, X6-10, X6-11, X6-12, X6-13, X6-14, X6-2, X6-3, X6-4, X6-5, X6-6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

Commit message: routing
Parts:
- removed C69: 10u, rcl:CPOL-EU153CLV-0405
- removed X6: 2514-, con-3m:2514-
- removed X7: 2516-, con-3m:2516-
- added C100, C101, C102, C103, C104, C105, C106, C107, C108, C109, C97, C98, C99: 10u, rcl:CPOL-EU153CLV-0405
- added TP1, TP2, TP3, TP4: TEST-POINT3, SparkFun-Passives:TEST-POINT3
- added X4: input, con-3m:2516-5
- added X5: output, con-3m:2514-5
- C74, C75: value (none) -> 10uF
- X2: value 2514- -> 2514-5; device con-3m:2514- -> con-3m:2514-5
Connections:
- net V_CENTER renamed V_FRONT1
- net V_SW renamed V_FRONT2
- net +15V: now also C103.+, C104.+, C105.+, TP1.1
- net +5V: now also C101.+, TP3.1
- net +5V/1: now also C109.+; no longer C69.+
- net +5V_PGA: now also C97.+, C98.+, C99.+
- net -15V: now also C102.-, C106.-, C107.-, TP2.1
- net -5V: now also C100.-, C108.-, TP4.1
- net AGND: now also C100.+, C101.-, C102.+, C103.-, C104.-, C105.-, C106.+, C107.+, C108.+, X2-10.KL, X2-2.KL, X2-4.KL, X2-6.KL, X2-8.KL, X4-1.KL, X4-10.KL, X4-13.KL, X4-15.KL, X4-4.KL, X4-7.KL, X5-10.KL, X5-12.KL, X5-14.KL, X5-2.KL, X5-4.KL, X5-6.KL, X5-8.KL; no longer X2-11.KL, X2-13.KL, X2-5.KL, X2-7.KL, X2-9.KL, X6-10.KL, X6-12.KL, X6-14.KL, X6-2.KL, X6-4.KL, X6-6.KL, X6-8.KL, X7-1.KL, X7-10.KL, X7-13.KL, X7-15.KL, X7-4.KL, X7-7.KL
- net CENTER: now also X4-14.KL; no longer X7-14.KL
- net CS1: now also U$11.36
- net CS3: now also U$11.31
- net DGND: now also C109.-, C97.-, C98.-, C99.-, X2-12.KL, X2-14.KL; no longer C69.-, X2-1.KL, X2-3.KL
- net FRONT_L: now also X4-2.KL; no longer X7-2.KL
- net FRONT_R: now also X4-3.KL; no longer X7-3.KL
- net LINE_L: now also X4-5.KL; no longer X7-5.KL
- net LINE_R: now also X4-6.KL; no longer X7-6.KL
- net M1: now also U$11.35
- net M3: now also U$11.29
- net M_CENTER: now also X5-11.KL; no longer X6-11.KL
- net M_FRONT_L: now also X5-5.KL; no longer X6-5.KL
- net M_FRONT_R: now also X5-3.KL; no longer X6-3.KL
- net M_REAR_L: now also X5-9.KL; no longer X6-9.KL
- net M_REAR_R: now also X5-7.KL; no longer X6-7.KL
- net M_SW: now also X5-13.KL; no longer X6-13.KL
- net N$85: now also X2-3.KL; no longer X2-12.KL
- net N$86: now also X2-5.KL; no longer X2-10.KL
- net N$88: now also X2-7.KL; no longer X2-8.KL
- net N$89: now also X2-9.KL; no longer X2-6.KL
- net N$90: now also X2-11.KL; no longer X2-4.KL
- net N$91: now also X2-13.KL; no longer X2-2.KL
- net REAR_L: now also X4-11.KL; no longer X7-11.KL
- net REAR_R: now also X4-12.KL; no longer X7-12.KL
- net SPDIF_L: now also X4-8.KL; no longer X7-8.KL
- net SPDIF_R: now also X4-9.KL; no longer X7-9.KL
- net SW: now also X4-16.KL; no longer X7-16.KL
Other:
- moved on the sheet: C26, C28, C29, C30, C31, C32, C34, C35, C36, C37, C38, C39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

Commit message: done routing the mixer
Parts:
- removed X2: 2514-5, con-3m:2514-5
- added R113: 0R_0805, Simplex-Jumpers:0R_0805
- added TP5, TP6, TP7: TEST-POINT3, SparkFun-Passives:TEST-POINT3
- added X6: 2512-5, Simplex-Connectors:2512-5
- X5: value output -> 2512-5; device con-3m:2514-5 -> Simplex-Connectors:2512-5
Connections:
- net +5V/1: now also TP5.1
- net +5V_PGA: now also TP7.1
- net 3V3: now also TP6.1
- net AGND: now also R113.P$1, X6-10.KL, X6-12.KL, X6-2.KL, X6-4.KL, X6-6.KL, X6-8.KL; no longer X2-10.KL, X2-2.KL, X2-4.KL, X2-6.KL, X2-8.KL, X5-10.KL, X5-12.KL, X5-14.KL
- net DGND: now also R113.P$2, X5-10.KL, X5-12.KL; no longer X2-12.KL, X2-14.KL
- net M_CENTER: now also X6-9.KL; no longer X5-11.KL
- net M_FRONT_L: now also X6-3.KL; no longer X5-5.KL
- net M_FRONT_R: now also X6-1.KL; no longer X5-3.KL
- net M_REAR_L: now also X6-7.KL; no longer X5-9.KL
- net M_REAR_R: now also X6-5.KL; no longer X5-7.KL
- net M_SW: now also X6-11.KL; no longer X5-13.KL
- net N$85: now also X5-1.KL; no longer X2-3.KL
- net N$86: now also X5-3.KL; no longer X2-5.KL
- net N$88: now also X5-5.KL; no longer X2-7.KL
- net N$89: now also X5-7.KL; no longer X2-9.KL
- net N$90: now also X5-9.KL; no longer X2-11.KL
- net N$91: now also X5-11.KL; no longer X2-13.KL

Commit message: mosfets purchased
Parts:
- removed C27: 220nF, rcl:C-EUC0805
Connections:
- removed net N$13: C27.1, U$11.43
- net DGND: no longer C27.2
Changed lines of the file:
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@@
 <part name="U$11" library="TI_MSP430_v16" deviceset="F55[0/1]X---PT48" device=""/>
 <part name="C23" library="rcl" deviceset="C-EU" device="C0805" value="470nF"/>
-<part name="C27" library="rcl" deviceset="C-EU" device="C0805" value="220nF"/>
 <part name="R22" library="rcl" deviceset="R-EU_" device="R0805W" value="2.2K"/>
 <part name="R27" library="rcl" deviceset="R-EU_" device="R0805W" value="2.2K"/>
@@
 <part name="SUPPLY51" library="supply2" deviceset="DGND" device=""/>
 <part name="SUPPLY52" library="supply2" deviceset="DGND" device=""/>
-<part name="SUPPLY53" library="supply2" deviceset="DGND" device=""/>
 <part name="SUPPLY54" library="supply2" deviceset="DGND" device=""/>
 <part name="SUPPLY55" library="supply2" deviceset="DGND" device=""/>
@@
 <instance part="U$11" gate="G$1" x="81.28" y="63.5"/>
 <instance part="C23" gate="G$1" x="40.64" y="60.96"/>
-<instance part="C27" gate="G$1" x="111.76" y="81.28" rot="R90"/>
 <instance part="R22" gate="G$1" x="114.3" y="58.42" rot="R180"/>
 <instance part="R27" gate="G$1" x="114.3" y="55.88" rot="R180"/>
@@
 <instance part="SUPPLY51" gate="G$1" x="25.4" y="86.36"/>
 <instance part="SUPPLY52" gate="G$1" x="116.84" y="30.48"/>
-<instance part="SUPPLY53" gate="G$1" x="119.38" y="73.66"/>
 <instance part="SUPPLY54" gate="G$1" x="127" y="78.74"/>
 <instance part="SUPPLY55" gate="G$1" x="132.08" y="60.96"/>
@@
 </segment>
 </net>
-<net name="N$13" class="0">
-<segment>
-<pinref part="U$11" gate="G$1" pin="43"/>
-<pinref part="C27" gate="G$1" pin="1"/>
-<wire x1="109.22" y1="81.28" x2="106.68" y2="81.28" width="0.1524" layer="91"/>
-</segment>
-</net>
 <net name="N$14" class="0">
 <segment>
@@
 </segment>
 <segment>
-<pinref part="C27" gate="G$1" pin="2"/>
-<wire x1="116.84" y1="81.28" x2="119.38" y2="81.28" width="0.1524" layer="91"/>
-<wire x1="119.38" y1="81.28" x2="119.38" y2="76.2" width="0.1524" layer="91"/>
-<pinref part="SUPPLY53" gate="G$1" pin="DGND"/>
-</segment>
-<segment>

Commit message: tweak filters
Parts:
- R1, R105, R106, R11, R13, R14, R3, R5, R7, R9: value 100K -> DNP
- R103, R104, R107, R108, R15, R16, R41, R43, R52, R53, R54, R55, R56, R57, R58, R59, R60, R61, R62, R63: value DNP -> 100K
- R33: value 100k -> 47k
Changed lines of the file:
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@@
 <part name="R31" library="rcl" deviceset="R-EU_" device="R0805W" value="47k"/>
 <part name="LED2" library="led" deviceset="LED" device="CHIPLED_0805" value="green"/>
-<part name="R33" library="rcl" deviceset="R-EU_" device="R0805W" value="100k"/>
+<part name="R33" library="rcl" deviceset="R-EU_" device="R0805W" value="47k"/>
 <part name="C57" library="rcl" deviceset="C-EU" device="C0805" value="100nF"/>
 <part name="R37" library="rcl" deviceset="R-EU_" device="R0805W" value="10K"/>
@@
 <part name="C91" library="rcl" deviceset="CPOL-EU" device="153CLV-0405" value="10u"/>
 <part name="C87" library="rcl" deviceset="CPOL-EU" device="153CLV-0405" value="10u"/>
-<part name="R52" library="rcl" deviceset="R-EU_" device="R0805W" value="DNP"/>
+<part name="R52" library="rcl" deviceset="R-EU_" device="R0805W" value="100K"/>
 <part name="SUPPLY65" library="supply2" deviceset="AGND" device=""/>
-<part name="R53" library="rcl" deviceset="R-EU_" device="R0805W" value="DNP"/>
+<part name="R53" library="rcl" deviceset="R-EU_" device="R0805W" value="100K"/>
 <part name="SUPPLY66" library="supply2" deviceset="AGND" device=""/>
-<part name="R54" library="rcl" deviceset="R-EU_" device="R0805W" value="DNP"/>
+<part name="R54" library="rcl" deviceset="R-EU_" device="R0805W" value="100K"/>
 <part name="SUPPLY67" library="supply2" deviceset="AGND" device=""/>
-<part name="R55" library="rcl" deviceset="R-EU_" device="R0805W" value="DNP"/>
+<part name="R55" library="rcl" deviceset="R-EU_" device="R0805W" value="100K"/>
 <part name="SUPPLY68" library="supply2" deviceset="AGND" device=""/>
-<part name="R56" library="rcl" deviceset="R-EU_" device="R0805W" value="DNP"/>
+<part name="R56" library="rcl" deviceset="R-EU_" device="R0805W" value="100K"/>
 <part name="SUPPLY69" library="supply2" deviceset="AGND" device=""/>
-<part name="R57" library="rcl" deviceset="R-EU_" device="R0805W" value="DNP"/>
+<part name="R57" library="rcl" deviceset="R-EU_" device="R0805W" value="100K"/>
 <part name="SUPPLY70" library="supply2" deviceset="AGND" device=""/>
-<part name="R60" library="rcl" deviceset="R-EU_" device="R0805W" value="DNP"/>
+<part name="R60" library="rcl" deviceset="R-EU_" device="R0805W" value="100K"/>
 <part name="SUPPLY73" library="supply2" deviceset="AGND" device=""/>
-<part name="R61" library="rcl" deviceset="R-EU_" device="R0805W" value="DNP"/>
+<part name="R61" library="rcl" deviceset="R-EU_" device="R0805W" value="100K"/>
 <part name="SUPPLY74" library="supply2" deviceset="AGND" device=""/>
 <part name="JP1" library="SparkFun-Connectors" deviceset="M03" device="PTH" value="J1"/>
 <part name="JP2" library="SparkFun-Connectors" deviceset="M03" device="PTH" value="J2"/>
-<part name="R1" library="rcl" deviceset="R-EU_" device="R0805W" value="100K"/>
+<part name="R1" library="rcl" deviceset="R-EU_" device="R0805W" value="DNP"/>
 <part name="SUPPLY21" library="supply2" deviceset="AGND" device=""/>
-<part name="R3" library="rcl" deviceset="R-EU_" device="R0805W" value="100K"/>
+<part name="R3" library="rcl" deviceset="R-EU_" device="R0805W" value="DNP"/>
 <part name="SUPPLY22" library="supply2" deviceset="AGND" device=""/>
-<part name="R5" library="rcl" deviceset="R-EU_" device="R0805W" value="100K"/>
+<part name="R5" library="rcl" deviceset="R-EU_" device="R0805W" value="DNP"/>
 <part name="SUPPLY23" library="supply2" deviceset="AGND" device=""/>
-<part name="R7" library="rcl" deviceset="R-EU_" device="R0805W" value="100K"/>
+<part name="R7" library="rcl" deviceset="R-EU_" device="R0805W" value="DNP"/>
 <part name="SUPPLY24" library="supply2" deviceset="AGND" device=""/>
-<part name="R9" library="rcl" deviceset="R-EU_" device="R0805W" value="100K"/>
+<part name="R9" library="rcl" deviceset="R-EU_" device="R0805W" value="DNP"/>
 <part name="SUPPLY71" library="supply2" deviceset="AGND" device=""/>
-<part name="R11" library="rcl" deviceset="R-EU_" device="R0805W" value="100K"/>
+<part name="R11" library="rcl" deviceset="R-EU_" device="R0805W" value="DNP"/>
 <part name="SUPPLY72" library="supply2" deviceset="AGND" device=""/>
-<part name="R13" library="rcl" deviceset="R-EU_" device="R0805W" value="100K"/>
+<part name="R13" library="rcl" deviceset="R-EU_" device="R0805W" value="DNP"/>
 <part name="SUPPLY75" library="supply2" deviceset="AGND" device=""/>
-<part name="R14" library="rcl" deviceset="R-EU_" device="R0805W" value="100K"/>
+<part name="R14" library="rcl" deviceset="R-EU_" device="R0805W" value="DNP"/>
 <part name="SUPPLY76" library="supply2" deviceset="AGND" device=""/>
-<part name="R15" library="rcl" deviceset="R-EU_" device="R0805W" value="DNP"/>
-<part name="R16" library="rcl" deviceset="R-EU_" device="R0805W" value="DNP"/>
-<part name="R41" library="rcl" deviceset="R-EU_" device="R0805W" value="DNP"/>
-<part name="R43" library="rcl" deviceset="R-EU_" device="R0805W" value="DNP"/>
-<part name="R58" library="rcl" deviceset="R-EU_" device="R0805W" value="DNP"/>
-<part name="R59" library="rcl" deviceset="R-EU_" device="R0805W" value="DNP"/>
-<part name="R62" library="rcl" deviceset="R-EU_" device="R0805W" value="DNP"/>
-<part name="R63" library="rcl" deviceset="R-EU_" device="R0805W" value="DNP"/>
+<part name="R15" library="rcl" deviceset="R-EU_" device="R0805W" value="100K"/>
+<part name="R16" library="rcl" deviceset="R-EU_" device="R0805W" value="100K"/>
+<part name="R41" library="rcl" deviceset="R-EU_" device="R0805W" value="100K"/>
+<part name="R43" library="rcl" deviceset="R-EU_" device="R0805W" value="100K"/>
+<part name="R58" library="rcl" deviceset="R-EU_" device="R0805W" value="100K"/>
+<part name="R59" library="rcl" deviceset="R-EU_" device="R0805W" value="100K"/>
+<part name="R62" library="rcl" deviceset="R-EU_" device="R0805W" value="100K"/>
+<part name="R63" library="rcl" deviceset="R-EU_" device="R0805W" value="100K"/>
 <part name="R67" library="rcl" deviceset="R-EU_" device="R0805W" value="4K7"/>
 <part name="SUPPLY78" library="supply2" deviceset="AGND" device=""/>
@@
 <part name="SUPPLY123" library="supply2" deviceset="AGND" device=""/>
 <part name="IC14" library="Simplex-ICs" deviceset="PGA2311" device=""/>
-<part name="SUPPLY124" library="supply2" deviceset="AGND" device=""/>
-<part name="SUPPLY125" library="supply2" deviceset="AGND" device=""/>
 <part name="SUPPLY126" library="supply2" deviceset="AGND" device=""/>
 <part name="SUPPLY127" library="supply2" deviceset="DGND" device=""/>
@@
 <part name="C67" library="rcl" deviceset="C-EU" device="C0805" value="1u"/>
 <part name="C68" library="rcl" deviceset="C-EU" device="C0805" value="1u"/>
-<part name="R103" library="rcl" deviceset="R-EU_" device="R0805W" value="DNP"/>
+<part name="R103" library="rcl" deviceset="R-EU_" device="R0805W" value="100K"/>
 <part name="SUPPLY137" library="supply2" deviceset="AGND" device=""/>
-<part name="R104" library="rcl" deviceset="R-EU_" device="R0805W" value="DNP"/>
+<part name="R104" library="rcl" deviceset="R-EU_" device="R0805W" value="100K"/>
 <part name="SUPPLY138" library="supply2" deviceset="AGND" device=""/>
-<part name="R105" library="rcl" deviceset="R-EU_" device="R0805W" value="100K"/>
+<part name="R105" library="rcl" deviceset="R-EU_" device="R0805W" value="DNP"/>
 <part name="SUPPLY139" library="supply2" deviceset="AGND" device=""/>
-<part name="R106" library="rcl" deviceset="R-EU_" device="R0805W" value="100K"/>
+<part name="R106" library="rcl" deviceset="R-EU_" device="R0805W" value="DNP"/>
 <part name="SUPPLY140" library="supply2" deviceset="AGND" device=""/>
-<part name="R107" library="rcl" deviceset="R-EU_" device="R0805W" value="DNP"/>
-<part name="R108" library="rcl" deviceset="R-EU_" device="R0805W" value="DNP"/>
+<part name="R107" library="rcl" deviceset="R-EU_" device="R0805W" value="100K"/>
+<part name="R108" library="rcl" deviceset="R-EU_" device="R0805W" value="100K"/>
 <part name="U1" library="SparkFun-PowerIC" deviceset="V_REG_LDO" device="SMD"/>
 <part name="SUPPLY141" library="supply2" deviceset="DGND" device=""/>
@@
 <instance part="SUPPLY123" gate="G$1" x="213.36" y="96.52"/>
 <instance part="IC14" gate="PGA2311" x="231.14" y="40.64"/>
-<instance part="SUPPLY124" gate="G$1" x="116.84" y="-5.08"/>
-<instance part="SUPPLY125" gate="G$1" x="124.46" y="-5.08"/>
 <instance part="SUPPLY126" gate="G$1" x="256.54" y="10.16"/>
 <instance part="SUPPLY127" gate="G$1" x="226.06" y="10.16"/>
