File: hardware/mixer.sch (EAGLE design)
At the start: 261 parts, among them IC1 PGA2311, IC10 OPA2134P, IC11 OPA2134P, IC12 OPA2134P, IC13 OPA2134P, IC14 PGA2311, IC2 PGA2311, IC3 PGA2311, IC4 PGA2311, IC5 PGA2311, IC6 OPA2134P, IC7 OPA2134P, IC8 OPA2134P, IC9 OPA2134P, Q1 SI2305, Q2 MOSFET-NCHANNEL_SOT23-3, U1 V_REG_LDOSMD, X1 MOLEX_6HORIZONTAL, X3 display, X4 input, X5 2512-5, X6 2512-5, Y1 32768Hz CFPX-217 12.5pF

Commit message: small tweaks
Parts:
- removed Q2: MOSFET-NCHANNEL_SOT23-3, Simplex-DiscreteSemi:MOSFET-NCHANNEL_SOT23-3
- removed R79: 0R, rcl:R-EU_R0805W
- added R114: 0R_0805, Simplex-Jumpers:0R_0805
- added T1: BC846, transistor:BC846
- R66: value 0R -> 0R_0805; device rcl:R-EU_R0805W -> Simplex-Jumpers:0R_0805
Connections:
- net DGND: now also T1.E; no longer Q2.S
- net N$4: now also R114.P$1; no longer R66.2
- net N$40: now also T1.C; no longer Q2.D
- net N$41: now also T1.B; no longer Q2.G
- net N$48: now also R114.P$2; no longer R66.1
- net N$50: now also R66.P$2; no longer R79.1
- net N$7: now also R66.P$1; no longer R79.2
Other:
- moved on the sheet: R66
Changed lines of the file:
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@@
 <part name="SUPPLY55" library="supply2" deviceset="DGND" device=""/>
 <part name="X1" library="Simplex-Connectors" deviceset="MOLEX_6" device="HORIZONTAL"/>
-<part name="Q2" library="Simplex-DiscreteSemi" deviceset="MOSFET-NCHANNEL" device="_SOT23-3"/>
 <part name="R38" library="rcl" deviceset="R-EU_" device="R0805W" value="10K"/>
 <part name="R46" library="rcl" deviceset="R-EU_" device="R0805W" value="10K"/>
@@
 <part name="IC6" library="burr-brown" deviceset="OPA2134" device="P"/>
 <part name="IC7" library="burr-brown" deviceset="OPA2134" device="P"/>
-<part name="R66" library="rcl" deviceset="R-EU_" device="R0805W" value="0R"/>
-<part name="R79" library="rcl" deviceset="R-EU_" device="R0805W" value="0R"/>
 <part name="R85" library="rcl" deviceset="R-EU_" device="R0805W" value="DNP"/>
 <part name="SUPPLY77" library="supply2" deviceset="AGND" device=""/>
@@
 <part name="X6" library="Simplex-Connectors" deviceset="2512-" device="5"/>
 <part name="X5" library="Simplex-Connectors" deviceset="2512-" device="5"/>
+<part name="T1" library="transistor" deviceset="BC846" device=""/>
+<part name="R114" library="Simplex-Jumpers" deviceset="0R" device="_0805"/>
+<part name="R66" library="Simplex-Jumpers" deviceset="0R" device="_0805"/>
 </parts>
 <sheets>
@@
 <instance part="IC7" gate="A" x="96.52" y="50.8" rot="R180"/>
 <instance part="IC7" gate="B" x="96.52" y="25.4" rot="R180"/>
-<instance part="R66" gate="G$1" x="96.52" y="66.04" rot="R180"/>
-<instance part="R79" gate="G$1" x="96.52" y="38.1" rot="R180"/>
 <instance part="R85" gate="G$1" x="281.94" y="317.5" rot="R270"/>
 <instance part="SUPPLY77" gate="G$1" x="281.94" y="307.34"/>
@@
 <instance part="X6" gate="-11" x="223.52" y="109.22" rot="MR0"/>
 <instance part="X6" gate="-12" x="223.52" y="111.76" rot="MR0"/>
+<instance part="R114" gate="G$1" x="96.52" y="66.04"/>
+<instance part="R66" gate="G$1" x="96.52" y="38.1"/>
 </instances>
 <busses>
@@
 <pinref part="IC2" gate="PGA2311" pin="VINL"/>
 <pinref part="IC7" gate="A" pin="OUT"/>
-<pinref part="R66" gate="G$1" pin="2"/>
 <wire x1="91.44" y1="66.04" x2="83.82" y2="66.04" width="0.1524" layer="91"/>
 <pinref part="R112" gate="G$1" pin="2"/>
 <wire x1="78.74" y1="20.32" x2="78.74" y2="50.8" width="0.1524" layer="91"/>
 <junction x="78.74" y="50.8"/>
+<pinref part="R114" gate="G$1" pin="P$1"/>
 </segment>
 </net>
@@
 <pinref part="IC2" gate="PGA2311" pin="VINR"/>
 <pinref part="IC7" gate="B" pin="OUT"/>
-<pinref part="R79" gate="G$1" pin="2"/>
 <wire x1="91.44" y1="38.1" x2="83.82" y2="38.1" width="0.1524" layer="91"/>
 <junction x="83.82" y="38.1"/>
@@
 <wire x1="83.82" y1="20.32" x2="83.82" y2="25.4" width="0.1524" layer="91"/>
 <junction x="83.82" y="25.4"/>
+<pinref part="R66" gate="G$1" pin="P$1"/>
 </segment>
 </net>
@@
 <wire x1="104.14" y1="53.34" x2="109.22" y2="53.34" width="0.1524" layer="91"/>
 <pinref part="IC7" gate="A" pin="-IN"/>
-<pinref part="R66" gate="G$1" pin="1"/>
 <wire x1="101.6" y1="66.04" x2="109.22" y2="66.04" width="0.1524" layer="91"/>
+<pinref part="R114" gate="G$1" pin="P$2"/>
 </segment>
 </net>
@@
 <wire x1="109.22" y1="27.94" x2="104.14" y2="27.94" width="0.1524" layer="91"/>
 <pinref part="IC7" gate="B" pin="-IN"/>
-<pinref part="R79" gate="G$1" pin="1"/>
 <wire x1="101.6" y1="38.1" x2="109.22" y2="38.1" width="0.1524" layer="91"/>
+<pinref part="R66" gate="G$1" pin="P$2"/>
 </segment>
 </net>
@@
 <instance part="SUPPLY55" gate="G$1" x="132.08" y="60.96"/>
 <instance part="X1" gate="G$1" x="177.8" y="45.72"/>
-<instance part="Q2" gate="G$1" x="68.58" y="144.78"/>
 <instance part="R38" gate="G$1" x="55.88" y="137.16" rot="R90"/>
 <instance part="R46" gate="G$1" x="45.72" y="144.78" rot="R180"/>
@@
 <instance part="X5" gate="-11" x="187.96" y="124.46" rot="R180"/>
 <instance part="X5" gate="-12" x="187.96" y="127" rot="R180"/>
+<instance part="T1" gate="G$1" x="66.04" y="144.78"/>
 </instances>
 <busses>
@@
 <wire x1="58.42" y1="157.48" x2="68.58" y2="157.48" width="0.1524" layer="91"/>
 <pinref part="Q1" gate="G$1" pin="G"/>
+<pinref part="T1" gate="G$1" pin="C"/>
 <wire x1="68.58" y1="149.86" x2="68.58" y2="157.48" width="0.1524" layer="91"/>
-<pinref part="Q2" gate="G$1" pin="D"/>
 </segment>
 </net>
@@
 </segment>
 <segment>
-<pinref part="SUPPLY46" gate="G$1" pin="DGND"/>
-<pinref part="Q2" gate="G$1" pin="S"/>
-<wire x1="68.58" y1="139.7" x2="68.58" y2="129.54" width="0.1524" layer="91"/>
-</segment>
-<segment>
 <pinref part="R38" gate="G$1" pin="1"/>
 <pinref part="SUPPLY56" gate="G$1" pin="DGND"/>
@@
 <wire x1="218.44" y1="106.68" x2="218.44" y2="101.6" width="0.1524" layer="91"/>
 </segment>
+<segment>
+<pinref part="T1" gate="G$1" pin="E"/>
+<pinref part="SUPPLY46" gate="G$1" pin="DGND"/>
+<wire x1="68.58" y1="139.7" x2="68.58" y2="129.54" width="0.1524" layer="91"/>
+</segment>
 </net>
 <net name="N$41" class="0">
 <segment>
 <pinref part="R46" gate="G$1" pin="1"/>
-<pinref part="Q2" gate="G$1" pin="G"/>
 <wire x1="50.8" y1="144.78" x2="55.88" y2="144.78" width="0.1524" layer="91"/>
 <pinref part="R38" gate="G$1" pin="2"/>
-<wire x1="55.88" y1="144.78" x2="60.96" y2="144.78" width="0.1524" layer="91"/>
+<wire x1="55.88" y1="144.78" x2="63.5" y2="144.78" width="0.1524" layer="91"/>
 <wire x1="55.88" y1="142.24" x2="55.88" y2="144.78" width="0.1524" layer="91"/>
 <junction x="55.88" y="144.78"/>
+<pinref part="T1" gate="G$1" pin="B"/>
 </segment>
 </net>
