File: hardware/mixer.sch (EAGLE design)
At the start: 261 parts, among them IC1 PGA2311, IC10 OPA2134P, IC11 OPA2134P, IC12 OPA2134P, IC13 OPA2134P, IC14 PGA2311, IC2 PGA2311, IC3 PGA2311, IC4 PGA2311, IC5 PGA2311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

Commit message: board rev 1.1
Parts:
- removed R97: 0R_0805, Simplex-Jumpers:0R_0805
- added R79: 10K, rcl:R-EU_R0805W
- R96: value 0R_0805 -> 10K; device Simplex-Jumpers:0R_0805 -> rcl:R-EU_R0805W
- R98, R99: value DNP -> 4K7
Connections:
- net N$36: now also R96.1; no longer R96.P$2
- net N$42: now also R96.2; no longer R96.P$1
- net N$79: now also R79.2; no longer R97.P$1
- net N$80: now also R79.1; no longer R97.P$2
Other:
- moved on the sheet: R96
Changed lines of the file:
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@@
 <part name="SUPPLY91" library="supply2" deviceset="+15V" device=""/>
 <part name="SUPPLY92" library="supply2" deviceset="+15V" device=""/>
-<part name="R96" library="Simplex-Jumpers" deviceset="0R" device="_0805"/>
-<part name="R97" library="Simplex-Jumpers" deviceset="0R" device="_0805"/>
-<part name="R98" library="rcl" deviceset="R-EU_" device="R0805W" value="DNP"/>
-<part name="R99" library="rcl" deviceset="R-EU_" device="R0805W" value="DNP"/>
+<part name="R98" library="rcl" deviceset="R-EU_" device="R0805W" value="4K7"/>
+<part name="R99" library="rcl" deviceset="R-EU_" device="R0805W" value="4K7"/>
 <part name="SUPPLY93" library="supply2" deviceset="AGND" device=""/>
 <part name="SUPPLY94" library="supply2" deviceset="AGND" device=""/>
@@
 <part name="R114" library="Simplex-Jumpers" deviceset="0R" device="_0805"/>
 <part name="R66" library="Simplex-Jumpers" deviceset="0R" device="_0805"/>
+<part name="R79" library="rcl" deviceset="R-EU_" device="R0805W" value="10K"/>
+<part name="R96" library="rcl" deviceset="R-EU_" device="R0805W" value="10K"/>
 </parts>
 <sheets>
@@
 <instance part="SUPPLY91" gate="+15V" x="414.02" y="347.98"/>
 <instance part="SUPPLY92" gate="+15V" x="414.02" y="271.78"/>
-<instance part="R96" gate="G$1" x="88.9" y="124.46"/>
-<instance part="R97" gate="G$1" x="88.9" y="111.76"/>
 <instance part="R98" gate="G$1" x="76.2" y="101.6" rot="R90"/>
 <instance part="R99" gate="G$1" x="81.28" y="101.6" rot="R90"/>
@@
 <instance part="R114" gate="G$1" x="96.52" y="66.04"/>
 <instance part="R66" gate="G$1" x="96.52" y="38.1"/>
+<instance part="R79" gate="G$1" x="88.9" y="111.76" rot="R180"/>
+<instance part="R96" gate="G$1" x="88.9" y="124.46" rot="R180"/>
 </instances>
 <busses>
@@
 <segment>
 <pinref part="JP1" gate="G$1" pin="2"/>
-<pinref part="R96" gate="G$1" pin="P$2"/>
 <wire x1="111.76" y1="124.46" x2="93.98" y2="124.46" width="0.1524" layer="91"/>
+<pinref part="R96" gate="G$1" pin="1"/>
 </segment>
 </net>
 <net name="N$42" class="0">
 <segment>
-<pinref part="R96" gate="G$1" pin="P$1"/>
 <pinref part="IC5" gate="PGA2311" pin="VINL"/>
 <wire x1="83.82" y1="124.46" x2="76.2" y2="124.46" width="0.1524" layer="91"/>
@@
 <wire x1="76.2" y1="106.68" x2="76.2" y2="124.46" width="0.1524" layer="91"/>
 <junction x="76.2" y="124.46"/>
+<pinref part="R96" gate="G$1" pin="2"/>
 </segment>
 </net>
 <net name="N$79" class="0">
 <segment>
-<pinref part="R97" gate="G$1" pin="P$1"/>
 <pinref part="IC5" gate="PGA2311" pin="VINR"/>
 <wire x1="83.82" y1="111.76" x2="81.28" y2="111.76" width="0.1524" layer="91"/>
@@
 <wire x1="81.28" y1="106.68" x2="81.28" y2="111.76" width="0.1524" layer="91"/>
 <junction x="81.28" y="111.76"/>
+<pinref part="R79" gate="G$1" pin="2"/>
 </segment>
 </net>
 <net name="N$80" class="0">
 <segment>
-<pinref part="R97" gate="G$1" pin="P$2"/>
 <pinref part="JP2" gate="G$1" pin="2"/>
 <wire x1="93.98" y1="111.76" x2="111.76" y2="111.76" width="0.1524" layer="91"/>
-</segment>
-</net>
+<pinref part="R79" gate="G$1" pin="1"/>
+</segment>
+</net>

Commit message: new power amp
Parts:
- added JP3: (no value), SparkFun-Passives:JUMPER-2SMD-NO
- added R115, R97: NA/4K7, rcl:R-EU_R0805W
Connections:
- net N$14 renamed P4.5
- net N$21 renamed P4.4
- removed net RX: R22.1, X1.5, X3.2
- removed net TX: R27.1, X1.6, X3.3
- new net N$13: JP3.1, R115.1, R97.1
- new net RX/SDA: R22.1, R97.2, X1.5, X3.2
- new net TX/SCL: R115.2, R27.1, X1.6, X3.3
- net 3V3: now also JP3.2
Other:
- moved on the sheet: X3
Changed lines of the file:
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@@
 <part name="R79" library="rcl" deviceset="R-EU_" device="R0805W" value="10K"/>
 <part name="R96" library="rcl" deviceset="R-EU_" device="R0805W" value="10K"/>
+<part name="R97" library="rcl" deviceset="R-EU_" device="R0805W" value="NA/4K7"/>
+<part name="R115" library="rcl" deviceset="R-EU_" device="R0805W" value="NA/4K7"/>
+<part name="JP3" library="SparkFun-Passives" deviceset="JUMPER-2" device="SMD-NO"/>
 </parts>
 <sheets>
@@
 <instance part="SUPPLY57" gate="G$1" x="144.78" y="30.48"/>
 <instance part="SUPPLY58" gate="G$1" x="172.72" y="30.48"/>
-<instance part="SUPPLY59" gate="G$1" x="165.1" y="60.96"/>
-<instance part="X3" gate="G$1" x="177.8" y="73.66"/>
+<instance part="SUPPLY59" gate="G$1" x="208.28" y="43.18"/>
+<instance part="X3" gate="G$1" x="220.98" y="55.88"/>
 <instance part="SUPPLY113" gate="+15V" x="142.24" y="134.62"/>
 <instance part="SUPPLY114" gate="+5V" x="157.48" y="134.62"/>
@@
 <instance part="U$19" gate="G$1" x="50.8" y="68.58" rot="R90"/>
 <instance part="SUPPLY41" gate="G$1" x="40.64" y="180.34"/>
-<instance part="U$20" gate="G$1" x="162.56" y="78.74"/>
+<instance part="U$20" gate="G$1" x="205.74" y="78.74"/>
 <instance part="U1" gate="G$1" x="170.18" y="180.34"/>
 <instance part="SUPPLY141" gate="G$1" x="152.4" y="165.1"/>
@@
 <instance part="X5" gate="-12" x="187.96" y="127" rot="R180"/>
 <instance part="T1" gate="G$1" x="66.04" y="144.78"/>
+<instance part="R97" gate="G$1" x="190.5" y="66.04" rot="R270"/>
+<instance part="R115" gate="G$1" x="185.42" y="66.04" rot="R270"/>
+<instance part="JP3" gate="A" x="195.58" y="81.28"/>
 </instances>
 <busses>
@@
 </segment>
 </net>
-<net name="N$14" class="0">
+<net name="P4.5" class="0">
 <segment>
 <pinref part="U$11" gate="G$1" pin="34"/>
@@
 </segment>
 </net>
-<net name="N$21" class="0">
+<net name="P4.4" class="0">
 <segment>
 <pinref part="U$11" gate="G$1" pin="33"/>
@@
 </segment>
 </net>
-<net name="RX" class="0">
+<net name="RX/SDA" class="0">
 <segment>
 <pinref part="R22" gate="G$1" pin="1"/>
@@
 </segment>
 <segment>
-<wire x1="175.26" y1="73.66" x2="165.1" y2="73.66" width="0.1524" layer="91"/>
-<label x="165.1" y="73.66" size="1.778" layer="95"/>
+<wire x1="218.44" y1="55.88" x2="190.5" y2="55.88" width="0.1524" layer="91"/>
+<label x="208.28" y="55.88" size="1.778" layer="95"/>
 <pinref part="X3" gate="G$1" pin="2"/>
+<pinref part="R97" gate="G$1" pin="2"/>
+<wire x1="190.5" y1="60.96" x2="190.5" y2="55.88" width="0.1524" layer="91"/>
 </segment>
 </net>
-<net name="TX" class="0">
+<net name="TX/SCL" class="0">
 <segment>
 <pinref part="R27" gate="G$1" pin="1"/>
@@
 </segment>
 <segment>
-<wire x1="175.26" y1="71.12" x2="165.1" y2="71.12" width="0.1524" layer="91"/>
-<label x="165.1" y="71.12" size="1.778" layer="95"/>
+<label x="208.28" y="53.34" size="1.778" layer="95"/>
 <pinref part="X3" gate="G$1" pin="3"/>
+<pinref part="R115" gate="G$1" pin="2"/>
+<wire x1="185.42" y1="60.96" x2="185.42" y2="53.34" width="0.1524" layer="91"/>
+<wire x1="185.42" y1="53.34" x2="218.44" y2="53.34" width="0.1524" layer="91"/>
 </segment>
 </net>
@@
 <segment>
 <pinref part="SUPPLY59" gate="G$1" pin="DGND"/>
-<wire x1="165.1" y1="68.58" x2="165.1" y2="63.5" width="0.1524" layer="91"/>
-<wire x1="175.26" y1="68.58" x2="165.1" y2="68.58" width="0.1524" layer="91"/>
+<wire x1="208.28" y1="50.8" x2="208.28" y2="45.72" width="0.1524" layer="91"/>
+<wire x1="218.44" y1="50.8" x2="208.28" y2="50.8" width="0.1524" layer="91"/>
 <pinref part="X3" gate="G$1" pin="4"/>
 </segment>
@@
 <segment>
 <pinref part="U$20" gate="G$1" pin="3V3"/>
-<wire x1="162.56" y1="78.74" x2="162.56" y2="76.2" width="0.1524" layer="91"/>
 <pinref part="X3" gate="G$1" pin="1"/>
-<wire x1="162.56" y1="76.2" x2="175.26" y2="76.2" width="0.1524" layer="91"/>
+<wire x1="205.74" y1="78.74" x2="205.74" y2="76.2" width="0.1524" layer="91"/>
+<wire x1="205.74" y1="76.2" x2="205.74" y2="58.42" width="0.1524" layer="91"/>
+<wire x1="205.74" y1="58.42" x2="218.44" y2="58.42" width="0.1524" layer="91"/>
+<pinref part="JP3" gate="A" pin="2"/>
+<wire x1="198.12" y1="78.74" x2="198.12" y2="76.2" width="0.1524" layer="91"/>
+<wire x1="198.12" y1="76.2" x2="205.74" y2="76.2" width="0.1524" layer="91"/>
+<junction x="205.74" y="76.2"/>
 </segment>
 <segment>
@@
 </segment>
 </net>
+<net name="N$13" class="0">
+<segment>
+<pinref part="R115" gate="G$1" pin="1"/>
+<pinref part="R97" gate="G$1" pin="1"/>
+<wire x1="190.5" y1="71.12" x2="190.5" y2="76.2" width="0.1524" layer="91"/>
+<wire x1="190.5" y1="76.2" x2="185.42" y2="76.2" width="0.1524" layer="91"/>
+<wire x1="185.42" y1="76.2" x2="185.42" y2="71.12" width="0.1524" layer="91"/>
+<pinref part="JP3" gate="A" pin="1"/>
+<wire x1="190.5" y1="76.2" x2="195.58" y2="76.2" width="0.1524" layer="91"/>
+<wire x1="195.58" y1="76.2" x2="195.58" y2="78.74" width="0.1524" layer="91"/>
+<junction x="190.5" y="76.2"/>
+</segment>
+</net>
