File: hardware/amp.sch (EAGLE design)
At the start: 37 parts, among them X1 2508-5

Commit message: board rev 1.1
Parts:
- C7, C8: device rcl:CPOL-EUF -> rcl:CPOL-EUD
- R10, R12, R13, R14, R15, R3, R4, R5, R6, R8, R9: device rcl:R-EU_0617/17 -> rcl:R-EU_0613/15
- R11, R7: device rcl:R-EU_0922/22 -> rcl:R-EU_0613/15
Connections:
- net IN_L: now also X1-3.KL; no longer X1-1.KL
- net IN_R: now also X1-1.KL; no longer X1-3.KL
- net N$12: now also R11.2; no longer R11.1
- net N$5: now also R7.2; no longer R7.1
- net OUT_L: now also R7.1, X1-7.KL; no longer R7.2, X1-5.KL
- net OUT_R: now also R11.1, X1-5.KL; no longer R11.2, X1-7.KL
Other:
- note added: "1.1"
- note removed: "01"
- moved on the sheet: R11, R7
Changed lines of the file:
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@@
 <part name="U$7" library="SparkFun" deviceset="OSHW-LOGO" device="M"/>
 <part name="GND1" library="supply1" deviceset="GND" device=""/>
-<part name="R3" library="rcl" deviceset="R-EU_" device="0617/17" value="330"/>
+<part name="R3" library="rcl" deviceset="R-EU_" device="0613/15" value="330"/>
 <part name="GND2" library="supply1" deviceset="GND" device=""/>
-<part name="R5" library="rcl" deviceset="R-EU_" device="0617/17" value="3K3"/>
-<part name="R6" library="rcl" deviceset="R-EU_" device="0617/17" value="1K"/>
-<part name="R7" library="rcl" deviceset="R-EU_" device="0922/22" value="0R33"/>
-<part name="R8" library="rcl" deviceset="R-EU_" device="0617/17" value="33K"/>
+<part name="R5" library="rcl" deviceset="R-EU_" device="0613/15" value="3K3"/>
+<part name="R6" library="rcl" deviceset="R-EU_" device="0613/15" value="1K"/>
+<part name="R8" library="rcl" deviceset="R-EU_" device="0613/15" value="33K"/>
 <part name="C4" library="rcl" deviceset="CPOL-EU" device="G" value="100u"/>
 <part name="C5" library="rcl" deviceset="CPOL-EU" device="F" value="47u"/>
-<part name="R9" library="rcl" deviceset="R-EU_" device="0617/17" value="4R7"/>
+<part name="R9" library="rcl" deviceset="R-EU_" device="0613/15" value="4R7"/>
 <part name="GND5" library="supply1" deviceset="GND" device=""/>
-<part name="R4" library="rcl" deviceset="R-EU_" device="0617/17" value="100R"/>
+<part name="R4" library="rcl" deviceset="R-EU_" device="0613/15" value="100R"/>
 <part name="C3" library="rcl" deviceset="CPOL-EU" device="G" value="100u"/>
 <part name="GND6" library="supply1" deviceset="GND" device=""/>
@@
 <part name="C1" library="rcl" deviceset="CPOL-EU" device="B" value="1u"/>
 <part name="GND9" library="supply1" deviceset="GND" device=""/>
-<part name="R11" library="rcl" deviceset="R-EU_" device="0922/22" value="0R33"/>
 <part name="GND11" library="supply1" deviceset="GND" device=""/>
 <part name="R16" library="rcl" deviceset="R-EU_" device="R0805W" value="33K"/>
@@
 <part name="C12" library="rcl" deviceset="C-EU" device="C0805" value="470p"/>
 <part name="C13" library="rcl" deviceset="CPOL-EU" device="B" value="1u"/>
-<part name="R15" library="rcl" deviceset="R-EU_" device="0617/17" value="330"/>
+<part name="R15" library="rcl" deviceset="R-EU_" device="0613/15" value="330"/>
 <part name="GND10" library="supply1" deviceset="GND" device=""/>
-<part name="R13" library="rcl" deviceset="R-EU_" device="0617/17" value="3K3"/>
-<part name="R14" library="rcl" deviceset="R-EU_" device="0617/17" value="1K"/>
-<part name="R12" library="rcl" deviceset="R-EU_" device="0617/17" value="33K"/>
+<part name="R13" library="rcl" deviceset="R-EU_" device="0613/15" value="3K3"/>
+<part name="R14" library="rcl" deviceset="R-EU_" device="0613/15" value="1K"/>
+<part name="R12" library="rcl" deviceset="R-EU_" device="0613/15" value="33K"/>
 <part name="C11" library="rcl" deviceset="CPOL-EU" device="G" value="100u"/>
 <part name="C10" library="rcl" deviceset="CPOL-EU" device="F" value="47u"/>
-<part name="R10" library="rcl" deviceset="R-EU_" device="0617/17" value="4R7"/>
+<part name="R10" library="rcl" deviceset="R-EU_" device="0613/15" value="4R7"/>
 <part name="GND14" library="supply1" deviceset="GND" device=""/>
 <part name="SUPPLY3" library="supply2" deviceset="-24V" device=""/>
 <part name="SUPPLY4" library="supply2" deviceset="-24V" device=""/>
-<part name="C8" library="rcl" deviceset="CPOL-EU" device="F" value="10u"/>
-<part name="C7" library="rcl" deviceset="CPOL-EU" device="F" value="10u"/>
+<part name="C8" library="rcl" deviceset="CPOL-EU" device="D" value="10u"/>
+<part name="C7" library="rcl" deviceset="CPOL-EU" device="D" value="10u"/>
 <part name="R18" library="rcl" deviceset="R-TRIMM" device="3339P" value="20K"/>
 <part name="R19" library="rcl" deviceset="R-TRIMM" device="3339P" value="20K"/>
@@
 <part name="C9" library="capacitor-wima" deviceset="C" device="10/5" value="100n"/>
 <part name="JP1" library="SparkFun-Connectors" deviceset="M03" device="PTH" value="power"/>
+<part name="R7" library="rcl" deviceset="R-EU_" device="0613/15" value="0R33"/>
+<part name="R11" library="rcl" deviceset="R-EU_" device="0613/15" value="0R33"/>
 </parts>
 <sheets>
 <sheet>
 <plain>
-<text x="464.82" y="25.4" size="3.81" layer="97">01</text>
+<text x="464.82" y="25.4" size="3.81" layer="97">1.1</text>
 </plain>
 <instances>
@@
 <instance part="R5" gate="G$1" x="284.48" y="121.92" rot="R90"/>
 <instance part="R6" gate="G$1" x="284.48" y="106.68" rot="R90"/>
-<instance part="R7" gate="G$1" x="294.64" y="154.94" rot="R90"/>
 <instance part="R8" gate="G$1" x="294.64" y="132.08" rot="R180"/>
 <instance part="C4" gate="G$1" x="274.32" y="121.92"/>
@@
 <instance part="C1" gate="G$1" x="231.14" y="149.86" rot="R90"/>
 <instance part="GND9" gate="1" x="279.4" y="73.66"/>
-<instance part="R11" gate="G$1" x="421.64" y="154.94" rot="MR90"/>
 <instance part="GND11" gate="1" x="391.16" y="132.08" rot="MR0"/>
 <instance part="R16" gate="G$1" x="383.54" y="142.24" rot="R90"/>
@@
 <instance part="C9" gate="G$1" x="439.42" y="121.92"/>
 <instance part="JP1" gate="G$1" x="297.18" y="40.64" rot="R180"/>
+<instance part="R7" gate="G$1" x="294.64" y="154.94" rot="R270"/>
+<instance part="R11" gate="G$1" x="421.64" y="154.94" rot="R270"/>
 </instances>
 <busses>
@@
 <net name="N$5" class="0">
 <segment>
-<pinref part="R7" gate="G$1" pin="1"/>
 <wire x1="292.1" y1="144.78" x2="294.64" y2="144.78" width="0.1524" layer="91"/>
 <wire x1="294.64" y1="144.78" x2="294.64" y2="149.86" width="0.1524" layer="91"/>
 <pinref part="U$1" gate="G$1" pin="6"/>
+<pinref part="R7" gate="G$1" pin="2"/>
 </segment>
 </net>
 <net name="OUT_L" class="0">
 <segment>
-<pinref part="R7" gate="G$1" pin="2"/>
 <wire x1="294.64" y1="160.02" x2="294.64" y2="162.56" width="0.1524" layer="91"/>
 <wire x1="294.64" y1="162.56" x2="284.48" y2="162.56" width="0.1524" layer="91"/>
@@
 <pinref part="U$1" gate="G$1" pin="7"/>
 <pinref part="C6" gate="G$1" pin="1"/>
-</segment>
-<segment>
-<pinref part="X1" gate="-5" pin="KL"/>
-<wire x1="228.6" y1="40.64" x2="223.52" y2="40.64" width="0.1524" layer="91"/>
-<label x="223.52" y="40.64" size="1.778" layer="95"/>
+<pinref part="R7" gate="G$1" pin="1"/>
+</segment>
+<segment>
+<pinref part="X1" gate="-7" pin="KL"/>
+<wire x1="228.6" y1="35.56" x2="223.52" y2="35.56" width="0.1524" layer="91"/>
+<label x="223.52" y="35.56" size="1.778" layer="95"/>
 </segment>
 </net>
@@
 <segment>
 <wire x1="421.64" y1="144.78" x2="419.1" y2="144.78" width="0.1524" layer="91"/>
-<pinref part="R11" gate="G$1" pin="1"/>
 <wire x1="421.64" y1="144.78" x2="421.64" y2="149.86" width="0.1524" layer="91"/>
 <pinref part="U$1" gate="G$2" pin="11"/>
+<pinref part="R11" gate="G$1" pin="2"/>
 </segment>
 </net>
@@
 <wire x1="439.42" y1="132.08" x2="439.42" y2="124.46" width="0.1524" layer="91"/>
 <junction x="439.42" y="132.08"/>
-<pinref part="R11" gate="G$1" pin="2"/>
 <wire x1="421.64" y1="160.02" x2="421.64" y2="162.56" width="0.1524" layer="91"/>
 <wire x1="421.64" y1="162.56" x2="411.48" y2="162.56" width="0.1524" layer="91"/>
@@
 <pinref part="U$1" gate="G$2" pin="10"/>
 <pinref part="C9" gate="G$1" pin="1"/>
-</segment>
-<segment>
-<pinref part="X1" gate="-7" pin="KL"/>
-<wire x1="228.6" y1="35.56" x2="223.52" y2="35.56" width="0.1524" layer="91"/>
-<label x="223.52" y="35.56" size="1.778" layer="95"/>
+<pinref part="R11" gate="G$1" pin="1"/>
+</segment>
+<segment>
+<pinref part="X1" gate="-5" pin="KL"/>
+<wire x1="228.6" y1="40.64" x2="223.52" y2="40.64" width="0.1524" layer="91"/>
+<label x="223.52" y="40.64" size="1.778" layer="95"/>
 </segment>
 </net>
@@
 </segment>
 <segment>
-<pinref part="X1" gate="-1" pin="KL"/>
-<wire x1="228.6" y1="50.8" x2="223.52" y2="50.8" width="0.1524" layer="91"/>
-<label x="223.52" y="50.8" size="1.778" layer="95"/>
+<pinref part="X1" gate="-3" pin="KL"/>
+<wire x1="228.6" y1="45.72" x2="223.52" y2="45.72" width="0.1524" layer="91"/>
+<label x="223.52" y="45.72" size="1.778" layer="95"/>
 </segment>
 </net>
@@
 </segment>
 <segment>
-<pinref part="X1" gate="-3" pin="KL"/>
-<wire x1="228.6" y1="45.72" x2="223.52" y2="45.72" width="0.1524" layer="91"/>
-<label x="223.52" y="45.72" size="1.778" layer="95"/>
-</segment>
-</net>
+<pinref part="X1" gate="-1" pin="KL"/>
+<wire x1="228.6" y1="50.8" x2="223.52" y2="50.8" width="0.1524" layer="91"/>
+<label x="223.52" y="50.8" size="1.778" layer="95"/>
+</segment>
+</net>
