File: hardware/amp_lm4780.brd (EAGLE design)
At the start: 100 x 100 mm, 99 parts, among them IC1 OPA2333, IC2 TLC3702, Q1 IRLML6246, Q2 IRLML6246, T1 BC856, X1 2508-5, X2 uC

Commit message: cleanup
Parts:
- C32, C33: value 100nF -> 1nF
- moved C31 2.10 mm to (87.0, 55.0)
- moved R48 2.10 mm to (87.0, 57.0)
Changed lines of the file:
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@@
 <element name="R47" library="rcl" package="R0805W" value="1K" x="92.85" y="52.85" rot="R180"/>
 <element name="C30" library="rcl" package="C0805" value="1nF" x="92.85" y="54.95" rot="R180"/>
-<element name="C31" library="rcl" package="C0805" value="1nF" x="86.95" y="57.05" rot="R180"/>
-<element name="R48" library="rcl" package="R0805W" value="100K" x="86.95" y="54.95" rot="R180"/>
+<element name="C31" library="rcl" package="C0805" value="1nF" x="86.95" y="54.95" rot="R180"/>
+<element name="R48" library="rcl" package="R0805W" value="100K" x="86.95" y="57.05" rot="R180"/>
 <element name="R49" library="rcl" package="R0805W" value="100K" x="92.85" y="57.05" rot="R180"/>
 <element name="C34" library="rcl" package="C1206K" value="10uF" x="88.15" y="77.25" rot="R180"/>
@@
 <element name="D5" library="diode" package="SOD-123_MINI-SMA" value="4148" x="93.7" y="59.65"/>
 <element name="D6" library="diode" package="SOD-123_MINI-SMA" value="1N4148" x="86.4" y="59.65"/>
-<element name="C32" library="rcl" package="C0805" value="100nF" x="30.75" y="94.3" rot="R180"/>
-<element name="C33" library="rcl" package="C0805" value="100nF" x="53.25" y="92.2"/>
+<element name="C32" library="rcl" package="C0805" value="1nF" x="30.75" y="94.3" rot="R180"/>
+<element name="C33" library="rcl" package="C0805" value="1nF" x="53.25" y="92.2"/>
 </elements>
 <signals>
@@
 <contactref element="C31" pad="2"/>
 <contactref element="R48" pad="2"/>
-<wire x1="85.8975" y1="54.95" x2="85.8975" y2="52.85" width="0.4064" layer="1"/>
-<wire x1="85.8975" y1="54.95" x2="86" y2="55.0525" width="0.4064" layer="1"/>
-<wire x1="86" y1="55.0525" x2="86" y2="57.05" width="0.4064" layer="1"/>
 <contactref element="IC1" pad="3"/>
 <wire x1="85.55" y1="66.715" x2="84.415" y2="66.715" width="0.4064" layer="1"/>
@@
 <contactref element="D6" pad="C"/>
 <wire x1="84.6" y1="62.25" x2="84.6" y2="59.65" width="0.4064" layer="1"/>
-<wire x1="86" y1="57.05" x2="86" y2="57.9" width="0.4064" layer="1"/>
-<wire x1="86" y1="57.9" x2="84.6" y2="59.65" width="0.4064" layer="1"/>
+<wire x1="85.8975" y1="52.85" x2="86" y2="52.85" width="0.4064" layer="1"/>
+<wire x1="86" y1="52.85" x2="86" y2="54.95" width="0.4064" layer="1"/>
+<wire x1="86" y1="54.95" x2="85.8975" y2="54.95" width="0.4064" layer="1"/>
+<wire x1="85.8975" y1="54.95" x2="85.8975" y2="57.05" width="0.4064" layer="1"/>
+<wire x1="85.8975" y1="57.9" x2="85.8975" y2="57.05" width="0.4064" layer="1"/>
+<wire x1="85.8975" y1="57.9" x2="84.6" y2="59.1975" width="0.4064" layer="1"/>
+<wire x1="84.6" y1="59.1975" x2="84.6" y2="59.65" width="0.4064" layer="1"/>
 </signal>
 <signal name="N$5">

Commit message: add debug window into ncurses cli
Parts:
- removed R13: 0R_0805, Simplex-Jumpers:R0805W
- added X3: MOLEX_2HORIZONTAL, Simplex-Connectors:0530480210
Connections:
- removed net +3V3D: C1.1, C20.2, C27.2, C34.1, IC1.8, IC2.8, OK2.1, OK2.3, R24.2, R30.2, SJ1.1, X2.2
- new net +3V3A: C1.1, C20.2, C27.2, C34.1, IC1.8, IC2.8, OK2.1, OK2.3, R24.2, R30.2, SJ1.1, X2.2, X3.2
- net GNDI: now also X3.1; no longer R13.1
- net GND_C: no longer R13.2
Routing:
- net +3V3A: track 0.00 -> 120.5 mm, vias 0 -> 4
- net +3V3D: track 118.8 -> 0.00 mm, vias 4 -> 0
- net GNDI: track 20.2 -> 18.3 mm
Changed lines of the file:
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@@
 <element name="R5" library="rcl" package="R0805W" value="1K" x="30.75" y="88" rot="R180"/>
 <element name="R7" library="rcl" package="R0805W" value="1K" x="53.25" y="85.9"/>
-<element name="R13" library="Simplex-Jumpers" package="R0805W" value="0R_0805" x="83.15" y="96.2" rot="R180"/>
 <element name="IC1" library="linear" package="SO08" value="OPA2333" x="88.15" y="67.35" rot="R270"/>
 <element name="R14" library="rcl" package="R0805W" value="10K" x="94.8" y="67.15" rot="R180"/>
@@
 <element name="C32" library="rcl" package="C0805" value="1nF" x="30.75" y="94.3" rot="R180"/>
 <element name="C33" library="rcl" package="C0805" value="1nF" x="53.25" y="92.2"/>
+<element name="X3" library="Simplex-Connectors" package="0530480210" value="MOLEX_2HORIZONTAL" x="93.9" y="73.25" rot="R90"/>
 </elements>
 <signals>
@@
 <wire x1="84.5628" y1="83.15" x2="84.55" y2="83.1628" width="0.3048" layer="1"/>
 <wire x1="92.4" y1="80.2" x2="89.05" y2="83.55" width="0.4064" layer="16"/>
-<contactref element="R13" pad="2"/>
 <wire x1="84.875" y1="92.525" x2="82.3" y2="95.1" width="0.4064" layer="1"/>
 <wire x1="82.3" y1="95.1" x2="82.3" y2="96.19" width="0.4064" layer="1"/>
-<wire x1="82.3" y1="96.19" x2="82.21" y2="96.2" width="0.4064" layer="1"/>
 </signal>
 <signal name="N$40">
@@
 <wire x1="92.6025" y1="88.15" x2="89.15" y2="88.15" width="0.3048" layer="1"/>
 </signal>
-<signal name="+3V3D">
+<signal name="+3V3A">
 <contactref element="R30" pad="2"/>
 <contactref element="OK2" pad="3"/>
-<contactref element="X2" pad="2"/>
 <contactref element="SJ1" pad="1"/>
 <contactref element="IC2" pad="8"/>
@@
 <wire x1="80.8" y1="81.55" x2="80.65" y2="81.55" width="0.3048" layer="16"/>
 <contactref element="C1" pad="1"/>
-<wire x1="93.05" y1="81.45" x2="93.9" y2="81.45" width="0.6096" layer="16"/>
 <wire x1="81.25" y1="94.3" x2="80.4" y2="95.15" width="0.6096" layer="1"/>
 <wire x1="80.4" y1="95.15" x2="64.15" y2="95.15" width="0.6096" layer="1"/>
@@
 <wire x1="80.745" y1="93.795" x2="79.91" y2="93.795" width="0.4064" layer="1"/>
 <wire x1="43" y1="94.35" x2="43" y2="94.3" width="0.4064" layer="1"/>
-<wire x1="93.05" y1="81.45" x2="90.1" y2="84.4" width="0.6096" layer="16"/>
 <wire x1="90.1" y1="84.4" x2="90.1" y2="90.05" width="0.6096" layer="16"/>
 <wire x1="90.1" y1="90.05" x2="85.85" y2="94.3" width="0.6096" layer="16"/>
@@
 <wire x1="94.85" y1="78.75" x2="95.6" y2="79.5" width="0.6096" layer="16"/>
 <wire x1="95.6" y1="79.5" x2="95.6" y2="81.1" width="0.6096" layer="16"/>
-<wire x1="95.6" y1="81.1" x2="95.25" y2="81.45" width="0.6096" layer="16"/>
-<wire x1="95.25" y1="81.45" x2="93.9" y2="81.45" width="0.6096" layer="16"/>
 <wire x1="90.75" y1="69.255" x2="90.7" y2="69.305" width="0.4064" layer="1"/>
 <wire x1="36.1025" y1="92.2" x2="36.6525" y2="92.75" width="0.4064" layer="1"/>
@@
 <wire x1="89.1" y1="71.35" x2="90.9" y2="69.6" width="0.4064" layer="1"/>
 <wire x1="90.9" y1="69.6" x2="91.095" y2="69.6" width="0.4064" layer="1"/>
-<wire x1="92.2" y1="77.25" x2="92.2" y2="69.6" width="0.6096" layer="16"/>
+<wire x1="92.2" y1="77.25" x2="92.2" y2="74.5" width="0.6096" layer="16"/>
+<wire x1="92.2" y1="74.5" x2="92.2" y2="69.6" width="0.6096" layer="16"/>
 <wire x1="93" y1="78.75" x2="92.2" y2="77.95" width="0.6096" layer="16"/>
 <wire x1="92.2" y1="77.95" x2="92.2" y2="77.25" width="0.6096" layer="16"/>
 <wire x1="89.65" y1="77.25" x2="92.2" y2="77.25" width="0.6096" layer="1"/>
+<contactref element="X3" pad="2"/>
+<wire x1="93.9" y1="74.5" x2="92.2" y2="74.5" width="0.6096" layer="16"/>
+<contactref element="X2" pad="2"/>
+<wire x1="90.1" y1="84.4" x2="93.05" y2="81.45" width="0.6096" layer="16"/>
+<wire x1="93.05" y1="81.45" x2="93.9" y2="81.45" width="0.6096" layer="16"/>
+<wire x1="93.9" y1="81.45" x2="95.25" y2="81.45" width="0.6096" layer="16"/>
+<wire x1="95.25" y1="81.45" x2="95.6" y2="81.1" width="0.6096" layer="16"/>
 </signal>
 <signal name="N$21">
@@
 <contactref element="Q2" pad="2"/>
 <wire x1="68.0025" y1="84.1" x2="69.9" y2="84.1" width="0.4064" layer="1"/>
-<contactref element="R13" pad="1"/>
 <contactref element="R20" pad="1"/>
 <contactref element="X1" pad="4"/>
@@
 <wire x1="84.15" y1="35.05" x2="83.9" y2="35.3" width="0.6096" layer="1"/>
 <via x="50.7" y="90.1" extent="1-16" drill="0.4"/>
-<wire x1="84.09" y1="96.2" x2="86" y2="96.2" width="0.6096" layer="1"/>
 <wire x1="67.9" y1="88.8975" x2="68.0025" y2="89" width="0.4064" layer="1"/>
 <contactref element="C33" pad="1"/>
@@
 <wire x1="87.2" y1="71.35" x2="87.6" y2="71" width="0.4064" layer="1"/>
 <wire x1="87.6" y1="71" x2="87.6" y2="69.95" width="0.4064" layer="1"/>
+<contactref element="X3" pad="1"/>
 </signal>
 <signal name="N$32">
