File: hardware/power_pre.brd (EAGLE design)
At the start: 100 x 100 mm, 37 parts, among them X1 2508-5

Commit message: add low voltage power source board
Parts:
- removed JP1: power, SparkFun-Connectors:1X03
- removed R17: 1K, rcl:R0805W
- removed R18, R19: 20K, rcl:RTRIM3339P
- removed R20: 0R_0805, Simplex-Jumpers:R0805W
- removed U$1: STK465HORIZ-BOTTOM, Simplex-ICs:STK465-HB
- removed X1: 2508-5, Simplex-Connectors:PAK100/2500-5-08
- added B1, B2, B3, B4: DF02S, rectifier:DFS
- added C14, C15, C16: 100n, rcl:C0805
- added C17, C18, C19, C20: 10n, rcl:C0805
- added C21: 4700u, rcl:E7,5-16
- added C22, C23, C24, C25: 1u, rcl:PANASONIC_B
- added C26, C27, C28, C29: 150p, capacitor-wima:C5B4.5
- added D1, D10, D2, D3, D4, D5, D6, D7, D8, D9: M4, diode:SMA
- added IC1: 7815, Simplex-ICs:D2PACK
- added IC2: 7915, Simplex-ICs:D2PACK
- added IC3, IC5: 7805, Simplex-ICs:D2PACK
- added IC4: 7905, Simplex-ICs:D2PACK
- C1: value 1u -> 4700uF; device rcl:PANASONIC_B -> rcl:E7,5-18
- C10: value 47u -> 10n; device rcl:PANASONIC_F -> rcl:C0805
- C11: value 100u -> 4700u; device rcl:PANASONIC_G -> rcl:E7,5-16
- C12: value 470p -> 1u; device rcl:C0805 -> rcl:PANASONIC_B
- C13: value 1u -> 100n; device rcl:PANASONIC_B -> rcl:C0805
- C2: value 470p -> 10n
- C3, C4: value 100u -> 10n; device rcl:PANASONIC_G -> rcl:C0805
- C5: value 47u -> 4700uF; device rcl:PANASONIC_F -> rcl:E7,5-18
- C6, C9: value 100n -> 10n; device capacitor-wima:C10B5 -> rcl:C0805
- C7, C8: value 10u -> 10n; device rcl:PANASONIC_F -> rcl:C0805
- R1: value 1K -> 470k
- R10, R9: value 4R7 -> 470k; device rcl:0617/17 -> rcl:R0805W
- R11, R7: value 0R33 -> 470k; device rcl:0922/22 -> rcl:R0805W
- R12, R8: value 33K -> 470k; device rcl:0617/17 -> rcl:R0805W
- R13, R5: value 3K3 -> 470k; device rcl:0617/17 -> rcl:R0805W
- R14, R6: value 1K -> 470k; device rcl:0617/17 -> rcl:R0805W
- R15, R3: value 330 -> 470k; device rcl:0617/17 -> rcl:R0805W
- R16, R2: value 33K -> 470k
- R4: value 100R -> 470k; device rcl:0617/17 -> rcl:R0805W
- moved U$7 101.9 mm to (113.5, 22.6)
- moved R15 95.6 mm to (94.8, 73.0)
- moved C3 91.7 mm to (94.8, 87.0)
- moved R16 90.3 mm to (94.8, 82.9), turned to 90 degrees
- moved C1 83.9 mm to (12.5, 62.9)
- moved C10 82.0 mm to (69.8, 77.1), turned to 90 degrees
- moved C8 79.1 mm to (69.8, 87.0), turned to 90 degrees
- moved R10 76.5 mm to (55.2, 82.9), turned to 270 degrees
- moved C9 72.9 mm to (55.2, 87.0), turned to 270 degrees
- moved R6 72.0 mm to (5.25, 82.9)
- moved R14 71.7 mm to (80.2, 82.9)
- moved R5 71.6 mm to (5.25, 73.0), turned to 270 degrees
- moved R13 71.2 mm to (80.2, 73.0), turned to 270 degrees
- moved R8 70.6 mm to (19.8, 82.9)
- moved R12 67.6 mm to (69.8, 73.0)
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Connections:
- removed net +24V: C7.+, JP1.1, R4.1, U$1.9
- removed net -24V: C8.-, JP1.3, R14.1, R6.1, U$1.12, U$1.5
- removed net GND_I: C12.2, C2.2, R16.1, R18.3, R19.3, R2.1, R20.1, X1.2, X1.4
- removed net IN_L: R18.1, X1.1
- removed net IN_R: R19.1, X1.3
- removed net N$13: C11.-, R15.2
- removed net N$3: C5.-, R5.1, R6.2
- removed net N$4: C6.2, R9.2
- removed net N$5: R7.1, U$1.6
- removed net N$7: R5.2, U$1.4
- removed net OUT_L: C5.+, C6.1, R7.2, R8.1, U$1.7, X1.5
- removed net OUT_R: C10.+, C9.1, R11.2, R12.1, U$1.10, X1.7
- new net +15VA: C12.+, D2.A, D6.C, IC1.3
- new net +5VA: C23.+, D4.A, D5.C, IC3.3
- new net +5VD: C25.+, D10.C, D9.A, IC5.3
- new net -15VA: C22.-, D1.C, D7.C, IC2.3
- new net -5VA: C24.-, D3.C, D8.C, IC4.3
- new net 15VAC_1: B1.AC1, C17.1, C18.2, C26.1
- new net 15VAC_2: B1.AC2, C19.1, C20.2, C26.2
- new net 15VAC_3: B2.AC1, C13.1, C14.2, C27.1
- new net 15VAC_4: B2.AC2, C15.1, C16.2, C27.2
- new net 5VAC_1: B3.AC1, C28.1, C7.1, C8.2
- new net 5VAC_2: B3.AC2, C10.2, C28.2, C9.1
- new net 5VAC_3: B4.AC1, C2.1, C29.1, C3.2
- new net 5VAC_4: B4.AC2, C29.2, C4.1, C6.2
- new net N$16: B2.-, C1.-, D1.A, IC2.4, R7.1, R8.1
- new net N$21: C9.2, R10.1
- new net N$23: C3.1, R16.2
- new net N$24: C2.2, R13.1
- new net N$25: C4.2, R14.1
- new net SPDIF: B3.+, C11.+, D4.C, D9.C, IC3.1, IC5.1, R10.2, R9.2
- net GND: now also B1.-, B2.+, B3.-, B4.+, C1.+, C11.-, C12.-, C21.+, C22.+, C23.-, C24.+, C25.-, C5.-, D10.A, D5.A, D6.A, D7.A, D8.A, IC1.4, IC2.1, IC3.4, IC4.1, IC5.4, R11.1, R12.1, R13.2, R14.2, R2.1, R5.2, R6.2; no longer C3.-, C7.-, C8.+, JP1.2, R10.1, R15.1, R20.2, R9.1, U$1.14, U$1.3, X1.6, X1.8
- net N$1: now also C7.2, R9.1; no longer C4.-, R3.2
- net N$10: now also B4.-, C21.-, D3.A, IC4.4, R15.1, R16.1; no longer C1.+, R18.2
- net N$11: now also C19.2, R4.1; no longer C13.+, R19.2
- net N$12: now also C20.1, R3.2; no longer R11.1, U$1.11
- net N$14: now also C6.1, R15.2; no longer R16.2, R17.1, U$1.16
- net N$15: now also C8.1, R11.2; no longer C12.1, C13.-, R17.2
- net N$17: now also C14.1, R8.2; no longer C11.+, R12.2, U$1.15
- net N$18: now also C16.1, R7.2; no longer C10.-, R13.1, R14.2
- net N$19: now also C15.2, R6.1; no longer R13.2, U$1.13
- net N$2: now also C18.1, R2.2; no longer C4.+, R8.2, U$1.2
- net N$20: now also C10.1, R12.2; no longer C9.2, R10.2
- net N$6: now also C13.2, R5.1; no longer C3.+, R4.2, U$1.8
- net N$8: now also B1.+, C5.+, D2.C, IC1.1, R1.2, R4.2; no longer R1.1, R2.2, U$1.1
- net N$9: now also C17.2, R1.1; no longer C1.-, C2.1, R1.2
Routing:
- net OUT_R: track 117.2 -> 0.00 mm, vias 1 -> 0
- net -24V: track 108.2 -> 0.00 mm, vias 4 -> 0
- net GND: track 25.2 -> 128.0 mm, vias 50 -> 0
- net N$11: track 93.4 -> 2.05 mm, vias 1 -> 0
- net OUT_L: track 91.0 -> 0.00 mm, vias 2 -> 0
- net SPDIF: track 0.00 -> 78.9 mm
- net +24V: track 76.9 -> 0.00 mm, vias 4 -> 0
- net N$16: track 0.00 -> 68.2 mm
- net N$10: track 17.2 -> 84.3 mm
- net N$6: track 43.4 -> 2.05 mm, vias 1 -> 0
- net IN_R: track 40.6 -> 0.00 mm
- net N$17: track 37.8 -> 2.05 mm, vias 1 -> 0
- net GND_I: track 33.7 -> 0.00 mm, vias 23 -> 0
- net N$14: track 32.9 -> 2.05 mm
- net 5VAC_4: track 0.00 -> 28.4 mm, vias 0 -> 1
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- removed copper zone on layer 1, net GND_I
- removed copper zone on layer 16, net GND_I

Commit message: tweaks
Parts:
- added C30, C33: 10uF, rcl:153CLV-0405
- added C31, C32, C34: 100n, rcl:C0805
- added JP1: spdif, SparkFun-Connectors:1X02
- added U$1: DEGSON_8, Simplex-Connectors:DEGSON_8
- added U1: V_REG_LDOSMD, SparkFun-PowerIC:SOT23-5
- added X1: 2512-5, Simplex-Connectors:PAK100/2500-5-12
- moved U$7 64.1 mm to (52.2, 3.95)
- moved C14 5.60 mm to (19.9, 81.3)
- moved C15 5.60 mm to (5.40, 81.3)
- moved C18 5.60 mm to (44.9, 81.3)
- moved C19 5.60 mm to (30.4, 81.3)
- moved C26 5.60 mm to (37.6, 83.8)
- moved C27 5.60 mm to (12.7, 83.8)
- moved C28 5.60 mm to (62.6, 83.8)
- moved C29 5.60 mm to (87.7, 83.8)
- moved C3 5.60 mm to (94.9, 81.3)
- moved C4 5.60 mm to (80.4, 81.3)
- moved C8 5.60 mm to (69.9, 81.3)
- moved C9 5.60 mm to (55.4, 81.3)
- moved R10 5.60 mm to (55.4, 77.3)
- moved R11 5.60 mm to (69.9, 77.3)
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Connections:
- new net +3V3D: C30.+, C32.2, U1.5, X1.11
- new net N$7: C34.2, U1.4
- net +15VA: now also X1.1
- net +5VA: now also X1.5
- net +5VD: now also C31.2, C33.+, U1.1, U1.3, X1.9
- net -15VA: now also X1.3
- net -5VA: now also X1.7
- net 15VAC_1: now also U$1.3
- net 15VAC_2: now also U$1.4
- net 15VAC_3: now also U$1.1
- net 15VAC_4: now also U$1.2
- net 5VAC_1: now also U$1.5
- net 5VAC_2: now also U$1.6
- net 5VAC_3: now also U$1.7
- net 5VAC_4: now also U$1.8
- net GND: now also C30.-, C31.1, C32.1, C33.-, C34.1, JP1.1, U1.2, X1.10, X1.12, X1.2, X1.4, X1.6, X1.8
- net SPDIF: now also JP1.2
Routing:
- net -5VA: track 14.1 -> 132.6 mm, vias 0 -> 6
- net +5VD: track 15.0 -> 120.1 mm, vias 0 -> 7
- net SPDIF: track 78.9 -> 158.7 mm, vias 0 -> 2
- net +5VA: track 13.9 -> 91.9 mm, vias 0 -> 6
- net -15VA: track 17.1 -> 84.4 mm, vias 0 -> 2
- net +15VA: track 14.1 -> 80.4 mm, vias 0 -> 2
- net +3V3D: track 0.00 -> 50.5 mm, vias 0 -> 1
- net 5VAC_3: track 27.1 -> 41.5 mm
- net 15VAC_4: track 27.7 -> 41.9 mm
- net 5VAC_4: track 28.4 -> 40.7 mm
- net 5VAC_1: track 27.4 -> 39.7 mm
- net 15VAC_3: track 27.3 -> 39.6 mm
- net 15VAC_2: track 28.2 -> 40.4 mm
- net 5VAC_2: track 27.9 -> 38.1 mm
- net 15VAC_1: track 27.9 -> 38.2 mm
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Other:
- board text added: "power circuit for mixer board rev 1.0 github.com/rodan/ampy author: petre rodan date: apr 2014"
- board text removed: "2x15W amplifier circuit rev 1.0 github.com/rodan/ampy author: petre rodan date: apr 2014"

Commit message: sent to manufacture
Parts:
- moved U$7 39.8 mm to (12.4, 4.15)
Routing:
- net GND: vias 40 -> 97
Changed lines of the file:
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@@
 <layer number="28" name="bValues" color="7" fill="1" visible="no" active="yes"/>
 <layer number="29" name="tStop" color="7" fill="3" visible="no" active="yes"/>
-<layer number="30" name="bStop" color="7" fill="6" visible="no" active="yes"/>
+<layer number="30" name="bStop" color="7" fill="6" visible="yes" active="yes"/>
 <layer number="31" name="tCream" color="7" fill="4" visible="yes" active="yes"/>
 <layer number="32" name="bCream" color="7" fill="5" visible="yes" active="yes"/>
@@
 <circle x="95" y="5" radius="3.27299375" width="0.4064" layer="42"/>
 <circle x="5" y="5" radius="3.27299375" width="0.4064" layer="42"/>
-<text x="57.8" y="1.65" size="0.8128" layer="108" font="vector" ratio="15">power circuit for mixer board rev 1.0
+<text x="16.2" y="2.3" size="0.8128" layer="108" font="vector" ratio="15">power circuit for mixer board rev 1.0
 github.com/rodan/ampy
 author: petre rodan
@@
 <text x="81.05" y="0.85" size="0.8128" layer="1" font="vector" ratio="20">1   </text>
 <text x="81.95" y="0.85" size="0.8128" layer="16" font="vector" ratio="20">2</text>
+<rectangle x1="36.7" y1="20.35" x2="58.55" y2="34.05" layer="30"/>
+<rectangle x1="63.75" y1="20.35" x2="76.5" y2="34" layer="30"/>
+<rectangle x1="80.1" y1="20.35" x2="98.4" y2="34.05" layer="30"/>
 </plain>
 <attributes>
@@
 </autorouter>
 <elements>
-<element name="U$7" library="SparkFun" package="OSHW-LOGO-M" value="OSHW-LOGOM" x="52.2" y="3.95"/>
+<element name="U$7" library="SparkFun" package="OSHW-LOGO-M" value="OSHW-LOGOM" x="12.45" y="4.15"/>
 <element name="D1" library="diode" package="SMA" value="M4" x="9.45" y="43.5" rot="R180"/>
 <element name="D2" library="diode" package="SMA" value="M4" x="33.35" y="43.5" rot="R180"/>
@@
 <via x="63.85" y="22" extent="1-16" drill="0.6"/>
 <via x="80.55" y="21" extent="1-16" drill="0.6"/>
-<via x="82.95" y="21" extent="1-16" drill="0.6"/>
+<via x="83.25" y="21" extent="1-16" drill="0.6"/>
 <via x="89.7" y="21" extent="1-16" drill="0.6"/>
 <via x="86.4" y="21" extent="1-16" drill="0.6"/>
@@
 <via x="94.4" y="50.55" extent="1-16" drill="0.6"/>
 <contactref element="JP1" pad="1"/>
+<via x="45.55" y="34" extent="1-16" drill="0.6"/>
+<via x="57.65" y="34" extent="1-16" drill="0.6"/>
+<via x="51.55" y="34" extent="1-16" drill="0.6"/>
+<via x="48.5" y="34" extent="1-16" drill="0.6"/>
+<via x="54.6" y="34" extent="1-16" drill="0.6"/>
+<via x="42.25" y="34.05" extent="1-16" drill="0.6"/>
+<via x="51.55" y="21.1" extent="1-16" drill="0.6"/>
+<via x="48.55" y="21.1" extent="1-16" drill="0.6"/>
+<via x="45.4" y="21.1" extent="1-16" drill="0.6"/>
+<via x="54.7" y="21.1" extent="1-16" drill="0.6"/>
+<via x="57.6" y="21.1" extent="1-16" drill="0.6"/>
+<via x="42.15" y="21" extent="1-16" drill="0.6"/>
+<via x="67.9" y="34" extent="1-16" drill="0.6"/>
+<via x="65.25" y="34" extent="1-16" drill="0.6"/>
+<via x="71" y="34" extent="1-16" drill="0.6"/>
+<via x="68.05" y="21" extent="1-16" drill="0.6"/>
+<via x="71.3" y="21" extent="1-16" drill="0.6"/>
+<via x="74.25" y="21" extent="1-16" drill="0.6"/>
+<via x="65.25" y="21" extent="1-16" drill="0.6"/>
+<via x="21.85" y="34.15" extent="1-16" drill="0.6"/>
+<via x="24.6" y="31.6" extent="1-16" drill="0.6"/>
+<via x="6.85" y="32.85" extent="1-16" drill="0.6"/>
+<via x="8.35" y="31.25" extent="1-16" drill="0.6"/>
+<via x="82.05" y="20.05" extent="1-16" drill="0.6"/>
+<via x="84.9" y="20.05" extent="1-16" drill="0.6"/>
+<via x="88.15" y="20.15" extent="1-16" drill="0.6"/>
+<via x="81.85" y="34.4" extent="1-16" drill="0.6"/>
+<via x="84.45" y="34.45" extent="1-16" drill="0.6"/>
 <wire x1="53.3" y1="9.75" x2="49.2" y2="9.3999" width="0" layer="19" extent="1-1"/>
+<via x="40.1" y="30.05" extent="1-16" drill="0.6"/>
+<via x="56.8" y="27.3" extent="1-16" drill="0.6"/>
+<via x="56.85" y="24.55" extent="1-16" drill="0.6"/>
+<via x="40.2" y="27.25" extent="1-16" drill="0.6"/>
+<via x="59.75" y="30.1" extent="1-16" drill="0.6"/>
+<via x="59.75" y="24.55" extent="1-16" drill="0.6"/>
+<via x="40.2" y="24.3" extent="1-16" drill="0.6"/>
+<via x="56.8" y="30.15" extent="1-16" drill="0.6"/>
+<via x="59.75" y="27.3" extent="1-16" drill="0.6"/>
+<via x="73.4" y="27.3" extent="1-16" drill="0.6"/>
+<via x="73.35" y="30.2" extent="1-16" drill="0.6"/>
+<via x="73.35" y="24.4" extent="1-16" drill="0.6"/>
+<via x="59.75" y="32.95" extent="1-16" drill="0.6"/>
+<via x="90.75" y="30.1" extent="1-16" drill="0.6"/>
+<via x="90.85" y="27.05" extent="1-16" drill="0.6"/>
+<via x="90.8" y="23.85" extent="1-16" drill="0.6"/>
+<via x="6.6" y="61.5" extent="1-16" drill="0.6"/>
+<via x="30.95" y="34" extent="1-16" drill="0.6"/>
+<via x="38" y="34.1" extent="1-16" drill="0.6"/>
+<via x="34" y="21.3" extent="1-16" drill="0.6"/>
+<via x="37.7" y="21.2" extent="1-16" drill="0.6"/>
+<via x="43.05" y="30.05" extent="1-16" drill="0.6"/>
+<via x="43" y="27.3" extent="1-16" drill="0.6"/>
+<via x="43.05" y="24.35" extent="1-16" drill="0.6"/>
+<via x="75.65" y="30.2" extent="1-16" drill="0.6"/>
+<via x="75.65" y="27.3" extent="1-16" drill="0.6"/>
+<via x="75.65" y="24.4" extent="1-16" drill="0.6"/>
+<via x="8.45" y="63.35" extent="1-16" drill="0.6"/>
+<via x="12.15" y="63.4" extent="1-16" drill="0.6"/>
 </signal>
 <signal name="+5VA">

Commit message: tweak filters
Parts:
- moved C24 0.15 mm to (79.0, 47.8)
- turned D7 to 180 degrees
- turned D8 to 180 degrees
Connections:
- net -15VA: now also D7.A; no longer D7.C
- net -5VA: now also D8.A; no longer D8.C
- net GND: now also D7.C, D8.C; no longer D7.A, D8.A
Routing:
- net GND: track 128.1 -> 131.2 mm
- net -15VA: track 84.4 -> 86.6 mm
- net -5VA: track 132.6 -> 131.9 mm
Other:
- board text added: "power circuit for mixer board rev 1.1 github.com/rodan/ampy author: petre rodan date: apr 2014"
- board text removed: "power circuit for mixer board rev 1.0 github.com/rodan/ampy author: petre rodan date: apr 2014"
Changed lines of the file:
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@@
 <circle x="95" y="5" radius="3.27299375" width="0.4064" layer="42"/>
 <circle x="5" y="5" radius="3.27299375" width="0.4064" layer="42"/>
-<text x="16.2" y="2.3" size="0.8128" layer="108" font="vector" ratio="15">power circuit for mixer board rev 1.0
+<text x="16.2" y="2.3" size="0.8128" layer="108" font="vector" ratio="15">power circuit for mixer board rev 1.1
 github.com/rodan/ampy
 author: petre rodan
@@
 <element name="B2" library="rectifier" package="DFS" value="DF02S" x="12.65" y="74.4"/>
 <element name="D6" library="diode" package="SMA" value="M4" x="26.05" y="43.5" rot="R180"/>
-<element name="D7" library="diode" package="SMA" value="M4" x="16.75" y="43.5"/>
+<element name="D7" library="diode" package="SMA" value="M4" x="16.75" y="43.5" rot="R180"/>
 <element name="C5" library="rcl" package="E7,5-18" value="4700uF" x="37.65" y="57.3"/>
 <element name="IC1" library="Simplex-ICs" package="D2PACK" value="7815" x="33.35" y="39.4" rot="R180"/>
@@
 <element name="B4" library="rectifier" package="DFS" value="DF02S" x="87.65" y="74.4"/>
 <element name="D5" library="diode" package="SMA" value="M4" x="42.65" y="43.5" rot="R180"/>
-<element name="D8" library="diode" package="SMA" value="M4" x="83.15" y="43.5"/>
+<element name="D8" library="diode" package="SMA" value="M4" x="83.15" y="43.5" rot="R180"/>
 <element name="IC3" library="Simplex-ICs" package="D2PACK" value="7805" x="49.95" y="39.4" rot="R180"/>
 <element name="IC4" library="Simplex-ICs" package="D2PACK" value="7905" x="83.15" y="39.4" rot="R180"/>
@@
 <element name="C22" library="rcl" package="PANASONIC_B" value="1u" x="22.5" y="47.75"/>
 <element name="C23" library="rcl" package="PANASONIC_B" value="1u" x="46.25" y="47.75" rot="R180"/>
-<element name="C24" library="rcl" package="PANASONIC_B" value="1u" x="79.15" y="47.75" rot="R180"/>
+<element name="C24" library="rcl" package="PANASONIC_B" value="1u" x="79" y="47.75" rot="R180"/>
 <element name="C25" library="rcl" package="PANASONIC_B" value="1u" x="57.1" y="47.75"/>
 <element name="R1" library="rcl" package="R0805W" value="470k" x="30.4" y="67.45" rot="R270"/>
@@
 <signal name="-15VA">
 <contactref element="IC2" pad="3"/>
-<contactref element="D7" pad="C"/>
 <contactref element="D1" pad="C"/>
 <contactref element="C22" pad="-"/>
-<wire x1="14.21" y1="43.5" x2="14.75" y2="43.5" width="2.1844" layer="1"/>
 <wire x1="14.21" y1="37.65" x2="14.21" y2="43.5" width="2.1844" layer="1"/>
-<wire x1="14.75" y1="43.5" x2="19" y2="47.75" width="2.1844" layer="1"/>
-<wire x1="19" y1="47.75" x2="20.9" y2="47.75" width="2.1844" layer="1"/>
 <contactref element="X1" pad="3"/>
 <wire x1="7.12" y1="18.89" x2="8.81" y2="18.89" width="1.27" layer="16"/>
@@
 <wire x1="11.45" y1="40.6" x2="11.45" y2="40.65" width="2.1844" layer="1"/>
 <wire x1="11.45" y1="40.65" x2="11.45" y2="43.5" width="2.1844" layer="1"/>
-<wire x1="11.45" y1="43.5" x2="14.21" y2="43.5" width="2.1844" layer="1"/>
+<wire x1="11.45" y1="43.5" x2="13.65" y2="43.5" width="2.1844" layer="1"/>
 <via x="11.45" y="40.65" extent="1-16" drill="0.8"/>
+<wire x1="13.65" y1="43.5" x2="14.21" y2="43.5" width="2.1844" layer="1"/>
 <wire x1="11.45" y1="40.65" x2="24.7" y2="27.4" width="1.27" layer="16"/>
 <wire x1="24.7" y1="27.4" x2="24.7" y2="8.25" width="1.27" layer="16"/>
@@
 <wire x1="12.35" y1="39.7" x2="12.35" y2="39.75" width="1.27" layer="1"/>
 <wire x1="12.35" y1="39.75" x2="11.45" y2="40.65" width="1.27" layer="1"/>
+<contactref element="D7" pad="A"/>
+<wire x1="14.21" y1="43.5" x2="14.21" y2="46.26" width="2.1844" layer="1"/>
+<wire x1="14.21" y1="46.26" x2="15.7" y2="47.75" width="2.1844" layer="1"/>
+<wire x1="15.7" y1="47.75" x2="20.9" y2="47.75" width="2.1844" layer="1"/>
+<wire x1="14.75" y1="43.5" x2="14.21" y2="43.5" width="2.1844" layer="1"/>
 </signal>
 <signal name="5VAC_3">
@@
 <contactref element="D3" pad="C"/>
 <contactref element="C24" pad="-"/>
-<contactref element="D8" pad="C"/>
 <wire x1="80.61" y1="37.65" x2="80.61" y2="43.5" width="2.1844" layer="1"/>
-<wire x1="80.61" y1="43.5" x2="81.15" y2="43.5" width="2.1844" layer="1"/>
-<wire x1="81.15" y1="43.5" x2="77.9" y2="43.5" width="2.1844" layer="1"/>
-<wire x1="81.15" y1="43.5" x2="80.75" y2="43.9" width="2.1844" layer="1"/>
-<wire x1="80.75" y1="43.9" x2="80.75" y2="47.75" width="2.1844" layer="1"/>
 <contactref element="X1" pad="7"/>
 <wire x1="7.12" y1="23.97" x2="10.58" y2="23.97" width="1.27" layer="16"/>
@@
 <wire x1="78.3" y1="39.3" x2="78.3" y2="40.2" width="1.27" layer="1"/>
 <wire x1="78.3" y1="40.2" x2="77.9" y2="40.6" width="1.27" layer="1"/>
+<contactref element="D8" pad="A"/>
+<wire x1="77.9" y1="43.5" x2="80.61" y2="43.5" width="2.1844" layer="1"/>
+<wire x1="80.61" y1="43.5" x2="81.15" y2="43.5" width="2.1844" layer="1"/>
+<wire x1="80.61" y1="47.75" x2="80.61" y2="43.5" width="2.1844" layer="1"/>
+<wire x1="80.6" y1="47.75" x2="80.61" y2="47.75" width="2.1844" layer="1"/>
 </signal>
 <signal name="GND">
 <contactref element="IC5" pad="4"/>
 <contactref element="D10" pad="A"/>
-<contactref element="D8" pad="A"/>
 <contactref element="IC4" pad="1"/>
 <contactref element="D5" pad="A"/>
 <contactref element="IC3" pad="4"/>
-<contactref element="D7" pad="A"/>
 <contactref element="IC2" pad="1"/>
 <contactref element="D6" pad="A"/>
@@
 <via x="81.85" y="34.4" extent="1-16" drill="0.6"/>
 <via x="84.45" y="34.45" extent="1-16" drill="0.6"/>
-<wire x1="53.3" y1="9.75" x2="49.2" y2="9.3999" width="0" layer="19" extent="1-1"/>
 <via x="40.1" y="30.05" extent="1-16" drill="0.6"/>
 <via x="56.8" y="27.3" extent="1-16" drill="0.6"/>
@@
 <via x="8.45" y="63.35" extent="1-16" drill="0.6"/>
 <via x="12.15" y="63.4" extent="1-16" drill="0.6"/>
+<contactref element="D7" pad="C"/>
+<contactref element="D8" pad="C"/>
+<wire x1="49.2" y1="9.3999" x2="49.2" y2="6.35" width="0.6096" layer="1"/>
 </signal>
 <signal name="+5VA">

Commit message: change +5v bridge rectifier in power_pre
Parts:
- B3: value DF02S -> B40S2A-DIO
Changed lines of the file:
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@@
 <element name="C9" library="rcl" package="C0805" value="10n" x="55.4" y="81.35" rot="R270"/>
 <element name="C10" library="rcl" package="C0805" value="10n" x="69.9" y="71.5" rot="R90"/>
-<element name="B3" library="rectifier" package="DFS" value="DF02S" x="62.65" y="74.4"/>
+<element name="B3" library="rectifier" package="DFS" value="B40S2A-DIO" x="62.65" y="74.4"/>
 <element name="B4" library="rectifier" package="DFS" value="DF02S" x="87.65" y="74.4"/>
 <element name="D5" library="diode" package="SMA" value="M4" x="42.65" y="43.5" rot="R180"/>
