File: hardware/power_pre.brd (EAGLE design)
At the start: 100 x 100 mm, 74 parts, among them IC1 7815, IC2 7915, IC3 7805, IC4 7905, IC5 7805, U1 V_REG_LDOSMD, X1 2512-5

Commit message: add debug window into ncurses cli
Parts:
- added JP2: JUMPER-31-2, SparkFun-Passives:SJ_3_PASTE1&2
Connections:
- new net N$4: C31.2, C33.+, JP2.2, U1.1, U1.3
- net +5VA: now also JP2.3
- net +5VD: now also JP2.1; no longer C31.2, C33.+, U1.1, U1.3
Routing:
- net N$4: track 0.00 -> 30.5 mm
- net +5VA: track 91.9 -> 105.9 mm, vias 6 -> 7
- net +5VD: track 120.1 -> 107.1 mm
- net GND: vias 97 -> 99
Changed lines of the file:
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@@
 <element name="C34" library="rcl" package="C0805" value="100n" x="49.2" y="14.5"/>
 <element name="JP1" library="SparkFun-Connectors" package="1X02" value="spdif" x="3.35" y="44.5" rot="R90"/>
+<element name="JP2" library="SparkFun-Passives" package="SJ_3_PASTE1&amp;2" value="JUMPER-31-2" x="42.7" y="17.7" rot="R270"/>
 </elements>
 <signals>
@@
 <wire x1="61.25" y1="45.2" x2="61.25" y2="43.5" width="2.1844" layer="1"/>
 <contactref element="X1" pad="9"/>
-<contactref element="U1" pad="1"/>
-<contactref element="C31" pad="2"/>
-<contactref element="C33" pad="+"/>
-<contactref element="U1" pad="3"/>
 <wire x1="7.12" y1="26.51" x2="11.44" y2="26.51" width="1.27" layer="16"/>
 <wire x1="11.44" y1="26.51" x2="16.85" y2="21.1" width="1.27" layer="16"/>
@@
 <wire x1="61.8" y1="21.4" x2="57.25" y2="16.85" width="1.27" layer="16"/>
 <wire x1="57.25" y1="16.85" x2="56.9" y2="16.85" width="1.27" layer="16"/>
-<wire x1="56.9" y1="16.85" x2="32.15" y2="16.85" width="1.27" layer="16"/>
-<wire x1="48.25" y1="9.3999" x2="48.25" y2="10.7" width="0.6096" layer="1"/>
-<wire x1="48.25" y1="10.7" x2="50.15" y2="10.7" width="0.6096" layer="1"/>
-<wire x1="50.15" y1="10.7" x2="50.15" y2="9.3999" width="0.6096" layer="1"/>
-<wire x1="53.3" y1="11.65" x2="52.1" y2="11.65" width="0.6096" layer="1"/>
-<wire x1="52.1" y1="11.65" x2="51.15" y2="10.7" width="0.6096" layer="1"/>
-<wire x1="51.15" y1="10.7" x2="50.15" y2="10.7" width="0.6096" layer="1"/>
-<wire x1="53.3" y1="11.65" x2="54.15" y2="12.5" width="0.6096" layer="1"/>
-<wire x1="54.15" y1="12.5" x2="57.05" y2="12.5" width="0.6096" layer="1"/>
-<via x="57.05" y="15.95" extent="1-16" drill="0.6"/>
-<wire x1="57.05" y1="15.95" x2="57.05" y2="12.5" width="0.6096" layer="1"/>
-<wire x1="57.05" y1="15.95" x2="57.05" y2="16.85" width="0.6096" layer="16"/>
+<via x="40.55" y="17.8" extent="1-16" drill="0.6"/>
+<wire x1="56.9" y1="16.85" x2="40.75" y2="16.85" width="1.27" layer="16"/>
+<wire x1="40.75" y1="16.85" x2="32.15" y2="16.85" width="1.27" layer="16"/>
 <wire x1="57.05" y1="16.85" x2="56.9" y2="16.85" width="0.6096" layer="16"/>
 <wire x1="61.8" y1="40.1" x2="61.25" y2="40.65" width="1.27" layer="16"/>
@@
 <wire x1="61.8" y1="39.45" x2="61.8" y2="40.1" width="1.27" layer="1"/>
 <wire x1="61.8" y1="40.1" x2="61.25" y2="40.65" width="1.27" layer="1"/>
+<contactref element="JP2" pad="1"/>
+<wire x1="40.55" y1="17.8" x2="40.55" y2="17.05" width="0.6096" layer="16"/>
+<wire x1="40.55" y1="17.05" x2="40.75" y2="16.85" width="0.6096" layer="16"/>
+<wire x1="42.7" y1="18.5128" x2="41.2628" y2="18.5128" width="0.6096" layer="1"/>
+<wire x1="41.2628" y1="18.5128" x2="40.55" y2="17.8" width="0.6096" layer="1"/>
 </signal>
 <signal name="N$10">
@@
 <via x="80.55" y="33.6" extent="1-16" drill="0.6"/>
 <via x="85.6" y="33.6" extent="1-16" drill="0.6"/>
-<via x="36.15" y="13.9" extent="1-16" drill="0.6"/>
+<via x="38" y="12.05" extent="1-16" drill="0.6"/>
 <via x="28.1" y="4.2" extent="1-16" drill="0.6"/>
 <via x="12.45" y="4.15" extent="1-16" drill="0.6"/>
@@
 <contactref element="D8" pad="C"/>
 <wire x1="49.2" y1="9.3999" x2="49.2" y2="6.35" width="0.6096" layer="1"/>
+<via x="44.45" y="13.9" extent="1-16" drill="0.6"/>
+<via x="46.55" y="14.8" extent="1-16" drill="0.6"/>
 </signal>
 <signal name="+5VA">
@@
 <via x="43.3" y="40.5" extent="1-16" drill="0.8"/>
 <wire x1="43.3" y1="40.5" x2="44.65" y2="40.5" width="1.27" layer="1"/>
+<contactref element="JP2" pad="3"/>
+<via x="42.5" y="15" extent="1-16" drill="0.6"/>
+<wire x1="32.1" y1="15" x2="42.5" y2="15" width="0.6096" layer="16"/>
+<wire x1="32.1" y1="15" x2="30.95" y2="13.85" width="0.6096" layer="16"/>
+<wire x1="42.7" y1="16.8872" x2="42.7" y2="15.2" width="0.6096" layer="1"/>
+<wire x1="42.7" y1="15.2" x2="42.5" y2="15" width="0.6096" layer="1"/>
 </signal>
 <signal name="N$2">
@@
 <wire x1="50.15" y1="12.0001" x2="50.15" y2="14.5" width="0.6096" layer="1"/>
 </signal>
+<signal name="N$4">
+<contactref element="U1" pad="3"/>
+<contactref element="JP2" pad="2"/>
+<contactref element="U1" pad="1"/>
+<contactref element="C31" pad="2"/>
+<contactref element="C33" pad="+"/>
+<wire x1="42.7" y1="17.7" x2="54.95" y2="17.7" width="0.6096" layer="1"/>
+<wire x1="54.95" y1="17.7" x2="57.05" y2="15.6" width="0.6096" layer="1"/>
+<wire x1="57.05" y1="15.6" x2="57.05" y2="12.5" width="0.6096" layer="1"/>
+<wire x1="57.05" y1="12.5" x2="54.15" y2="12.5" width="0.6096" layer="1"/>
+<wire x1="54.15" y1="12.5" x2="53.3" y2="11.65" width="0.6096" layer="1"/>
+<wire x1="53.3" y1="11.65" x2="52.35" y2="10.7" width="0.4064" layer="1"/>
+<wire x1="52.35" y1="10.7" x2="50.25" y2="10.7" width="0.4064" layer="1"/>
+<wire x1="50.15" y1="10.7" x2="48.25" y2="10.7" width="0.4064" layer="1"/>
+<wire x1="48.25" y1="10.7" x2="48.25" y2="9.3999" width="0.4064" layer="1"/>
+<wire x1="50.15" y1="9.3999" x2="50.15" y2="10.7" width="0.4064" layer="1"/>
+<wire x1="50.15" y1="10.7" x2="50.25" y2="10.7" width="0.4064" layer="1"/>
+</signal>
 </signals>
